Commit message: edit: techpod.xacro

File: tobas_description/urdf/techpod.xacro (robot description, xacro)
@@ -14,5 +14,6 @@
 <robot name="techpod" xmlns:xacro="http://ros.org/wiki/xacro">
   <!-- Global properties -->
-  <xacro:property name="namespace" value="$(arg namespace)" />
+  <!-- <xacro:property name="namespace" value="$(arg namespace)" /> -->
+  <xacro:property name="namespace" value="techpod" />
   <xacro:property name="rotor_velocity_slowdown_sim" value="10" />
   <xacro:property name="use_mesh" value="true" />
@@ -97,7 +98,8 @@
   </xacro:property>
   <!-- Included URDF Files -->
-  <xacro:include filename="$(find rotors_description)/urdf/fixed_wing_base.xacro" />
+  <!-- <xacro:include filename="$(find rotors_description)/urdf/fixed_wing_base.xacro" /> -->
+  <xacro:include filename="$(find tobas_description)/urdf/fixed_wing_base.xacro" />
   <!-- Instantiate fixed_wing_base_macro once -->
-  <xacro:fixed_wing_base_macro
+  <!-- <xacro:fixed_wing_base_macro
     robot_namespace="${namespace}"
     mass="${mass_fuselage}"
@@ -113,5 +115,22 @@
     <origin xyz="0 0 0" rpy="0 0 0" />
     <xacro:insert_block name="body_inertia" />
+  </xacro:fixed_wing_base_macro> -->
+  <!-- Added from here -->
+  <xacro:fixed_wing_base_macro
+    robot_namespace="${namespace}"
+    mass="${mass_fuselage}"
+    length="${body_length}"
+    width="${body_width}"
+    height="${body_height}"
+    color="${body_color}"
+    use_mesh_file="${use_mesh}"
+    mesh_file="${body_mesh_file}"
+    aero_params_yaml="hoge"
+    vehicle_params_yaml="fuga"
+    is_input_joystick="piyo">
+    <origin xyz="0 0 0" rpy="0 0 0" />
+    <xacro:insert_block name="body_inertia" />
   </xacro:fixed_wing_base_macro>
+  <!-- Added to here -->
   <!-- Instantiate the ailerons -->
   <xacro:control_surface

Commit message: edit: techpod.xacro
ホイールを追加
プロペラの回転軸をX軸正方向に

File: tobas_description/urdf/techpod.xacro (robot description, xacro)
@@ -120,4 +120,80 @@
   </xacro:fixed_wing_base_macro>
   <!-- Added to here -->
+  <!-- Instantiate the wheels -->
+	<joint name="techpod/wheel_left_joint" type="continuous">
+		<parent link="techpod/base_link"/>
+		<child link="techpod/wheel_left"/>
+		<origin xyz="0.3 0.2 -0.2" rpy="1.5707963267948966 0 0" />
+		<axis xyz="0 0 1" />
+	</joint>
+	<link name="techpod/wheel_left">
+		<inertial>
+			<mass value="1e-3" />
+			<inertia ixx="1e-3" ixy="0" ixz="0" iyy="1e-3" iyz="0" izz="1e-3" />
+		</inertial>
+		<visual>
+			<geometry>
+				<cylinder length="0.025" radius="0.05"/>
+			</geometry>
+		</visual>
+		<collision>
+			<geometry>
+				<cylinder length="0.025" radius="0.05"/>
+			</geometry>
+		</collision>
+	</link>
+	<gazebo reference="techpod/wheel_left">
+		<material>Gazebo/Black</material>
+	</gazebo>
+	<joint name="techpod/wheel_right_joint" type="continuous">
+		<parent link="techpod/base_link"/>
+		<child link="techpod/wheel_right"/>
+		<origin xyz="0.3 -0.2 -0.2" rpy="1.5707963267948966 0 0" />
+		<axis xyz="0 0 1" />
+	</joint>
+	<link name="techpod/wheel_right">
+		<inertial>
+			<mass value="1e-3" />
+			<inertia ixx="1e-3" ixy="0" ixz="0" iyy="1e-3" iyz="0" izz="1e-3" />
+		</inertial>
+		<visual>
+			<geometry>
+				<cylinder length="0.025" radius="0.05"/>
+			</geometry>
+		</visual>
+		<collision>
+			<geometry>
+				<cylinder length="0.025" radius="0.05"/>
+			</geometry>
+		</collision>
+	</link>
+	<gazebo reference="techpod/wheel_right">
+		<material>Gazebo/Black</material>
+	</gazebo>
+	<joint name="techpod/wheel_rear_joint" type="continuous">
+		<parent link="techpod/base_link"/>
+		<child link="techpod/wheel_rear"/>
+		<origin xyz="-0.3 0 -0.2" rpy="1.5707963267948966 0 0" />
+		<axis xyz="0 0 1" />
+	</joint>
+	<link name="techpod/wheel_rear">
+		<inertial>
+			<mass value="1e-3" />
+			<inertia ixx="1e-3" ixy="0" ixz="0" iyy="1e-3" iyz="0" izz="1e-3" />
+		</inertial>
+		<visual>
+			<geometry>
+				<cylinder length="0.025" radius="0.05"/>
+			</geometry>
+		</visual>
+		<collision>
+			<geometry>
+				<cylinder length="0.025" radius="0.05"/>
+			</geometry>
+		</collision>
+	</link>
+	<gazebo reference="techpod/wheel_rear">
+		<material>Gazebo/Black</material>
+	</gazebo>
   <!-- Instantiate the ailerons -->
   <xacro:control_surface
@@ -242,5 +318,5 @@
     use_mesh_file="${use_mesh}"
     mesh_file="${propeller_mesh_file}">
-    <origin xyz="-0.025 0 0.15" rpy="0 ${-0.5*PI} 0" />
+    <origin xyz="-0.025 0 0.15" rpy="0 ${0.5*PI} 0" />
     <xacro:insert_block name="propeller_inertia" />
   </xacro:propeller>

Commit message: 制御面候補の条件で関節リミットもチェック

File: tobas_description/urdf/techpod.xacro (robot description, xacro)
@@ -7,4 +7,5 @@
   <!-- Constants -->
   <xacro:property name="PI" value="3.1415926535897931" />
+  <xacro:property name="DEG2RAD" value="${PI / 180.0}" />
   <!-- Component masses -->
   <xacro:property name="mass_fuselage" value="2.05" /> <!-- [kg] -->
@@ -24,6 +25,6 @@
   <xacro:property name="aileron_width" value="0.349" /> <!-- [m] -->
   <xacro:property name="aileron_height" value="0.013" /> <!-- [m] -->
-  <xacro:property name="aileron_min_angle" value="-0.349066" /> <!-- [rad] -->
-  <xacro:property name="aileron_max_angle" value="0.349066" /> <!-- [rad] -->
+  <xacro:property name="aileron_min_angle" value="-${20.0 * DEG2RAD}" /> <!-- [rad] -->
+  <xacro:property name="aileron_max_angle" value="${20.0 * DEG2RAD}" /> <!-- [rad] -->
   <xacro:property name="aileron_max_velocity" value="10.0" /> <!-- [rad/s] -->
   <xacro:property name="aileron_max_effort" value="1e+6" /> <!-- [Nm] -->
@@ -35,6 +36,6 @@
   <xacro:property name="elevator_width" value="0.457" /> <!-- [m] -->
   <xacro:property name="elevator_height" value="0.012" /> <!-- [m] -->
-  <xacro:property name="elevator_min_angle" value="-0.349066" /> <!-- [rad] -->
-  <xacro:property name="elevator_max_angle" value="0.349066" /> <!-- [rad] -->
+  <xacro:property name="elevator_min_angle" value="-${20.0 * DEG2RAD}" /> <!-- [rad] -->
+  <xacro:property name="elevator_max_angle" value="${20.0 * DEG2RAD}" /> <!-- [rad] -->
   <xacro:property name="elevator_max_velocity" value="10.0" /> <!-- [rad/s] -->
   <xacro:property name="elevator_max_effort" value="1e+6" /> <!-- [Nm] -->
@@ -45,6 +46,6 @@
   <xacro:property name="flap_width" value="0.459" /> <!-- [m] -->
   <xacro:property name="flap_height" value="0.016" /> <!-- [m] -->
-  <xacro:property name="flap_min_angle" value="0.0" /> <!-- [rad] -->
-  <xacro:property name="flap_max_angle" value="0.0" /> <!-- [rad] -->
+  <xacro:property name="flap_min_angle" value="-${20.0 * DEG2RAD}" /> <!-- [rad] -->
+  <xacro:property name="flap_max_angle" value="${20.0 * DEG2RAD}" /> <!-- [rad] -->
   <xacro:property name="flap_max_velocity" value="10.0" /> <!-- [rad/s] -->
   <xacro:property name="flap_max_effort" value="1e+6" /> <!-- [Nm] -->
@@ -56,6 +57,6 @@
   <xacro:property name="rudder_width" value="0.018" />
   <xacro:property name="rudder_height" value="0.241" />
-  <xacro:property name="rudder_min_angle" value="-0.349066" />
-  <xacro:property name="rudder_max_angle" value="0.349066" />
+  <xacro:property name="rudder_min_angle" value="-${20.0 * DEG2RAD}" />
+  <xacro:property name="rudder_max_angle" value="${20.0 * DEG2RAD}" />
   <xacro:property name="rudder_max_velocity" value="10.0" />
   <xacro:property name="rudder_max_effort" value="1e+6" />
@@ -90,5 +91,5 @@
   <!-- Inertia of the propeller, assuming it is a cylinder -->
   <xacro:property name="propeller_inertia">
-    <xacro:cylinder_inertia r="${propeller_radius}" h="${propeller_height}" mass="${mass_propeller*rotor_velocity_slowdown_sim}" />
+    <xacro:cylinder_inertia r="${propeller_radius}" h="${propeller_height}" mass="${mass_propeller * rotor_velocity_slowdown_sim}" />
   </xacro:property>
   <!-- Included URDF Files -->
@@ -338,5 +339,5 @@
     use_mesh_file="${use_mesh}"
     mesh_file="${propeller_mesh_file}">
-    <origin xyz="-0.025 0 0.15" rpy="0 ${0.5*PI} 0" />
+    <origin xyz="-0.025 0 0.15" rpy="0 ${0.5 * PI} 0" />
     <xacro:insert_block name="propeller_inertia" />
   </xacro:propeller>
