Commit message: techpodのURDFに関節制限をつける

File: tobas_description/urdf/fixed_wing_base.xacro (robot description, xacro)
@@ -55,5 +55,5 @@
   <xacro:macro name="control_surface"
     params="robot_namespace surface_name parent mass_surface min_angle
-      max_angle color use_mesh_file mesh_file surface_length surface_width
+      max_angle max_velocity max_effort color use_mesh_file mesh_file surface_length surface_width
       surface_height *axis *joint_origin *link_origin *inertia">
     <joint name="${robot_namespace}/${surface_name}_joint" type="revolute">
@@ -62,5 +62,5 @@
       <parent link="${parent}" />
       <child link="${robot_namespace}/${surface_name}" />
-      <limit upper="0" lower="0" effort="0" velocity="0" />
+      <limit lower="${min_angle}" upper="${max_angle}" velocity="${max_velocity}" effort="${max_effort}" />
     </joint>
     <link name="${robot_namespace}/${surface_name}">

File: tobas_description/urdf/techpod.xacro (robot description, xacro)
@@ -26,4 +26,6 @@
   <xacro:property name="aileron_min_angle" value="-0.349066" /> <!-- [rad] -->
   <xacro:property name="aileron_max_angle" value="0.349066" /> <!-- [rad] -->
+  <xacro:property name="aileron_max_velocity" value="10.0" /> <!-- [rad/s] -->
+  <xacro:property name="aileron_max_effort" value="1e+6" /> <!-- [Nm] -->
   <xacro:property name="aileron_color" value="Red" />
   <xacro:property name="aileron_left_mesh_file" value="package://tobas_description/meshes/techpod/techpod_aileron_left.dae" />
@@ -35,4 +37,6 @@
   <xacro:property name="elevator_min_angle" value="-0.349066" /> <!-- [rad] -->
   <xacro:property name="elevator_max_angle" value="0.349066" /> <!-- [rad] -->
+  <xacro:property name="elevator_max_velocity" value="10.0" /> <!-- [rad/s] -->
+  <xacro:property name="elevator_max_effort" value="1e+6" /> <!-- [Nm] -->
   <xacro:property name="elevator_color" value="Blue" />
   <xacro:property name="elevator_mesh_file" value="package://tobas_description/meshes/techpod/techpod_elevator.dae" />
@@ -43,4 +47,6 @@
   <xacro:property name="flap_min_angle" value="0.0" /> <!-- [rad] -->
   <xacro:property name="flap_max_angle" value="0.0" /> <!-- [rad] -->
+  <xacro:property name="flap_max_velocity" value="10.0" /> <!-- [rad/s] -->
+  <xacro:property name="flap_max_effort" value="1e+6" /> <!-- [Nm] -->
   <xacro:property name="flap_color" value="Yellow" />
   <xacro:property name="flap_left_mesh_file" value="package://tobas_description/meshes/techpod/techpod_flap_left.dae" />
@@ -52,4 +58,6 @@
   <xacro:property name="rudder_min_angle" value="-0.349066" />
   <xacro:property name="rudder_max_angle" value="0.349066" />
+  <xacro:property name="rudder_max_velocity" value="10.0" />
+  <xacro:property name="rudder_max_effort" value="1e+6" />
   <xacro:property name="rudder_color" value="Orange" />
   <xacro:property name="rudder_mesh_file" value="package://tobas_description/meshes/techpod/techpod_rudder.dae" />
@@ -204,4 +212,6 @@
     min_angle="${aileron_min_angle}"
     max_angle="${aileron_max_angle}"
+    max_velocity="${aileron_max_velocity}"
+    max_effort="${aileron_max_effort}"
     color="${aileron_color}"
     use_mesh_file="${use_mesh}"
@@ -222,4 +232,6 @@
     min_angle="${aileron_min_angle}"
     max_angle="${aileron_max_angle}"
+    max_velocity="${aileron_max_velocity}"
+    max_effort="${aileron_max_effort}"
     color="${aileron_color}"
     use_mesh_file="${use_mesh}"
@@ -241,4 +253,6 @@
     min_angle="${elevator_min_angle}"
     max_angle="${elevator_max_angle}"
+    max_velocity="${elevator_max_velocity}"
+    max_effort="${elevator_max_effort}"
     color="${elevator_color}"
     use_mesh_file="${use_mesh}"
@@ -260,4 +274,6 @@
     min_angle="${flap_min_angle}"
     max_angle="${flap_max_angle}"
+    max_velocity="${flap_max_velocity}"
+    max_effort="${flap_max_effort}"
     color="${flap_color}"
     use_mesh_file="${use_mesh}"
@@ -278,4 +294,6 @@
     min_angle="${flap_min_angle}"
     max_angle="${flap_max_angle}"
+    max_velocity="${flap_max_velocity}"
+    max_effort="${flap_max_effort}"
     color="${flap_color}"
     use_mesh_file="${use_mesh}"
@@ -297,4 +315,6 @@
     min_angle="${rudder_min_angle}"
     max_angle="${rudder_max_angle}"
+    max_velocity="${rudder_max_velocity}"
+    max_effort="${rudder_max_effort}"
     color="${rudder_color}"
     use_mesh_file="${use_mesh}"

Commit message: techpodのwheelをマクロに

File: tobas_description/urdf/fixed_wing_base.xacro (robot description, xacro)
@@ -3,19 +3,19 @@
   <!-- Macro for the inertia of a box -->
   <xacro:macro name="box_inertia" params="x y z mass">
-    <inertia ixx="${0.0833333 * mass * (y*y + z*z)}" ixy="0.0" ixz="0.0"
-      iyy="${0.0833333 * mass * (x*x + z*z)}" iyz="0.0"
-      izz="${0.0833333 * mass * (x*x + y*y)}" />
+    <inertia ixx="${0.0833333 * mass * (y*y + z*z)}" ixy="0.0" ixz="0.0" iyy="${0.0833333 * mass * (x*x + z*z)}" iyz="0.0" izz="${0.0833333 * mass * (x*x + y*y)}" />
   </xacro:macro>
   <!-- Macro for the inertia of a cylinder -->
   <xacro:macro name="cylinder_inertia" params="r h mass">
-    <inertia ixx="${0.0833333 * mass * (3*r*r + h*h)}" ixy="0.0" ixz="0.0"
-      iyy="${0.0833333 * mass * (3*r*r + h*h)}" iyz="0.0"
-      izz="${0.5 * mass * r * r}" />
+    <inertia ixx="${0.0833333 * mass * (3*r*r + h*h)}" ixy="0.0" ixz="0.0" iyy="${0.0833333 * mass * (3*r*r + h*h)}" iyz="0.0" izz="${0.5 * mass * r * r}" />
   </xacro:macro>
   <!-- Fixed-wing main body link -->
-  <xacro:macro name="fixed_wing_base_macro"
-    params="robot_namespace mass length width height color use_mesh_file
-      mesh_file aero_params_yaml vehicle_params_yaml is_input_joystick
-      *origin *inertia">
+  <xacro:macro name="fixed_wing_base_macro" params="robot_namespace
+      mass length
+      width height
+      color
+      use_mesh_file
+      mesh_file
+      *origin
+      *inertia">
     <link name="${robot_namespace}/base_link"></link>
     <joint name="${robot_namespace}/base_joint" type="fixed">
@@ -53,8 +53,22 @@
   </xacro:macro>
   <!-- Control surface joint and link -->
-  <xacro:macro name="control_surface"
-    params="robot_namespace surface_name parent mass_surface min_angle
-      max_angle max_velocity max_effort color use_mesh_file mesh_file surface_length surface_width
-      surface_height *axis *joint_origin *link_origin *inertia">
+  <xacro:macro name="control_surface" params="robot_namespace
+      surface_name
+      parent
+      mass_surface
+      min_angle
+      max_angle
+      max_velocity
+      max_effort
+      color
+      use_mesh_file
+      mesh_file
+      surface_length
+      surface_width
+      surface_height
+      *axis
+      *joint_origin
+      *link_origin
+      *inertia">
     <joint name="${robot_namespace}/${surface_name}_joint" type="revolute">
       <xacro:insert_block name="joint_origin" />
@@ -98,7 +112,14 @@
   </xacro:macro>
   <!-- Propeller joint and link -->
-  <xacro:macro name="propeller"
-    params="robot_namespace suffix parent mass_propeller propeller_radius color
-      use_mesh_file mesh_file *origin *inertia">
+  <xacro:macro name="propeller" params="robot_namespace
+      suffix
+      parent
+      mass_propeller
+      propeller_radius
+      color
+      use_mesh_file
+      mesh_file
+      *origin
+      *inertia">
     <joint name="${robot_namespace}/propeller_{suffix}_joint" type="continuous">
       <xacro:insert_block name="origin" />
@@ -115,6 +136,5 @@
         <geometry>
           <xacro:if value="${use_mesh_file}">
-            <mesh filename="${mesh_file}"
-              scale="${propeller_radius} ${propeller_radius} ${propeller_radius}" />
+            <mesh filename="${mesh_file}" scale="${propeller_radius} ${propeller_radius} ${propeller_radius}" />
           </xacro:if>
           <xacro:unless value="${use_mesh_file}">
@@ -126,6 +146,5 @@
         <geometry>
           <xacro:if value="${use_mesh_file}">
-            <mesh filename="${mesh_file}"
-              scale="${propeller_radius} ${propeller_radius} ${propeller_radius}" />
+            <mesh filename="${mesh_file}" scale="${propeller_radius} ${propeller_radius} ${propeller_radius}" />
           </xacro:if>
           <xacro:unless value="${use_mesh_file}">
@@ -139,3 +158,39 @@
     </gazebo>
   </xacro:macro>
+  <!-- Wheel joint and link -->
+  <xacro:macro name="wheel" params="robot_namespace
+      suffix
+      parent
+      mass
+      height
+      radius
+      color
+      *origin
+      *inertia">
+    <joint name="techpod/wheel_${suffix}_joint" type="continuous">
+      <parent link="${parent}"/>
+      <child link="techpod/wheel_${suffix}"/>
+      <xacro:insert_block name="origin" />
+      <axis xyz="0 0 1" />
+    </joint>
+    <link name="techpod/wheel_${suffix}">
+      <inertial>
+        <mass value="${mass}" />
+        <xacro:insert_block name="inertia" />
+      </inertial>
+      <visual>
+        <geometry>
+          <cylinder length="${height}" radius="${radius}"/>
+        </geometry>
+      </visual>
+      <collision>
+        <geometry>
+          <cylinder length="${height}" radius="${radius}"/>
+        </geometry>
+      </collision>
+    </link>
+    <gazebo reference="techpod/wheel_${suffix}">
+      <material>Gazebo/${color}</material>
+    </gazebo>
+  </xacro:macro>
 </robot>

File: tobas_description/urdf/multirotor_base.xacro (robot description, xacro)
@@ -14,5 +14,11 @@
   </xacro:macro>
   <!-- Main multirotor link -->
-  <xacro:macro name="multirotor_base_macro" params="robot_namespace mass body_width body_height use_mesh_file mesh_file *inertia">
+  <xacro:macro name="multirotor_base_macro" params="robot_namespace
+      mass
+      body_width
+      body_height
+      use_mesh_file
+      mesh_file
+      *inertia">
     <link name="${robot_namespace}/base_link"></link>
     <joint name="${robot_namespace}/base_joint" type="fixed">
@@ -47,5 +53,15 @@
   </xacro:macro>
   <!-- Rotor joint and link -->
-  <xacro:macro name="vertical_rotor" params="robot_namespace direction parent mass_rotor radius_rotor motor_number color use_own_mesh mesh *origin *inertia">
+  <xacro:macro name="vertical_rotor" params="robot_namespace
+      direction
+      parent
+      mass_rotor
+      radius_rotor
+      motor_number
+      color
+      use_own_mesh
+      mesh
+      *origin
+      *inertia">
     <joint name="${robot_namespace}/rotor_${motor_number}_joint" type="continuous">
       <xacro:insert_block name="origin" />

File: tobas_description/urdf/techpod.xacro (robot description, xacro)
@@ -69,4 +69,9 @@
   <xacro:property name="propeller_color" value="Gray" />
   <xacro:property name="propeller_mesh_file" value="package://tobas_description/meshes/propeller_${propeller_direction}.dae" />
+  <!-- Wheel properties -->
+  <xacro:property name="wheel_mass" value="0.1"/>
+  <xacro:property name="wheel_radius" value="0.05"/>
+  <xacro:property name="wheel_height" value="0.025"/>
+  <xacro:property name="wheel_color" value="Black"/>
   <!-- Inertia of the main body -->
   <xacro:property name="body_inertia">
@@ -93,9 +98,12 @@
     <xacro:cylinder_inertia r="${propeller_radius}" h="${propeller_height}" mass="${mass_propeller * rotor_velocity_slowdown_sim}" />
   </xacro:property>
+  <!-- Inertia of the wheels, assuming it is a cylinder -->
+  <xacro:property name="wheel_inertia">
+    <xacro:cylinder_inertia r="${wheel_radius}" h="${wheel_height}" mass="${wheel_mass}" />
+  </xacro:property>
   <!-- Included URDF Files -->
   <!-- <xacro:include filename="$(find rotors_description)/urdf/fixed_wing_base.xacro" /> -->
   <xacro:include filename="$(find tobas_description)/urdf/fixed_wing_base.xacro" />
-  <!-- Instantiate fixed_wing_base_macro once -->
-  <!-- <xacro:fixed_wing_base_macro
+  <xacro:fixed_wing_base_macro
     robot_namespace="${namespace}"
     mass="${mass_fuselage}"
@@ -105,104 +113,42 @@
     color="${body_color}"
     use_mesh_file="${use_mesh}"
-    mesh_file="${body_mesh_file}"
-    aero_params_yaml="$(arg aero_params_yaml_file)"
-    vehicle_params_yaml="$(arg vehicle_params_yaml_file)"
-    is_input_joystick="$(arg is_input_joystick)">
-    <origin xyz="0 0 0" rpy="0 0 0" />
-    <xacro:insert_block name="body_inertia" />
-  </xacro:fixed_wing_base_macro> -->
-  <!-- Added from here -->
-  <xacro:fixed_wing_base_macro
-    robot_namespace="${namespace}"
-    mass="${mass_fuselage}"
-    length="${body_length}"
-    width="${body_width}"
-    height="${body_height}"
-    color="${body_color}"
-    use_mesh_file="${use_mesh}"
-    mesh_file="${body_mesh_file}"
-    aero_params_yaml="hoge"
-    vehicle_params_yaml="fuga"
-    is_input_joystick="piyo">
+    mesh_file="${body_mesh_file}">
     <origin xyz="0 0 0" rpy="0 0 0" />
     <xacro:insert_block name="body_inertia" />
   </xacro:fixed_wing_base_macro>
-  <!-- Added to here -->
   <!-- Instantiate the wheels -->
-	<joint name="techpod/wheel_left_joint" type="continuous">
-		<parent link="techpod/base_link"/>
-		<child link="techpod/wheel_left"/>
-		<origin xyz="0.3 0.2 -0.2" rpy="1.5707963267948966 0 0" />
-		<axis xyz="0 0 1" />
-	</joint>
-	<link name="techpod/wheel_left">
-		<inertial>
-			<mass value="1e-3" />
-			<inertia ixx="1e-3" ixy="0" ixz="0" iyy="1e-3" iyz="0" izz="1e-3" />
-		</inertial>
-		<visual>
-			<geometry>
-				<cylinder length="0.025" radius="0.05"/>
-			</geometry>
-		</visual>
-		<collision>
-			<geometry>
-				<cylinder length="0.025" radius="0.05"/>
-			</geometry>
-		</collision>
-	</link>
-	<gazebo reference="techpod/wheel_left">
-		<material>Gazebo/Black</material>
-	</gazebo>
-	<joint name="techpod/wheel_right_joint" type="continuous">
-		<parent link="techpod/base_link"/>
-		<child link="techpod/wheel_right"/>
-		<origin xyz="0.3 -0.2 -0.2" rpy="1.5707963267948966 0 0" />
-		<axis xyz="0 0 1" />
-	</joint>
-	<link name="techpod/wheel_right">
-		<inertial>
-			<mass value="1e-3" />
-			<inertia ixx="1e-3" ixy="0" ixz="0" iyy="1e-3" iyz="0" izz="1e-3" />
-		</inertial>
-		<visual>
-			<geometry>
-				<cylinder length="0.025" radius="0.05"/>
-			</geometry>
-		</visual>
-		<collision>
-			<geometry>
-				<cylinder length="0.025" radius="0.05"/>
-			</geometry>
-		</collision>
-	</link>
-	<gazebo reference="techpod/wheel_right">
-		<material>Gazebo/Black</material>
-	</gazebo>
-	<joint name="techpod/wheel_rear_joint" type="continuous">
-		<parent link="techpod/base_link"/>
-		<child link="techpod/wheel_rear"/>
-		<origin xyz="-0.3 0 -0.2" rpy="1.5707963267948966 0 0" />
-		<axis xyz="0 0 1" />
-	</joint>
-	<link name="techpod/wheel_rear">
-		<inertial>
-			<mass value="1e-3" />
-			<inertia ixx="1e-3" ixy="0" ixz="0" iyy="1e-3" iyz="0" izz="1e-3" />
-		</inertial>
-		<visual>
-			<geometry>
-				<cylinder length="0.025" radius="0.05"/>
-			</geometry>
-		</visual>
-		<collision>
-			<geometry>
-				<cylinder length="0.025" radius="0.05"/>
-			</geometry>
-		</collision>
-	</link>
-	<gazebo reference="techpod/wheel_rear">
-		<material>Gazebo/Black</material>
-	</gazebo>
+  <xacro:wheel
+    robot_namespace="${namespace}"
+    suffix="left"
+    parent="${namespace}/base_link"
+    mass="${wheel_mass}"
+    height="${wheel_height}"
+    radius="${wheel_radius}"
+    color="${wheel_color}">
+		<origin xyz="0.3 0.2 -0.2" rpy="${PI / 2} 0 0" />
+    <xacro:insert_block name="wheel_inertia" />
+  </xacro:wheel>
+  <xacro:wheel
+    robot_namespace="${namespace}"
+    suffix="right"
+    parent="${namespace}/base_link"
+    mass="${wheel_mass}"
+    height="${wheel_height}"
+    radius="${wheel_radius}"
+    color="${wheel_color}">
+		<origin xyz="0.3 -0.2 -0.2" rpy="${PI / 2} 0 0" />
+    <xacro:insert_block name="wheel_inertia" />
+  </xacro:wheel>
+  <xacro:wheel
+    robot_namespace="${namespace}"
+    suffix="rear"
+    parent="${namespace}/base_link"
+    mass="${wheel_mass}"
+    height="${wheel_height}"
+    radius="${wheel_radius}"
+    color="${wheel_color}">
+		<origin xyz="-0.3 0 -0.2" rpy="${PI / 2} 0 0" />
+    <xacro:insert_block name="wheel_inertia" />
+  </xacro:wheel>
   <!-- Instantiate the ailerons -->
   <xacro:control_surface
@@ -266,45 +212,4 @@
     <origin xyz="0 0 0" rpy="0 0 0" />   <!-- Link origin -->
     <xacro:insert_block name="elevator_inertia" />
-  </xacro:control_surface>
-  <!-- Instantiate the flaps -->
-  <xacro:control_surface
-    robot_namespace="${namespace}"
-    surface_name="flap_left"
-    parent="${namespace}/base_link"
-    mass_surface="${mass_flap}"
-    min_angle="${flap_min_angle}"
-    max_angle="${flap_max_angle}"
-    max_velocity="${flap_max_velocity}"
-    max_effort="${flap_max_effort}"
-    color="${flap_color}"
-    use_mesh_file="${use_mesh}"
-    mesh_file="${flap_left_mesh_file}"
-    surface_length="${flap_length}"
-    surface_width="${flap_width}"
-    surface_height="${flap_height}">
-    <axis xyz="0 -1 0" />   <!-- Joint axis -->
-    <origin xyz="0.101 0.382 0.1185" rpy="0 0 0" />   <!-- Joint origin -->
-    <origin xyz="0 0 0" rpy="0 0 0" />   <!-- Link origin -->
-    <xacro:insert_block name="flap_inertia" />
-  </xacro:control_surface>
-  <xacro:control_surface
-    robot_namespace="${namespace}"
-    surface_name="flap_right"
-    parent="${namespace}/base_link"
-    mass_surface="${mass_flap}"
-    min_angle="${flap_min_angle}"
-    max_angle="${flap_max_angle}"
-    max_velocity="${flap_max_velocity}"
-    max_effort="${flap_max_effort}"
-    color="${flap_color}"
-    use_mesh_file="${use_mesh}"
-    mesh_file="${flap_right_mesh_file}"
-    surface_length="${flap_length}"
-    surface_width="${flap_width}"
-    surface_height="${flap_height}">
-    <axis xyz="0 1 0" />   <!-- Joint axis -->
-    <origin xyz="0.101 -0.382 0.1185" rpy="0 0 0" />   <!-- Joint origin -->
-    <origin xyz="0 0 0" rpy="0 0 0" />   <!-- Link origin -->
-    <xacro:insert_block name="flap_inertia" />
   </xacro:control_surface>
   <!-- Instantiate the rudder -->
@@ -339,6 +244,47 @@
     use_mesh_file="${use_mesh}"
     mesh_file="${propeller_mesh_file}">
-    <origin xyz="-0.025 0 0.15" rpy="0 ${0.5 * PI} 0" />
+    <origin xyz="-0.025 0 0.15" rpy="0 ${PI / 2} 0" />
     <xacro:insert_block name="propeller_inertia" />
   </xacro:propeller>
+  <!-- Instantiate the flaps -->
+  <xacro:control_surface
+    robot_namespace="${namespace}"
+    surface_name="flap_left"
+    parent="${namespace}/base_link"
+    mass_surface="${mass_flap}"
+    min_angle="${flap_min_angle}"
+    max_angle="${flap_max_angle}"
+    max_velocity="${flap_max_velocity}"
+    max_effort="${flap_max_effort}"
+    color="${flap_color}"
+    use_mesh_file="${use_mesh}"
+    mesh_file="${flap_left_mesh_file}"
+    surface_length="${flap_length}"
+    surface_width="${flap_width}"
+    surface_height="${flap_height}">
+    <axis xyz="0 -1 0" />   <!-- Joint axis -->
+    <origin xyz="0.101 0.382 0.1185" rpy="0 0 0" />   <!-- Joint origin -->
+    <origin xyz="0 0 0" rpy="0 0 0" />   <!-- Link origin -->
+    <xacro:insert_block name="flap_inertia" />
+  </xacro:control_surface>
+  <xacro:control_surface
+    robot_namespace="${namespace}"
+    surface_name="flap_right"
+    parent="${namespace}/base_link"
+    mass_surface="${mass_flap}"
+    min_angle="${flap_min_angle}"
+    max_angle="${flap_max_angle}"
+    max_velocity="${flap_max_velocity}"
+    max_effort="${flap_max_effort}"
+    color="${flap_color}"
+    use_mesh_file="${use_mesh}"
+    mesh_file="${flap_right_mesh_file}"
+    surface_length="${flap_length}"
+    surface_width="${flap_width}"
+    surface_height="${flap_height}">
+    <axis xyz="0 1 0" />   <!-- Joint axis -->
+    <origin xyz="0.101 -0.382 0.1185" rpy="0 0 0" />   <!-- Joint origin -->
+    <origin xyz="0 0 0" rpy="0 0 0" />   <!-- Link origin -->
+    <xacro:insert_block name="flap_inertia" />
+  </xacro:control_surface>
 </robot>
