Commit message: x500v2のモデルを修正

File: tobas_description/urdf/x500v2.urdf (robot description, URDF)
Before this commit: robot x500v2, 6 links, 5 joints
Links:
- link base_link_inertia: mass 0.988937 -> 1.62

Commit message: x500v2のcollisionを単純化してシミュレーションの解像度を上げた

File: tobas_description/urdf/x500v2.urdf (robot description, URDF)
Before this commit: robot x500v2, 6 links, 5 joints
Links:
- link base_link_inertia: geometry collision box size=0.3 0.3 0.25; collision box size=0.4 0.4 0.05
