Commit message: fix: s900.xacro

File: tobas_description/urdf/s900.xacro (robot description, xacro)
@@ -3,6 +3,6 @@
   xmlns:xacro="http://ros.org/wiki/xacro">
   <!-- Included URDF Files -->
-  <xacro:include filename="$(find tobas_description)/urdf/multirotor_base.xacro"/>
-  <!-- Properties -->
+  <xacro:include filename="$(find tobas_description)/urdf/components/multirotor_base.xacro"/>
+  <!-- Properties: https://www.dji.com/jp/spreading-wings-s900 -->
   <xacro:property name="center_frame_width" value="0.3"/>
   <xacro:property name="center_frame_height" value="0.15"/>
@@ -25,4 +25,5 @@
   <xacro:property name="motor_height" value="0.027"/>
   <xacro:property name="motor_mass" value="0.158"/>
+  <xacro:property name="propeller_radius" value="0.191"/>
   <xacro:property name="propeller_height" value="0.011"/>
   <xacro:property name="propeller_mass" value="0.013"/>
@@ -32,10 +33,10 @@
       <mass value="${center_frame_mass}"/>
       <origin xyz="0 0 ${-center_frame_height/2}" rpy="0 0 0"/>
-      <xacro:box_inertia x="${center_frame_width}" y="{center_frame_width}" z="{center_frame_height}" mass="${center_frame_mass}"/>
+      <xacro:box_inertia x="${center_frame_width}" y="${center_frame_width}" z="${center_frame_height}" mass="${center_frame_mass}"/>
     </inertial>
     <visual>
       <origin xyz="0 0 0" rpy="0 0 0"/>
       <geometry>
-        <mesh filename="package://tobas_description/meshes/s900/cener_frame.stl" scale="1e-3 1e-3 1e-3"/>
+        <mesh filename="package://tobas_description/meshes/s900/center_frame.stl" scale="1e-3 1e-3 1e-3"/>
       </geometry>
       <material name="White">
@@ -46,5 +47,5 @@
       <origin xyz="0 0 ${-center_frame_height/2}" rpy="0 0 0"/>
       <geometry>
-        <box size="${center_frame_width} ${center_frame_width} {center_frame_height}"/>
+        <box size="${center_frame_width} ${center_frame_width} ${center_frame_height}"/>
       </geometry>
     </collision>
@@ -60,5 +61,5 @@
       <mass value="${battery_mass}"/>
       <origin xyz="0 0 0" rpy="0 0 0"/>
-      <xacro:box_inertia x="${battery_width}" y="{battery_width}" z="{battery_height}" mass="${battery_mass}"/>
+      <xacro:box_inertia x="${battery_x}" y="${battery_y}" z="${battery_z}" mass="${battery_mass}"/>
     </inertial>
     <visual>
@@ -73,5 +74,5 @@
       <origin xyz="0 0 0" rpy="0 0 0"/>
       <geometry>
-        <box size="${battery_width} ${battery_width} ${battery_height}"/>
+        <box size="${battery_x} ${battery_y} ${battery_z}"/>
       </geometry>
     </collision>
@@ -147,5 +148,5 @@
       <inertial>
         <mass value="${arm_mass}"/>
-        <origin xyz="${arm_length/2} 0 0" rpy="0 0 0"/>
+        <origin xyz="${arm_length/2} 0 0" rpy="0 ${pi/2} 0"/>
         <xacro:cylinder_inertia radius="${arm_radius}" length="${arm_length}" mass="${arm_mass}"/>
       </inertial>
@@ -159,5 +160,5 @@
       </visual>
       <collision>
-        <origin xyz="${arm_length/2} 0 0" rpy="0 0 0"/>
+        <origin xyz="${arm_length/2} 0 0" rpy="0 ${pi/2} 0"/>
         <geometry>
           <cylinder radius="${arm_radius}" length="${arm_length}"/>
@@ -168,5 +169,5 @@
     <joint name="motor_${index}_joint" type="fixed">
       <origin xyz="0.251 0 0.005" rpy="0 0 0"/>
-      <parent link="arm_${index}_joint"/>
+      <parent link="arm_${index}"/>
       <child link="motor_${index}"/>
     </joint>
@@ -196,8 +197,8 @@
       <origin xyz="0 0 ${motor_height}" rpy="0 0 0"/>
       <axis xyz="0 0 1"/>
-      <parent link="base_link"/>
-      <child link="propeller_{index}"/>
-    </joint>
-    <link name="propeller_{index}">
+      <parent link="motor_${index}"/>
+      <child link="propeller_${index}"/>
+    </joint>
+    <link name="propeller_${index}">
       <inertial>
         <mass value="${propeller_mass}"/>
@@ -222,7 +223,8 @@
   </xacro:macro>
   <xacro:propulsion_system index="0" yaw_deg="30" origin_x="${arm_offset*cos30}" origin_y="${arm_offset*sin30}" direction="ccw"/>
-  <xacro:propulsion_system index="0" yaw_deg="90" origin_x="0" origin_y="${arm_offset}" direction="cw"/>
-  <xacro:propulsion_system index="0" yaw_deg="150" origin_x="${-arm_offset*cos30}" origin_y="${arm_offset*sin30}" direction="ccw"/>
-  <xacro:propulsion_system index="0" yaw_deg="210" origin_x="${-arm_offset*cos30}" origin_y="${-arm_offset*sin30}" direction="cw"/>
-  <xacro:propulsion_system index="0" yaw_deg="270" origin_x="0" origin_y="${-arm_offset}" direction="ccw"/>
-  <xacro:propulsion_system index="0" yaw_deg="330" origin_x="${arm_offset*cos30}" origin_y="${-arm_offset*sin30}" direction="cw"/>
+  <xacro:propulsion_system index="1" yaw_deg="90" origin_x="0" origin_y="${arm_offset}" direction="cw"/>
+  <xacro:propulsion_system index="2" yaw_deg="150" origin_x="${-arm_offset*cos30}" origin_y="${arm_offset*sin30}" direction="ccw"/>
+  <xacro:propulsion_system index="3" yaw_deg="210" origin_x="${-arm_offset*cos30}" origin_y="${-arm_offset*sin30}" direction="cw"/>
+  <xacro:propulsion_system index="4" yaw_deg="270" origin_x="0" origin_y="${-arm_offset}" direction="ccw"/>
+  <xacro:propulsion_system index="5" yaw_deg="330" origin_x="${arm_offset*cos30}" origin_y="${-arm_offset*sin30}" direction="cw"/>
+</robot>

Commit message: .

File: tobas_description/urdf/s900.xacro (robot description, xacro)
@@ -13,7 +13,7 @@
   <xacro:property name="battery_mass" value="1.424"/>
   <xacro:property name="landing_gear_upper_radius" value="0.0125"/>
-  <xacro:property name="landing_gear_upper_length" value="0.358"/>
+  <xacro:property name="landing_gear_upper_length" value="0.35"/>
   <xacro:property name="landing_gear_upper_mass" value="0.06"/>
-  <xacro:property name="landing_gear_lower_radius" value="0.008"/>
+  <xacro:property name="landing_gear_lower_radius" value="0.009"/>
   <xacro:property name="landing_gear_lower_length" value="0.457"/>
   <xacro:property name="landing_gear_lower_mass" value="0.06"/>
@@ -30,4 +30,13 @@
   <!-- Center Frame -->
   <link name="base_link">
+    <visual>
+      <origin xyz="0 0 0" rpy="0 0 0"/>
+      <geometry>
+        <mesh filename="package://tobas_description/meshes/s900/center_frame.stl" scale="1e-3 1e-3 1e-3"/>
+      </geometry>
+      <material name="White">
+        <color rgba="1 1 1 1"/>
+      </material>
+    </visual>
     <inertial>
       <mass value="${center_frame_mass}"/>
@@ -35,13 +44,4 @@
       <xacro:box_inertia x="${center_frame_width}" y="${center_frame_width}" z="${center_frame_height}" mass="${center_frame_mass}"/>
     </inertial>
-    <visual>
-      <origin xyz="0 0 0" rpy="0 0 0"/>
-      <geometry>
-        <mesh filename="package://tobas_description/meshes/s900/center_frame.stl" scale="1e-3 1e-3 1e-3"/>
-      </geometry>
-      <material name="White">
-        <color rgba="1 1 1 1"/>
-      </material>
-    </visual>
     <collision>
       <origin xyz="0 0 ${-center_frame_height/2}" rpy="0 0 0"/>
@@ -58,4 +58,12 @@
   </joint>
   <link name="battery">
+    <visual>
+      <geometry>
+        <mesh filename="package://tobas_description/meshes/s900/battery.stl" scale="1e-3 1e-3 1e-3"/>
+      </geometry>
+      <material name="Black">
+        <color rgba="0 0 0 1"/>
+      </material>
+    </visual>
     <inertial>
       <mass value="${battery_mass}"/>
@@ -63,12 +71,4 @@
       <xacro:box_inertia x="${battery_x}" y="${battery_y}" z="${battery_z}" mass="${battery_mass}"/>
     </inertial>
-    <visual>
-      <geometry>
-        <mesh filename="package://tobas_description/meshes/s900/battery.stl" scale="1e-3 1e-3 1e-3"/>
-      </geometry>
-      <material name="Black">
-        <color rgba="0 0 0 1"/>
-      </material>
-    </visual>
     <collision>
       <origin xyz="0 0 0" rpy="0 0 0"/>
@@ -87,19 +87,19 @@
     </joint>
     <link name="landing_gear_${suffix}_upper">
+      <visual>
+        <geometry>
+          <mesh filename="package://tobas_description/meshes/s900/landing_gear_upper.stl" scale="1e-3 1e-3 1e-3"/>
+        </geometry>
+        <material name="Black">
+          <color rgba="0 0 0 1"/>
+        </material>
+      </visual>
       <inertial>
         <mass value="${landing_gear_upper_mass}"/>
-        <origin xyz="0 0 ${landing_gear_upper_length/2}" rpy="0 0 0"/>
+        <origin xyz="0 0 ${-landing_gear_upper_length/2}" rpy="0 0 0"/>
         <xacro:cylinder_inertia radius="${landing_gear_upper_radius}" length="${landing_gear_upper_length}" mass="${landing_gear_upper_mass}"/>
       </inertial>
-      <visual>
-        <geometry>
-          <mesh filename="package://tobas_description/meshes/s900/landing_gear_upper.stl" scale="1e-3 1e-3 1e-3"/>
-        </geometry>
-        <material name="Black">
-          <color rgba="0 0 0 1"/>
-        </material>
-      </visual>
-      <collision>
-        <origin xyz="0 0 ${landing_gear_upper_length/2}" rpy="0 0 0"/>
+      <collision>
+        <origin xyz="0 0 ${-landing_gear_upper_length/2}" rpy="0 0 0"/>
         <geometry>
           <cylinder radius="${landing_gear_upper_radius}" length="${landing_gear_upper_length}"/>
@@ -114,4 +114,12 @@
     </joint>
     <link name="landing_gear_${suffix}_lower">
+      <visual>
+        <geometry>
+          <mesh filename="package://tobas_description/meshes/s900/landing_gear_lower.stl" scale="1e-3 1e-3 1e-3"/>
+        </geometry>
+        <material name="Black">
+          <color rgba="0 0 0 1"/>
+        </material>
+      </visual>
       <inertial>
         <mass value="${landing_gear_lower_mass}"/>
@@ -119,12 +127,4 @@
         <xacro:cylinder_inertia radius="${landing_gear_lower_radius}" length="${landing_gear_lower_length}" mass="${landing_gear_lower_mass}"/>
       </inertial>
-      <visual>
-        <geometry>
-          <mesh filename="package://tobas_description/meshes/s900/landing_gear_lower.stl" scale="1e-3 1e-3 1e-3"/>
-        </geometry>
-        <material name="Black">
-          <color rgba="0 0 0 1"/>
-        </material>
-      </visual>
       <collision>
         <origin xyz="0 0 0" rpy="0 ${pi/2} 0"/>
@@ -146,4 +146,12 @@
     </joint>
     <link name="arm_${index}">
+      <visual>
+        <geometry>
+          <mesh filename="package://tobas_description/meshes/s900/arm.stl" scale="1e-3 1e-3 1e-3"/>
+        </geometry>
+        <material name="Black">
+          <color rgba="0 0 0 1"/>
+        </material>
+      </visual>
       <inertial>
         <mass value="${arm_mass}"/>
@@ -151,12 +159,4 @@
         <xacro:cylinder_inertia radius="${arm_radius}" length="${arm_length}" mass="${arm_mass}"/>
       </inertial>
-      <visual>
-        <geometry>
-          <mesh filename="package://tobas_description/meshes/s900/arm.stl" scale="1e-3 1e-3 1e-3"/>
-        </geometry>
-        <material name="Black">
-          <color rgba="0 0 0 1"/>
-        </material>
-      </visual>
       <collision>
         <origin xyz="${arm_length/2} 0 0" rpy="0 ${pi/2} 0"/>
@@ -173,4 +173,12 @@
     </joint>
     <link name="motor_${index}">
+      <visual>
+        <geometry>
+          <mesh filename="package://tobas_description/meshes/s900/motor.stl" scale="1e-3 1e-3 1e-3"/>
+        </geometry>
+        <material name="Black">
+          <color rgba="0 0 0 1"/>
+        </material>
+      </visual>
       <inertial>
         <mass value="${motor_mass}"/>
@@ -178,12 +186,4 @@
         <xacro:cylinder_inertia radius="${motor_radius}" length="${motor_height}" mass="${motor_mass}"/>
       </inertial>
-      <visual>
-        <geometry>
-          <mesh filename="package://tobas_description/meshes/s900/motor.stl" scale="1e-3 1e-3 1e-3"/>
-        </geometry>
-        <material name="Black">
-          <color rgba="0 0 0 1"/>
-        </material>
-      </visual>
       <collision>
         <origin xyz="0 0 ${motor_height/2}" rpy="0 0 0"/>
@@ -201,4 +201,12 @@
     </joint>
     <link name="propeller_${index}">
+      <visual>
+        <geometry>
+          <mesh filename="package://tobas_description/meshes/s900/propeller_${direction}.stl" scale="1e-3 1e-3 1e-3"/>
+        </geometry>
+        <material name="Black">
+          <color rgba="0.0 0.0 0.0 1.0"/>
+        </material>
+      </visual>
       <inertial>
         <mass value="${propeller_mass}"/>
@@ -206,12 +214,4 @@
         <xacro:cylinder_inertia radius="${propeller_radius}" length="${propeller_height}" mass="${propeller_mass}"/>
       </inertial>
-      <visual>
-        <geometry>
-          <mesh filename="package://tobas_description/meshes/s900/propeller_${direction}.stl" scale="1e-3 1e-3 1e-3"/>
-        </geometry>
-        <material name="Black">
-          <color rgba="0.0 0.0 0.0 1.0"/>
-        </material>
-      </visual>
       <collision>
         <origin xyz="0 0 ${propeller_height/2}" rpy="0 0 0"/>

Commit message: .

File: tobas_description/urdf/s900.xacro (robot description, xacro)
@@ -28,6 +28,13 @@
   <xacro:property name="propeller_height" value="0.011"/>
   <xacro:property name="propeller_mass" value="0.013"/>
+  <!-- Base Link -->
+  <link name="base_link"/>
   <!-- Center Frame -->
-  <link name="base_link">
+  <joint name="center_frame_joint" type="fixed">
+    <origin xyz="0 0 0" rpy="0 0 0"/>
+    <parent link="base_link"/>
+    <child link="center_frame"/>
+  </joint>
+  <link name="center_frame">
     <visual>
       <origin xyz="0 0 0" rpy="0 0 0"/>

Commit message: .

File: tobas_description/urdf/s900.xacro (robot description, xacro)
@@ -140,5 +140,5 @@
     <!-- Arm -->
     <joint name="arm_${index}_joint" type="fixed">
-      <origin xyz="${origin_x} ${origin_y} -0.015" rpy="${-3.238*deg2rad} 0 ${yaw_deg*deg2rad}"/>
+      <origin xyz="${origin_x} ${origin_y} -0.015" rpy="0 ${-3.238*deg2rad} ${yaw_deg*deg2rad}"/>
       <parent link="base_link"/>
       <child link="arm_${index}"/>
