Commit message: f550_non_planar -> f550_np

File: tobas_description/urdf/f550_np.xacro (robot description, xacro)
@@ -1,8 +1,8 @@
 <?xml version="1.0"?>
-<robot name="f550_non_planar"
+<robot name="f550_np"
   xmlns:xacro="http://ros.org/wiki/xacro">
   <!-- Included URDF Files -->
   <xacro:include filename="$(find tobas_description)/urdf/components/multirotor_base.xacro"/>
-  <!-- Properties: https://www.dji.com/jp/spreading-wings-f550_non_planar -->
+  <!-- Properties -->
   <xacro:property name="frame_radius" value="0.294"/>
   <xacro:property name="frame_height" value="0.056"/>
@@ -26,5 +26,5 @@
       <origin xyz="0 0 0" rpy="0 0 0"/>
       <geometry>
-        <mesh filename="package://tobas_description/meshes/f550_non_planar/frame.stl" scale="1e-3 1e-3 1e-3"/>
+        <mesh filename="package://tobas_description/meshes/f550_np/frame.stl" scale="1e-3 1e-3 1e-3"/>
       </geometry>
       <xacro:insert_block name="black"/>
@@ -48,5 +48,5 @@
       <visual>
         <geometry>
-          <mesh filename="package://tobas_description/meshes/f550_non_planar/phantom3_0945_${direction}.stl" scale="1e-3 1e-3 1e-3"/>
+          <mesh filename="package://tobas_description/meshes/f550_np/phantom3_0945_${direction}.stl" scale="1e-3 1e-3 1e-3"/>
         </geometry>
         <xacro:insert_block name="white"/>

Commit message: edit: f550_np.xacro

File: tobas_description/urdf/f550_np.xacro (robot description, xacro)
@@ -7,5 +7,9 @@
   <xacro:property name="frame_radius" value="0.294"/>
   <xacro:property name="frame_height" value="0.056"/>
-  <xacro:property name="frame_mass" value="1.615"/>
+  <xacro:property name="frame_mass" value="1.423"/>
+  <xacro:property name="battery_x" value="0.155"/>
+  <xacro:property name="battery_y" value="0.048"/>
+  <xacro:property name="battery_z" value="0.032"/>
+  <xacro:property name="battery_mass" value="0.496"/>
   <xacro:property name="propeller_diameter" value="${9*inch2meter}"/>
   <xacro:property name="propeller_radius" value="${propeller_diameter/2}"/>
@@ -32,8 +36,34 @@
     <inertial>
       <mass value="${frame_mass}"/>
-      <origin xyz="5.5e-4 1.04e-3 9.895e-3" rpy="0 0 0"/>
-      <inertia ixx="3.720e-2" ixy="4.6919e-8" ixz="-6.275258e-6" iyy="3.725e-2" iyz="-5.9311674e-5" izz="7.102e-2"/>
+      <origin xyz="0.624e-3 1.181e-3 14.463e-3" rpy="0 0 0"/>
+      <inertia ixx="3.692e-2" ixy="1.71388e-7" ixz="-2.219266e-6" iyy="3.681e-2" iyz="-5.1639988e-5" izz="7.082e-2"/>
     </inertial>
     <xacro:hexagonal_prism_collision side="${frame_radius}" height="${frame_height}" x0="0" y0="0" z0="${-frame_height/2}"/>
+  </link>
+  <!-- Battery -->
+  <joint name="battery_joint" type="fixed">
+    <origin xyz="0 0 -0.021" rpy="0 0 0"/>
+    <parent link="base_link"/>
+    <child link="battery"/>
+  </joint>
+  <link name="battery">
+    <visual>
+      <origin xyz="0 0 0" rpy="0 0 0"/>
+      <geometry>
+        <box size="${battery_x} ${battery_y} ${battery_z}"/>
+      </geometry>
+      <xacro:insert_block name="black"/>
+    </visual>
+    <inertial>
+      <mass value="${battery_mass}"/>
+      <origin xyz="0 0 0" rpy="0 0 0"/>
+      <xacro:box_inertia x="${battery_x}" y="${battery_y}" z="${battery_z}" mass="${battery_mass}"/>
+    </inertial>
+    <collision>
+      <origin xyz="0 0 0" rpy="0 0 0"/>
+      <geometry>
+        <box size="${battery_x} ${battery_y} ${battery_z}"/>
+      </geometry>
+    </collision>
   </link>
   <!-- Propellers -->
