Commit message: add: matrice300

File: tobas_description/urdf/matrice300.urdf (robot description, URDF)
Before this commit: robot matrice300, 11 links, 10 joints
Links:
- removed link motor_0_1
- removed link motor_1_2
- removed link propeller_0_4
- removed link propeller_0_5
- removed link propeller_0_5_6
- added link motor_2, mass 0.3; collision cylinder length=0.12 radius=0.04; visual mesh filename=package://tobas_description/meshes/matrice300/arm_tip_rear.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 scale=0.001 0.001 0.001
- added link motor_3, mass 0.3; collision cylinder length=0.12 radius=0.04; visual mesh filename=package://tobas_description/meshes/matrice300/arm_tip_rear.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 scale=0.001 0.001 0.001
- added link propeller_1, mass 0.05; collision cylinder length=0.04 radius=0.274; visual mesh filename=package://tobas_description/meshes/matrice300/propeller_cw.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 scale=0.001 0.001 0.001
- added link propeller_2, mass 0.05; collision cylinder length=0.04 radius=0.274; visual mesh filename=package://tobas_description/meshes/matrice300/propeller_ccw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 scale=0.001 0.001 0.001
- added link propeller_3, mass 0.05; collision cylinder length=0.04 radius=0.274; visual mesh filename=package://tobas_description/meshes/matrice300/propeller_cw.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 scale=0.001 0.001 0.001
- link battery: geometry collision box size=0.137 0.1 0.178; visual mesh filename=package://tobas_description/meshes/matrice300/battery.stl scale=0.001 0.001 0.001
- link frame: geometry collision box size=0.26 0.15 0.16; collision box size=0.4 0.42 0.25
- link motor_0: geometry collision cylinder length=0.14 radius=0.04; visual mesh filename=package://tobas_description/meshes/matrice300/arm_tip_front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 scale=0.001 0.001 0.001
- link motor_1: geometry collision cylinder length=0.14 radius=0.04; visual mesh filename=package://tobas_description/meshes/matrice300/arm_tip_front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 scale=0.001 0.001 0.001
- link propeller_0: geometry collision cylinder length=0.04 radius=0.274; visual mesh filename=package://tobas_description/meshes/matrice300/propeller_ccw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 scale=0.001 0.001 0.001
Joints:
- removed joint battery_to_frame_joint
- removed joint frame_to_root_joint
- removed joint motor_0_to_frame_joint
- removed joint motor_0_to_frame_joint_1
- removed joint motor_1_to_frame_joint
- removed joint motor_1_to_frame_joint_2
- removed joint propeller_0_to_motor_0_joint
- removed joint propeller_0_to_motor_0_joint_4
- removed joint propeller_0_to_motor_0_joint_5
- removed joint propeller_0_to_motor_0_joint_5_6
- added joint battery_joint: type fixed, parent frame, child battery, origin xyz=0 0 0.002 rpy=1.57 0 1.57, axis 0 0 0
- added joint frame_joint: type fixed, parent root, child frame, origin xyz=0 0 0 rpy=0 -0 0, axis 0 0 0
- added joint motor_0_joint: type fixed, parent frame, child motor_0, origin xyz=0.285 -0.367 0.002 rpy=1.57 0 -1.06, axis 0 0 0
- added joint motor_1_joint: type fixed, parent frame, child motor_1, origin xyz=0.285 0.367 0.002 rpy=1.57 0 1.1, axis 0 0 0
- added joint motor_2_joint: type fixed, parent frame, child motor_2, origin xyz=-0.306 0.319 0.002 rpy=1.57 0 2.2, axis 0 0 0
- added joint motor_3_joint: type fixed, parent frame, child motor_3, origin xyz=-0.306 -0.319 0.002 rpy=1.57 0 -2.2, axis 0 0 0
- added joint propeller_0_joint: type continuous, parent motor_0, child propeller_0, origin xyz=0.037 -0.061 0 rpy=-0.05 1.57 -3.14, axis 0 -1 0
- added joint propeller_1_joint: type continuous, parent motor_1, child propeller_1, origin xyz=0.037 -0.061 0 rpy=-0.05 1.57 -3.14, axis 0 -1 0
- added joint propeller_2_joint: type continuous, parent motor_2, child propeller_2, origin xyz=0.037 -0.061 0 rpy=-0.05 1.57 -3.14, axis 0 -1 0
- added joint propeller_3_joint: type continuous, parent motor_3, child propeller_3, origin xyz=0.037 -0.061 0 rpy=-0.05 1.57 -3.14, axis 0 -1 0
