Commit message: edit: f550_np_rmx52.xacro

File: tobas_description/urdf/f550_np_rmx52.xacro (robot description, xacro)
@@ -5,5 +5,5 @@
   <xacro:include filename="$(find tobas_description)/urdf/components/multirotor_base.xacro"/>
   <!-- Properties -->
-  <xacro:property name="frame_mass" value="1.619"/>
+  <xacro:property name="frame_mass" value="1.579"/>
   <xacro:property name="battery_x" value="0.155"/>
   <xacro:property name="battery_y" value="0.048"/>
@@ -34,6 +34,6 @@
     <inertial>
       <mass value="${frame_mass}"/>
-      <origin xyz="0.549e-3 1.038e-3 2.206e-3" rpy="0 0 0"/>
-      <inertia ixx="4.255e-2" ixy="1.7385e-8" ixz="-1.3101809e-5" iyy="4.217e-2" iyz="-7.2223721e-5" izz="7.701e-2"/>
+      <origin xyz="0.562e-3 1.064e-3 3.537e-3" rpy="0 0 0"/>
+      <inertia ixx="4.242e-2" ixy="5.5253e-8" ixz="-1.192013e-5" iyy="4.204e-2" iyz="-6.9988639e-5" izz="7.699e-2"/>
     </inertial>
     <collision>

Commit message: edit: f550_np_rmx52

File: tobas_description/urdf/f550_np_rmx52.xacro (robot description, xacro)
@@ -6,14 +6,14 @@
   <xacro:include filename="$(find tobas_description)/urdf/components/rmx52/rmx52.xacro"/>
   <!-- Properties -->
-  <xacro:property name="frame_mass" value="1.579"/>
+  <xacro:property name="frame_mass" value="1.665"/>
   <xacro:property name="battery_x" value="0.155"/>
   <xacro:property name="battery_y" value="0.048"/>
-  <xacro:property name="battery_z" value="0.032"/>
-  <xacro:property name="battery_mass" value="0.496"/>
+  <xacro:property name="battery_z" value="0.048"/>
+  <xacro:property name="battery_mass" value="0.725"/>
   <xacro:property name="propeller_diameter" value="${9*inch2meter}"/>
   <xacro:property name="propeller_radius" value="${propeller_diameter/2}"/>
   <xacro:property name="propeller_height" value="0.01"/>
   <xacro:property name="propeller_mass" value="0.011"/>
-  <xacro:property name="propeller_origin_z" value="0.060597"/>
+  <xacro:property name="propeller_origin_z" value="0.048597"/>
   <xacro:property name="rotor_tilt" value="${30*deg2rad}"/>
   <!-- Base Link -->
@@ -35,6 +35,6 @@
     <inertial>
       <mass value="${frame_mass}"/>
-      <origin xyz="0.562e-3 1.064e-3 3.537e-3" rpy="0 0 0"/>
-      <inertia ixx="4.242e-2" ixy="5.5253e-8" ixz="-1.192013e-5" iyy="4.204e-2" iyz="-6.9988639e-5" izz="7.699e-2"/>
+      <origin xyz="0.486e-3 1.081e-3 -4.42e-3" rpy="0 0 0"/>
+      <inertia ixx="3.962e-2" ixy="-2.133e-6" ixz="-2.014-5" iyy="3.769e-2" iyz="-7.798e-5" izz="7.291e-2"/>
     </inertial>
     <collision>
@@ -47,5 +47,5 @@
   <!-- Battery -->
   <joint name="battery_joint" type="fixed">
-    <origin xyz="0 0 -0.021" rpy="0 0 0"/>
+    <origin xyz="0 0 -0.024" rpy="0 0 0"/>
     <parent link="base_link"/>
     <child link="battery"/>
@@ -71,4 +71,36 @@
     </collision>
   </link>
+  <!-- Landing Gears -->
+  <xacro:macro name="landing_gear" params="direction reverse suffix">
+    <joint name="landing_gear_${suffix}_lower_joint" type="fixed">
+      <origin xyz="0 ${direction*0.0825} -0.063" rpy="0 0 ${reverse*pi}"/>
+      <parent link="base_link"/>
+      <child link="landing_gear_${suffix}"/>
+      <axis xyz="1 0 0"/>
+      <limit velocity="1" effort="1" lower="0" upper="${75*rad2deg}"/>  <!-- TODO -->
+      <dynamics damping="0" friction="0.01"/>
+    </joint>
+    <link name="landing_gear_${suffix}">
+      <visual>
+        <geometry>
+          <mesh filename="package://tobas_description/meshes/f550_np_rmx52/landing_gear.stl" scale="1e-3 1e-3 1e-3"/>
+        </geometry>
+        <xacro:insert_block name="black"/>
+      </visual>
+      <inertial>
+        <mass value="0.072}"/>
+        <origin xyz="-0.046 0.211 0" rpy="0 0 0"/>
+        <inertia ixx="7.171e-4" ixy="1.208e-4" ixz="-3.102e-9" iyy="2.613e-4" iyz="1.235e-8" izz="5.198e-4"/>
+      </inertial>
+      <collision>
+        <origin xyz="0 0 0" rpy="0 0 0"/>
+        <geometry>
+          <mesh filename="package://tobas_description/meshes/f550_np_rmx52/landing_gear.stl" scale="1e-3 1e-3 1e-3"/>
+        </geometry>
+      </collision>
+    </link>
+  </xacro:macro>
+  <xacro:landing_gear direction="1" reverse="0" suffix="left"/>
+  <xacro:landing_gear direction="-1" reverse="1" suffix="right"/>
   <!-- Propellers -->
   <xacro:macro name="propeller" params="index direction *origin">

Commit message: .

File: tobas_description/urdf/f550_np_rmx52.xacro (robot description, xacro)
@@ -15,5 +15,5 @@
   <xacro:property name="propeller_height" value="0.01"/>
   <xacro:property name="propeller_mass" value="0.011"/>
-  <xacro:property name="propeller_origin_z" value="0.048597"/>
+  <xacro:property name="propeller_origin_z" value="0.050597"/>
   <xacro:property name="rotor_tilt" value="${30*deg2rad}"/>
   <!-- Base Link -->
@@ -151,5 +151,5 @@
   <!-- Robot Arm -->
   <joint name="rmx52_joint" type="fixed">
-    <origin xyz="0.004 0 -0.0445" rpy="${pi} 0 0"/>
+    <origin xyz="0.004 0 -0.0545" rpy="${pi} 0 0"/>
     <parent link="base_link"/>
     <child link="rmx52/link1"/>

Commit message: edit: f550_np_rmx52.xacro

File: tobas_description/urdf/f550_np_rmx52.xacro (robot description, xacro)
@@ -9,5 +9,5 @@
   <xacro:property name="battery_x" value="0.155"/>
   <xacro:property name="battery_y" value="0.048"/>
-  <xacro:property name="battery_z" value="0.048"/>
+  <xacro:property name="battery_z" value="0.042"/>
   <xacro:property name="battery_mass" value="0.725"/>
   <xacro:property name="propeller_diameter" value="${9*inch2meter}"/>
@@ -36,5 +36,5 @@
       <mass value="${frame_mass}"/>
       <origin xyz="0.486e-3 1.081e-3 -4.42e-3" rpy="0 0 0"/>
-      <inertia ixx="3.962e-2" ixy="-2.133e-6" ixz="-2.014-5" iyy="3.769e-2" iyz="-7.798e-5" izz="7.291e-2"/>
+      <inertia ixx="3.962e-2" ixy="-2.133e-6" ixz="-2.014e-5" iyy="3.769e-2" iyz="-7.798e-5" izz="7.291e-2"/>
     </inertial>
     <collision>
@@ -47,5 +47,5 @@
   <!-- Battery -->
   <joint name="battery_joint" type="fixed">
-    <origin xyz="0 0 -0.024" rpy="0 0 0"/>
+    <origin xyz="0 0 -0.023" rpy="0 0 0"/>
     <parent link="base_link"/>
     <child link="battery"/>
@@ -73,13 +73,13 @@
   <!-- Landing Gears -->
   <xacro:macro name="landing_gear" params="direction reverse suffix">
-    <joint name="landing_gear_${suffix}_lower_joint" type="fixed">
+    <joint name="lg_${suffix}_joint" type="revolute">
       <origin xyz="0 ${direction*0.0825} -0.063" rpy="0 0 ${reverse*pi}"/>
       <parent link="base_link"/>
-      <child link="landing_gear_${suffix}"/>
+      <child link="lg_${suffix}"/>
       <axis xyz="1 0 0"/>
-      <limit velocity="1" effort="1" lower="0" upper="${75*rad2deg}"/>  <!-- TODO -->
+      <limit velocity="${pi/2}" effort="1" lower="0" upper="${75*deg2rad}"/>  <!-- TODO -->
       <dynamics damping="0" friction="0.01"/>
     </joint>
-    <link name="landing_gear_${suffix}">
+    <link name="lg_${suffix}">
       <visual>
         <geometry>
@@ -89,5 +89,5 @@
       </visual>
       <inertial>
-        <mass value="0.072}"/>
+        <mass value="0.072"/>
         <origin xyz="-0.046 0.211 0" rpy="0 0 0"/>
         <inertia ixx="7.171e-4" ixy="1.208e-4" ixz="-3.102e-9" iyy="2.613e-4" iyz="1.235e-8" izz="5.198e-4"/>
@@ -100,4 +100,5 @@
       </collision>
     </link>
+    <xacro:simple_transmission_position jnt_name="lg_${suffix}_joint"/>
   </xacro:macro>
   <xacro:landing_gear direction="1" reverse="0" suffix="left"/>

Commit message: edit: f550_np_rmx52.xacro

File: tobas_description/urdf/f550_np_rmx52.xacro (robot description, xacro)
@@ -6,5 +6,5 @@
   <xacro:include filename="$(find tobas_description)/urdf/components/rmx52/rmx52.xacro"/>
   <!-- Properties -->
-  <xacro:property name="frame_mass" value="1.665"/>
+  <xacro:property name="frame_mass" value="1.357"/>
   <xacro:property name="battery_x" value="0.155"/>
   <xacro:property name="battery_y" value="0.048"/>
@@ -15,5 +15,5 @@
   <xacro:property name="propeller_height" value="0.01"/>
   <xacro:property name="propeller_mass" value="0.011"/>
-  <xacro:property name="propeller_origin_z" value="0.050597"/>
+  <xacro:property name="propeller_origin_z" value="0.030816"/>
   <xacro:property name="rotor_tilt" value="${30*deg2rad}"/>
   <!-- Base Link -->
@@ -35,6 +35,6 @@
     <inertial>
       <mass value="${frame_mass}"/>
-      <origin xyz="0.486e-3 1.081e-3 -4.42e-3" rpy="0 0 0"/>
-      <inertia ixx="3.962e-2" ixy="-2.133e-6" ixz="-2.014e-5" iyy="3.769e-2" iyz="-7.798e-5" izz="7.291e-2"/>
+      <origin xyz="0.596e-3 1.327e-3 -0.0135" rpy="0 0 0"/>
+      <inertia ixx="2.720e-2" ixy="-1.897e-6" ixz="-2.766e-5" iyy="2.527e-2" iyz="-9.461e-5" izz="4.993e-2"/>
     </inertial>
     <collision>
@@ -133,20 +133,20 @@
   </xacro:macro>
   <xacro:propeller index="0" direction="ccw">
-    <origin xyz="0.242082 0.130702 ${propeller_origin_z}" rpy="${rotor_tilt} 0 ${30*deg2rad}"/>
+    <origin xyz="0.24372 0.127865 ${propeller_origin_z}" rpy="${rotor_tilt} 0 ${30*deg2rad}"/>
   </xacro:propeller>
   <xacro:propeller index="1" direction="cw">
-    <origin xyz="-0.007851 0.27500 ${propeller_origin_z}" rpy="${-rotor_tilt} 0 ${90*deg2rad}"/>
+    <origin xyz="-0.011216 0.27500 ${propeller_origin_z}" rpy="${-rotor_tilt} 0 ${90*deg2rad}"/>
   </xacro:propeller>
   <xacro:propeller index="2" direction="ccw">
-    <origin xyz="-0.234232 0.144298 ${propeller_origin_z}" rpy="${rotor_tilt} 0 ${150*deg2rad}"/>
+    <origin xyz="-0.232594 0.147135 ${propeller_origin_z}" rpy="${rotor_tilt} 0 ${150*deg2rad}"/>
   </xacro:propeller>
   <xacro:propeller index="3" direction="cw">
-    <origin xyz="-0.234232 -0.144645 ${propeller_origin_z}" rpy="${-rotor_tilt} 0 ${210*deg2rad}"/>
+    <origin xyz="-0.232594 -0.147135 ${propeller_origin_z}" rpy="${-rotor_tilt} 0 ${210*deg2rad}"/>
   </xacro:propeller>
   <xacro:propeller index="4" direction="ccw">
-    <origin xyz="-0.007851 -0.27500 ${propeller_origin_z}" rpy="${rotor_tilt} 0 ${270*deg2rad}"/>
+    <origin xyz="-0.011216 -0.27500 ${propeller_origin_z}" rpy="${rotor_tilt} 0 ${270*deg2rad}"/>
   </xacro:propeller>
   <xacro:propeller index="5" direction="cw">
-    <origin xyz="0.242082 -0.130355 ${propeller_origin_z}" rpy="${-rotor_tilt} 0 ${330*deg2rad}"/>
+    <origin xyz="0.24372 -0.127865 ${propeller_origin_z}" rpy="${-rotor_tilt} 0 ${330*deg2rad}"/>
   </xacro:propeller>
   <!-- Robot Arm -->

Commit message: edit: f550_np_rmx52.xacro

File: tobas_description/urdf/f550_np_rmx52.xacro (robot description, xacro)
@@ -78,5 +78,5 @@
       <child link="lg_${suffix}"/>
       <axis xyz="1 0 0"/>
-      <limit velocity="${pi/2}" effort="1" lower="0" upper="${75*deg2rad}"/>  <!-- TODO -->
+      <limit velocity="${75*deg2rad/6}" effort="1" lower="0" upper="${75*deg2rad}"/>
       <dynamics damping="0" friction="0.01"/>
     </joint>
