Commit message: メッシュ類をtobas_descriptionに移植

File: tobas_description/urdf/ardrone.xacro (robot description, xacro)
@@ -6,5 +6,5 @@
   <xacro:property name="rotor_velocity_slowdown_sim" value="10" />
   <xacro:property name="use_mesh_file" value="true" />
-  <xacro:property name="mesh_file" value="package://rotors_description/meshes/ardrone.dae" />
+  <xacro:property name="mesh_file" value="package://tobas_description/meshes/ardrone.dae" />
   <xacro:property name="mass" value="1.5" /> <!-- [kg] -->
   <xacro:property name="body_width" value="0.3" /> <!-- [m] -->

File: tobas_description/urdf/firefly.xacro (robot description, xacro)
@@ -22,5 +22,5 @@
   <xacro:property name="rotor_velocity_slowdown_sim" value="10" />
   <xacro:property name="use_mesh_file" value="true" />
-  <xacro:property name="mesh_file" value="package://rotors_description/meshes/firefly.dae" />
+  <xacro:property name="mesh_file" value="package://tobas_description/meshes/firefly.dae" />
   <xacro:property name="mass" value="1.5" /> <!-- [kg] -->
   <xacro:property name="body_width" value="0.1" /> <!-- [m] -->

File: tobas_description/urdf/harrier/multirotor_base_harrier.xacro (robot description, xacro)
@@ -22,9 +22,9 @@
   <xacro:property name="use_embedded_controller" value="$(arg use_embedded_controller)"/> -->
   <!-- <xacro:if value="$(arg load_manipulator)"> -->
-	   <xacro:include filename="$(find aerial_manipulation)/urdf/j2s7s300.xacro"/>
+	   <xacro:include filename="$(find tobas_description)/urdf/harrier/j2s7s300.xacro"/>
   	   <xacro:j2s7s300 base_parent="${namespace}/base_link" ns="${namespace}" is_inverted="1"/>
   <!-- </xacro:if> -->
   <!-- <xacro:if value="$(arg with_landing_gear)"> -->
-	  <xacro:include filename="$(find aerial_manipulation)/urdf/landing_gear.xacro"/>
+	  <xacro:include filename="$(find tobas_description)/urdf/harrier/landing_gear.xacro"/>
   <!-- </xacro:if> -->
   <!-- <xacro:if value="$(arg use_embedded_controller)">
@@ -121,5 +121,5 @@
           </xacro:if>
           <xacro:unless value="${use_own_mesh}">
-            <mesh filename="package://aerial_manipulation/meshes/black_propeller.stl"
+            <mesh filename="package://tobas_description/meshes/harrier/black_propeller.stl"
               scale="${radius_rotor} ${radius_rotor} ${radius_rotor}" /> <!-- The propeller meshes have a radius of 1m -->
             <!-- <box size="${2*radius_rotor} 0.01 0.005"/> -->

File: tobas_description/urdf/hummingbird.xacro (robot description, xacro)
@@ -23,5 +23,5 @@
   <xacro:property name="rotor_velocity_slowdown_sim" value="10" />
   <xacro:property name="use_mesh_file" value="true" />
-  <xacro:property name="mesh_file" value="package://rotors_description/meshes/hummingbird.dae" />
+  <xacro:property name="mesh_file" value="package://tobas_description/meshes/hummingbird.dae" />
   <xacro:property name="mass" value="0.68" /> <!-- [kg] -->
   <xacro:property name="body_width" value="0.1" /> <!-- [m] -->

File: tobas_description/urdf/iris.xacro (robot description, xacro)
@@ -6,5 +6,5 @@
   <xacro:property name="rotor_velocity_slowdown_sim" value="10" />
   <xacro:property name="use_mesh_file" value="true" />
-  <xacro:property name="mesh_file" value="package://rotors_description/meshes/iris.dae" />
+  <xacro:property name="mesh_file" value="package://tobas_description/meshes/iris.dae" />
   <xacro:property name="mass" value="1.5" /> <!-- [kg] -->
   <xacro:property name="body_width" value="0.47" /> <!-- [m] -->

File: tobas_description/urdf/multirotor_base.xacro (robot description, xacro)
@@ -97,5 +97,5 @@
           </xacro:if>
           <xacro:unless value="${use_own_mesh}">
-            <mesh filename="package://rotors_description/meshes/propeller_${direction}.dae"
+            <mesh filename="package://tobas_description/meshes/propeller_${direction}.dae"
               scale="${radius_rotor} ${radius_rotor} ${radius_rotor}" /> <!-- The propeller meshes have a radius of 1m -->
             <!-- <box size="${2*radius_rotor} 0.01 0.005"/> -->

File: tobas_description/urdf/neo11.xacro (robot description, xacro)
@@ -22,5 +22,5 @@
   <xacro:property name="rotor_velocity_slowdown_sim" value="10" />
   <xacro:property name="use_mesh_file" value="true" />
-  <xacro:property name="mesh_file" value="package://rotors_description/meshes/neo11.dae" />
+  <xacro:property name="mesh_file" value="package://tobas_description/meshes/neo11.dae" />
   <xacro:property name="mass" value="3.42" /> <!-- [kg] -->
   <xacro:property name="body_width" value="0.2" /> <!-- [m] -->
@@ -85,5 +85,5 @@
     color="Red"
     use_own_mesh="true"
-    mesh="package://rotors_description/meshes/neo11_propeller_ccw.dae">
+    mesh="package://tobas_description/meshes/neo11_propeller_ccw.dae">
     <origin xyz="${front_propeller_x} ${front_propeller_y} ${rotor_offset_top}" rpy="${5*pi/180} 0 ${30*pi/180}" />
     <xacro:insert_block name="rotor_inertia" />
@@ -106,5 +106,5 @@
     color="Blue"
     use_own_mesh="true"
-    mesh="package://rotors_description/meshes/neo11_propeller_cw.dae">
+    mesh="package://tobas_description/meshes/neo11_propeller_cw.dae">
     <origin xyz="${side_propeller_x} ${side_propeller_y} ${rotor_offset_top}" rpy="0 ${-5*pi/180} 0" />
     <xacro:insert_block name="rotor_inertia" />
@@ -126,5 +126,5 @@
     color="Blue"
     use_own_mesh="true"
-    mesh="package://rotors_description/meshes/neo11_propeller_ccw.dae">
+    mesh="package://tobas_description/meshes/neo11_propeller_ccw.dae">
     <origin xyz="${back_propeller_x} ${back_propeller_y} ${rotor_offset_top}" rpy="${5*pi/180} 0 ${150*pi/180}" />
     <xacro:insert_block name="rotor_inertia" />
@@ -146,5 +146,5 @@
     color="Blue"
     use_own_mesh="true"
-    mesh="package://rotors_description/meshes/neo11_propeller_cw.dae">
+    mesh="package://tobas_description/meshes/neo11_propeller_cw.dae">
     <origin xyz="${back_propeller_x} -${back_propeller_y} ${rotor_offset_top}" rpy="${-5*pi/180} 0 ${-150*pi/180}" />
     <xacro:insert_block name="rotor_inertia" />
@@ -167,5 +167,5 @@
     color="Blue"
     use_own_mesh="true"
-    mesh="package://rotors_description/meshes/neo11_propeller_ccw.dae">
+    mesh="package://tobas_description/meshes/neo11_propeller_ccw.dae">
     <origin xyz="${side_propeller_x} -${side_propeller_y} ${rotor_offset_top}" rpy="0 ${5*pi/180} ${pi}" />
     <xacro:insert_block name="rotor_inertia" />
@@ -188,5 +188,5 @@
     color="Red"
     use_own_mesh="true"
-    mesh="package://rotors_description/meshes/neo11_propeller_cw.dae">
+    mesh="package://tobas_description/meshes/neo11_propeller_cw.dae">
     <origin xyz="${front_propeller_x} -${front_propeller_y} ${rotor_offset_top}" rpy="${-5*pi/180} 0 ${-30*pi/180}" />
     <xacro:insert_block name="rotor_inertia" />

File: tobas_description/urdf/neo9.xacro (robot description, xacro)
@@ -22,5 +22,5 @@
   <xacro:property name="rotor_velocity_slowdown_sim" value="10" />
   <xacro:property name="use_mesh_file" value="true" />
-  <xacro:property name="mesh_file" value="package://rotors_description/meshes/neo9.dae" />
+  <xacro:property name="mesh_file" value="package://tobas_description/meshes/neo9.dae" />
   <xacro:property name="mass" value="2.662" /> <!-- [kg] -->
   <xacro:property name="body_width" value="0.2" /> <!-- [m] -->
@@ -85,5 +85,5 @@
     color="Red"
     use_own_mesh="true"
-    mesh="package://rotors_description/meshes/neo9_propeller_ccw.dae">
+    mesh="package://tobas_description/meshes/neo9_propeller_ccw.dae">
     <origin xyz="${front_propeller_x} ${front_propeller_y} ${rotor_offset_top}" rpy="${5*pi/180} 0 ${30*pi/180}" />
     <xacro:insert_block name="rotor_inertia" />
@@ -106,5 +106,5 @@
     color="Blue"
     use_own_mesh="true"
-    mesh="package://rotors_description/meshes/neo9_propeller_cw.dae">
+    mesh="package://tobas_description/meshes/neo9_propeller_cw.dae">
     <origin xyz="${side_propeller_x} ${side_propeller_y} ${rotor_offset_top}" rpy="0 ${-5*pi/180} 0" />
     <xacro:insert_block name="rotor_inertia" />
@@ -126,5 +126,5 @@
     color="Blue"
     use_own_mesh="true"
-    mesh="package://rotors_description/meshes/neo9_propeller_ccw.dae">
+    mesh="package://tobas_description/meshes/neo9_propeller_ccw.dae">
     <origin xyz="${back_propeller_x} ${back_propeller_y} ${rotor_offset_top}" rpy="${5*pi/180} 0 ${150*pi/180}" />
     <xacro:insert_block name="rotor_inertia" />
@@ -146,5 +146,5 @@
     color="Blue"
     use_own_mesh="true"
-    mesh="package://rotors_description/meshes/neo9_propeller_cw.dae">
+    mesh="package://tobas_description/meshes/neo9_propeller_cw.dae">
     <origin xyz="${back_propeller_x} -${back_propeller_y} ${rotor_offset_top}" rpy="${-5*pi/180} 0 ${-150*pi/180}" />
     <xacro:insert_block name="rotor_inertia" />
@@ -167,5 +167,5 @@
     color="Blue"
     use_own_mesh="true"
-    mesh="package://rotors_description/meshes/neo9_propeller_ccw.dae">
+    mesh="package://tobas_description/meshes/neo9_propeller_ccw.dae">
     <origin xyz="${side_propeller_x} -${side_propeller_y} ${rotor_offset_top}" rpy="0 ${5*pi/180} ${pi}" />
     <xacro:insert_block name="rotor_inertia" />
@@ -188,5 +188,5 @@
     color="Red"
     use_own_mesh="true"
-    mesh="package://rotors_description/meshes/neo9_propeller_cw.dae">
+    mesh="package://tobas_description/meshes/neo9_propeller_cw.dae">
     <origin xyz="${front_propeller_x} -${front_propeller_y} ${rotor_offset_top}" rpy="${-5*pi/180} 0 ${-30*pi/180}" />
     <xacro:insert_block name="rotor_inertia" />

File: tobas_description/urdf/pelican.xacro (robot description, xacro)
@@ -23,5 +23,5 @@
   <xacro:property name="rotor_velocity_slowdown_sim" value="10" />
   <xacro:property name="use_mesh_file" value="true" />
-  <xacro:property name="mesh_file" value="package://rotors_description/meshes/pelican.dae" />
+  <xacro:property name="mesh_file" value="package://tobas_description/meshes/pelican.dae" />
   <xacro:property name="mass" value="1.0" /> <!-- [kg] -->
   <xacro:property name="body_width" value="0.1" /> <!-- [m] -->

File: tobas_description/urdf/techpod.xacro (robot description, xacro)
@@ -32,5 +32,5 @@
   <xacro:property name="body_height" value="0.303" /> <!-- [m] -->
   <xacro:property name="body_color" value="Gray" />
-  <xacro:property name="body_mesh_file" value="package://rotors_description/meshes/techpod/techpod_body.dae" />
+  <xacro:property name="body_mesh_file" value="package://tobas_description/meshes/techpod/techpod_body.dae" />
   <!-- Aileron properties -->
   <xacro:property name="aileron_length" value="0.053" /> <!-- [m] -->
@@ -40,6 +40,6 @@
   <xacro:property name="aileron_max_angle" value="0.349066" /> <!-- [rad] -->
   <xacro:property name="aileron_color" value="Red" />
-  <xacro:property name="aileron_left_mesh_file" value="package://rotors_description/meshes/techpod/techpod_aileron_left.dae" />
-  <xacro:property name="aileron_right_mesh_file" value="package://rotors_description/meshes/techpod/techpod_aileron_right.dae" />
+  <xacro:property name="aileron_left_mesh_file" value="package://tobas_description/meshes/techpod/techpod_aileron_left.dae" />
+  <xacro:property name="aileron_right_mesh_file" value="package://tobas_description/meshes/techpod/techpod_aileron_right.dae" />
   <!-- Elevator properties -->
   <xacro:property name="elevator_length" value="0.051" /> <!-- [m] -->
@@ -49,5 +49,5 @@
   <xacro:property name="elevator_max_angle" value="0.349066" /> <!-- [rad] -->
   <xacro:property name="elevator_color" value="Blue" />
-  <xacro:property name="elevator_mesh_file" value="package://rotors_description/meshes/techpod/techpod_elevator.dae" />
+  <xacro:property name="elevator_mesh_file" value="package://tobas_description/meshes/techpod/techpod_elevator.dae" />
   <!-- Flap properties -->
   <xacro:property name="flap_length" value="0.076" /> <!-- [m] -->
@@ -57,6 +57,6 @@
   <xacro:property name="flap_max_angle" value="0.0" /> <!-- [rad] -->
   <xacro:property name="flap_color" value="Yellow" />
-  <xacro:property name="flap_left_mesh_file" value="package://rotors_description/meshes/techpod/techpod_flap_left.dae" />
-  <xacro:property name="flap_right_mesh_file" value="package://rotors_description/meshes/techpod/techpod_flap_right.dae" />
+  <xacro:property name="flap_left_mesh_file" value="package://tobas_description/meshes/techpod/techpod_flap_left.dae" />
+  <xacro:property name="flap_right_mesh_file" value="package://tobas_description/meshes/techpod/techpod_flap_right.dae" />
   <!-- Rudder properties -->
   <xacro:property name="rudder_length" value="0.129" />
@@ -66,5 +66,5 @@
   <xacro:property name="rudder_max_angle" value="0.349066" />
   <xacro:property name="rudder_color" value="Orange" />
-  <xacro:property name="rudder_mesh_file" value="package://rotors_description/meshes/techpod/techpod_rudder.dae" />
+  <xacro:property name="rudder_mesh_file" value="package://tobas_description/meshes/techpod/techpod_rudder.dae" />
   <!-- Propeller properties -->
   <xacro:property name="propeller_direction" value="cw" />
@@ -72,5 +72,5 @@
   <xacro:property name="propeller_height" value="0.003" />
   <xacro:property name="propeller_color" value="Gray" />
-  <xacro:property name="propeller_mesh_file" value="package://rotors_description/meshes/propeller_${propeller_direction}.dae" />
+  <xacro:property name="propeller_mesh_file" value="package://tobas_description/meshes/propeller_${propeller_direction}.dae" />
   <!-- Inertia of the main body -->
   <xacro:property name="body_inertia">

Commit message: .

File: tobas_description/urdf/ardrone.xacro (robot description, xacro)
@@ -1,6 +1,7 @@
 <?xml version="1.0"?>
 <robot name="ardrone" xmlns:xacro="http://ros.org/wiki/xacro">
+  <!-- Included URDF Files -->
+  <xacro:include filename="$(find tobas_description)/urdf/multirotor_base.xacro" />
   <!-- Properties -->
-  <!-- <xacro:property name="namespace" value="$(arg namespace)" /> -->
   <xacro:property name="namespace" value="ardrone" />
   <xacro:property name="rotor_velocity_slowdown_sim" value="10" />
@@ -32,7 +33,4 @@
     <xacro:box_inertia x="${radius_rotor}" y="0.015" z="0.003" mass="${mass_rotor*rotor_velocity_slowdown_sim}" />
   </xacro:property>
-  <!-- Included URDF Files -->
-  <!-- <xacro:include filename="$(find rotors_description)/urdf/multirotor_base.xacro" /> -->
-  <xacro:include filename="$(find tobas_description)/urdf/multirotor_base.xacro" />
   <!-- Instantiate multirotor_base_macro once -->
   <xacro:multirotor_base_macro

File: tobas_description/urdf/asymmetric_quadrotor.xacro (robot description, xacro)
@@ -2,8 +2,6 @@
 <robot name="asymmetric_quadrotor" xmlns:xacro="http://ros.org/wiki/xacro">
   <!-- Included URDF Files -->
-  <!-- <xacro:include filename="$(find rotors_description)/urdf/multirotor_base.xacro" /> -->
   <xacro:include filename="$(find tobas_description)/urdf/multirotor_base.xacro" />
   <!-- Properties  -->
-  <!-- <xacro:property name="namespace" value="$(arg namespace)" /> -->
   <xacro:property name="namespace" value="asymmetric_quadrotor" />
   <xacro:property name="use_mesh_file" value="false" />

File: tobas_description/urdf/firefly.xacro (robot description, xacro)
@@ -1,6 +1,7 @@
 <?xml version="1.0"?>
 <robot name="firefly" xmlns:xacro="http://ros.org/wiki/xacro">
+  <!-- Included URDF Files -->
+  <xacro:include filename="$(find tobas_description)/urdf/multirotor_base.xacro" />
   <!-- Properties -->
-  <!-- <xacro:property name="namespace" value="$(arg namespace)" /> -->
   <xacro:property name="namespace" value="firefly" />
   <xacro:property name="rotor_velocity_slowdown_sim" value="10" />
@@ -31,7 +32,4 @@
     <xacro:box_inertia x="${radius_rotor}" y="0.015" z="0.003" mass="${mass_rotor*rotor_velocity_slowdown_sim}" />
   </xacro:property>
-  <!-- Included URDF Files -->
-  <!-- <xacro:include filename="$(find rotors_description)/urdf/multirotor_base.xacro" /> -->
-  <xacro:include filename="$(find tobas_description)/urdf/multirotor_base.xacro" />
   <!-- Instantiate multirotor_base_macro once -->
   <xacro:multirotor_base_macro

File: tobas_description/urdf/harrierD7.xacro (robot description, xacro)
@@ -1,4 +1,6 @@
 <?xml version="1.0"?>
 <robot name="harrier" xmlns:xacro="http://ros.org/wiki/xacro">
+  <!-- Included URDF Files -->
+  <xacro:include filename="$(find tobas_description)/urdf/harrier/multirotor_base_harrier.xacro" />
   <!-- Properties  -->
   <xacro:property name="namespace" value="harrier" />
@@ -29,6 +31,4 @@
     <xacro:box_inertia x="${radius_rotor}" y="0.1" z="0.003" mass="${mass_rotor*rotor_velocity_slowdown_sim}" />
   </xacro:property>
-  <!-- Included URDF Files -->
-  <xacro:include filename="$(find tobas_description)/urdf/harrier/multirotor_base_harrier.xacro" />
   <!-- Instantiate multirotor_base_macro once -->
   <xacro:multirotor_base_macro

File: tobas_description/urdf/hummingbird.xacro (robot description, xacro)
@@ -1,7 +1,7 @@
 <?xml version="1.0"?>
 <robot name="hummingbird" xmlns:xacro="http://ros.org/wiki/xacro">
-  <!-- Properties (Taken from Novel Dynamic Inversion Architecture Design
-for Quadrocopter Control by Jian Wang et al.) -->
-  <!-- <xacro:property name="namespace" value="$(arg namespace)" /> -->
+  <!-- Included URDF Files -->
+  <xacro:include filename="$(find tobas_description)/urdf/multirotor_base.xacro" />
+  <!-- Properties (Taken from Novel Dynamic Inversion Architecture Design for Quadrocopter Control by Jian Wang et al.) -->
   <xacro:property name="namespace" value="hummingbird" />
   <xacro:property name="rotor_velocity_slowdown_sim" value="10" />
@@ -30,7 +30,4 @@
     <xacro:box_inertia x="${radius_rotor}" y="0.015" z="0.003" mass="${mass_rotor*rotor_velocity_slowdown_sim}" />
   </xacro:property>
-  <!-- Included URDF Files -->
-  <!-- <xacro:include filename="$(find rotors_description)/urdf/multirotor_base.xacro" /> -->
-  <xacro:include filename="$(find tobas_description)/urdf/multirotor_base.xacro" />
   <!-- Instantiate multirotor_base_macro once -->
   <xacro:multirotor_base_macro

File: tobas_description/urdf/iris.xacro (robot description, xacro)
@@ -1,6 +1,7 @@
 <?xml version="1.0"?>
 <robot name="iris" xmlns:xacro="http://ros.org/wiki/xacro">
+  <!-- Included URDF Files -->
+  <xacro:include filename="$(find tobas_description)/urdf/multirotor_base.xacro" />
   <!-- Properties -->
-  <!-- <xacro:property name="namespace" value="$(arg namespace)" /> -->
   <xacro:property name="namespace" value="iris" />
   <xacro:property name="rotor_velocity_slowdown_sim" value="10" />
@@ -35,7 +36,4 @@
     <xacro:box_inertia x="${radius_rotor}" y="0.015" z="0.003" mass="${mass_rotor*rotor_velocity_slowdown_sim}" />
   </xacro:property>
-  <!-- Included URDF Files -->
-  <!-- <xacro:include filename="$(find rotors_description)/urdf/multirotor_base.xacro" /> -->
-  <xacro:include filename="$(find tobas_description)/urdf/multirotor_base.xacro" />
   <!-- Instantiate multirotor_base_macro once -->
   <xacro:multirotor_base_macro

File: tobas_description/urdf/neo11.xacro (robot description, xacro)
@@ -1,6 +1,7 @@
 <?xml version="1.0"?>
 <robot name="neo11" xmlns:xacro="http://ros.org/wiki/xacro">
+  <!-- Included URDF Files -->
+  <xacro:include filename="$(find tobas_description)/urdf/multirotor_base.xacro" />
   <!-- Properties -->
-  <!-- <xacro:property name="namespace" value="$(arg namespace)" /> -->
   <xacro:property name="namespace" value="neo11" />
   <xacro:property name="rotor_velocity_slowdown_sim" value="10" />
@@ -37,7 +38,4 @@
     <xacro:box_inertia x="${radius_rotor}" y="0.015" z="0.003" mass="${mass_rotor*rotor_velocity_slowdown_sim}" />
   </xacro:property>
-  <!-- Included URDF Files -->
-  <!-- <xacro:include filename="$(find rotors_description)/urdf/multirotor_base.xacro" /> -->
-  <xacro:include filename="$(find tobas_description)/urdf/multirotor_base.xacro" />
   <!-- Instantiate multirotor_base_macro once -->
   <xacro:multirotor_base_macro

File: tobas_description/urdf/neo9.xacro (robot description, xacro)
@@ -1,6 +1,7 @@
 <?xml version="1.0"?>
 <robot name="neo9" xmlns:xacro="http://ros.org/wiki/xacro">
+  <!-- Included URDF Files -->
+  <xacro:include filename="$(find tobas_description)/urdf/multirotor_base.xacro" />
   <!-- Properties -->
-  <!-- <xacro:property name="namespace" value="$(arg mav_name)" /> -->
   <xacro:property name="namespace" value="neo9" />
   <xacro:property name="rotor_velocity_slowdown_sim" value="10" />
@@ -37,7 +38,4 @@
     <xacro:box_inertia x="${radius_rotor}" y="0.015" z="0.003" mass="${mass_rotor*rotor_velocity_slowdown_sim}" />
   </xacro:property>
-  <!-- Included URDF Files -->
-  <!-- <xacro:include filename="$(find rotors_description)/urdf/multirotor_base.xacro" /> -->
-  <xacro:include filename="$(find tobas_description)/urdf/multirotor_base.xacro" />
   <!-- Instantiate multirotor_base_macro once -->
   <xacro:multirotor_base_macro

File: tobas_description/urdf/pelican.xacro (robot description, xacro)
@@ -1,7 +1,7 @@
 <?xml version="1.0"?>
 <robot name="pelican" xmlns:xacro="http://ros.org/wiki/xacro">
+  <!-- Included URDF Files -->
+  <xacro:include filename="$(find tobas_description)/urdf/multirotor_base.xacro" />
   <!-- Properties  -->
-  <!-- TODO(ff): Update these params when identifying the model. -->
-  <!-- <xacro:property name="namespace" value="$(arg namespace)" /> -->
   <xacro:property name="namespace" value="pelican" />
   <xacro:property name="rotor_velocity_slowdown_sim" value="10" />
@@ -30,7 +30,4 @@
     <xacro:box_inertia x="${radius_rotor}" y="0.015" z="0.003" mass="${mass_rotor*rotor_velocity_slowdown_sim}" />
   </xacro:property>
-  <!-- Included URDF Files -->
-  <!-- <xacro:include filename="$(find rotors_description)/urdf/multirotor_base.xacro" /> -->
-  <xacro:include filename="$(find tobas_description)/urdf/multirotor_base.xacro" />
   <!-- Instantiate multirotor_base_macro once -->
   <xacro:multirotor_base_macro

File: tobas_description/urdf/techpod.xacro (robot description, xacro)
@@ -2,5 +2,4 @@
 <robot name="techpod" xmlns:xacro="http://ros.org/wiki/xacro">
   <!-- Global properties -->
-  <!-- <xacro:property name="namespace" value="$(arg namespace)" /> -->
   <xacro:property name="namespace" value="techpod" />
   <xacro:property name="rotor_velocity_slowdown_sim" value="10" />
