Commit message: 使っていない定数を削除

File: tobas_description/urdf/ardrone.xacro (robot description, xacro)
@@ -3,7 +3,10 @@
   <!-- Included URDF Files -->
   <xacro:include filename="$(find tobas_description)/urdf/components/multirotor_base.xacro" />
+  <!-- Constants -->
+  <xacro:property name="sin30" value="0.5" />
+  <xacro:property name="cos30" value="0.866025403784" />
+  <xacro:property name="sqrt2" value="1.4142135623730951" />
   <!-- Properties -->
   <xacro:property name="namespace" value="ardrone" />
-  <xacro:property name="rotor_velocity_slowdown_sim" value="10" />
   <xacro:property name="use_mesh_file" value="true" />
   <xacro:property name="mesh_file" value="package://tobas_description/meshes/ardrone.dae" />
@@ -15,21 +18,11 @@
   <xacro:property name="rotor_offset_top" value="0.023" /> <!-- [m] -->
   <xacro:property name="radius_rotor" value="0.1" /> <!-- [m] -->
-  <xacro:property name="motor_constant" value="8.54858e-06" /> <!-- [kg.m/s^2] -->
-  <xacro:property name="moment_constant" value="0.016" /> <!-- [m] -->
-  <xacro:property name="time_constant_up" value="0.0125" /> <!-- [s] -->
-  <xacro:property name="time_constant_down" value="0.025" /> <!-- [s] -->
-  <xacro:property name="max_rot_velocity" value="838" /> <!-- [rad/s] -->
-  <xacro:property name="sin30" value="0.5" />
-  <xacro:property name="cos30" value="0.866025403784" />
-  <xacro:property name="sqrt2" value="1.4142135623730951" />
-  <xacro:property name="rotor_drag_coefficient" value="8.06428e-05" />
-  <xacro:property name="rolling_moment_coefficient" value="0.000001" />
   <!-- Property Blocks -->
   <xacro:property name="body_inertia">
-    <inertia ixx="0.0347563" ixy="0.0" ixz="0.0" iyy="0.0458929" iyz="0.0" izz="0.0977" /> <!-- [kg.m^2] [kg.m^2] [kg.m^2] [kg.m^2] [kg.m^2] [kg.m^2] -->
+    <inertia ixx="0.0347563" ixy="0.0" ixz="0.0" iyy="0.0458929" iyz="0.0" izz="0.0977" /> <!-- [kg.m^2] -->
   </xacro:property>
   <!-- inertia of a single rotor, assuming it is a cuboid. Height=3mm, width=15mm -->
   <xacro:property name="rotor_inertia">
-    <xacro:box_inertia x="${radius_rotor}" y="0.015" z="0.003" mass="${mass_rotor*rotor_velocity_slowdown_sim}" />
+    <xacro:box_inertia x="${radius_rotor}" y="0.015" z="0.003" mass="${mass_rotor}" />
   </xacro:property>
   <!-- Instantiate multirotor_base_macro once -->

File: tobas_description/urdf/asymmetric_quadrotor.xacro (robot description, xacro)
@@ -6,5 +6,4 @@
   <xacro:property name="namespace" value="asymmetric_quadrotor" />
   <xacro:property name="use_mesh_file" value="false" />
-  <xacro:property name="rotor_velocity_slowdown_sim" value="10" />
   <xacro:property name="mass_arm" value="0.01" /> <!-- [kg] -->
   <xacro:property name="mass" value="1.0" /> <!-- [kg] -->
@@ -15,18 +14,11 @@
   <xacro:property name="rotor_offset_top" value="0.03" /> <!-- [m] -->
   <xacro:property name="radius_rotor" value="0.128" /> <!-- [m] -->
-  <xacro:property name="motor_constant" value="9.9865e-06" /> <!-- [kg m/s^2] -->
-  <xacro:property name="moment_constant" value="0.016" /> <!-- [m] -->
-  <xacro:property name="time_constant_up" value="0.0125" /> <!-- [s] -->
-  <xacro:property name="time_constant_down" value="0.025" /> <!-- [s] -->
-  <xacro:property name="max_rot_velocity" value="1000" /> <!-- [rad/s] -->
-  <xacro:property name="rotor_drag_coefficient" value="8.06428e-05" />
-  <xacro:property name="rolling_moment_coefficient" value="0.000001" />
   <!-- Property Blocks -->
   <xacro:property name="body_inertia">
-    <inertia ixx="0.01" ixy="0.0" ixz="0.0" iyy="0.01" iyz="0.0" izz="0.02" /> <!-- [kg m^2] [kg m^2] [kg m^2] [kg m^2] [kg m^2] [kg m^2] -->
+    <inertia ixx="0.01" ixy="0.0" ixz="0.0" iyy="0.01" iyz="0.0" izz="0.02" /> <!-- [kg m^2] -->
   </xacro:property>
   <!-- inertia of a single rotor, assuming it is a cuboid. Height=3mm, width=15mm -->
   <xacro:property name="rotor_inertia">
-    <xacro:box_inertia x="${radius_rotor}" y="0.015" z="0.003" mass="${mass_rotor*rotor_velocity_slowdown_sim}" />
+    <xacro:box_inertia x="${radius_rotor}" y="0.015" z="0.003" mass="${mass_rotor}" />
   </xacro:property>
   <!-- Instantiate multirotor_base_macro once -->

File: tobas_description/urdf/firefly.xacro (robot description, xacro)
@@ -3,7 +3,9 @@
   <!-- Included URDF Files -->
   <xacro:include filename="$(find tobas_description)/urdf/components/multirotor_base.xacro" />
+  <!-- Constants -->
+  <xacro:property name="sin30" value="0.5" />
+  <xacro:property name="cos30" value="0.866025403784" />
   <!-- Properties -->
   <xacro:property name="namespace" value="firefly" />
-  <xacro:property name="rotor_velocity_slowdown_sim" value="10" />
   <xacro:property name="use_mesh_file" value="true" />
   <xacro:property name="mesh_file" value="package://tobas_description/meshes/firefly.dae" />
@@ -15,20 +17,11 @@
   <xacro:property name="rotor_offset_top" value="0.037" /> <!-- [m] -->
   <xacro:property name="radius_rotor" value="0.1" /> <!-- [m] -->
-  <xacro:property name="motor_constant" value="8.54858e-06" /> <!-- [kg m/s^2] -->
-  <xacro:property name="moment_constant" value="0.016" /> <!-- [m] -->
-  <xacro:property name="time_constant_up" value="0.0125" /> <!-- [s] -->
-  <xacro:property name="time_constant_down" value="0.025" /> <!-- [s] -->
-  <xacro:property name="max_rot_velocity" value="838" /> <!-- [rad/s] -->
-  <xacro:property name="sin30" value="0.5" />
-  <xacro:property name="cos30" value="0.866025403784" />
-  <xacro:property name="rotor_drag_coefficient" value="8.06428e-05" />
-  <xacro:property name="rolling_moment_coefficient" value="0.000001" />
   <!-- Property Blocks -->
   <xacro:property name="body_inertia">
-    <inertia ixx="0.0347563" ixy="0.0" ixz="0.0" iyy="0.0458929" iyz="0.0" izz="0.0977" /> <!-- [kg m^2] [kg m^2] [kg m^2] [kg m^2] [kg m^2] [kg m^2] -->
+    <inertia ixx="0.0347563" ixy="0.0" ixz="0.0" iyy="0.0458929" iyz="0.0" izz="0.0977" /> <!-- [kg m^2] -->
   </xacro:property>
   <!-- inertia of a single rotor, assuming it is a cuboid. Height=3mm, width=15mm -->
   <xacro:property name="rotor_inertia">
-    <xacro:box_inertia x="${radius_rotor}" y="0.015" z="0.003" mass="${mass_rotor*rotor_velocity_slowdown_sim}" />
+    <xacro:box_inertia x="${radius_rotor}" y="0.015" z="0.003" mass="${mass_rotor}" />
   </xacro:property>
   <!-- Instantiate multirotor_base_macro once -->

File: tobas_description/urdf/harrierD7.xacro (robot description, xacro)
@@ -3,5 +3,4 @@
   <!-- Properties  -->
   <xacro:property name="namespace" value="harrier" />
-  <xacro:property name="rotor_velocity_slowdown_sim" value="10" />
   <xacro:property name="use_mesh_file" value="true" />
   <xacro:property name="mesh_file" value="package://tobas_description/meshes/harrier/HarrierD7_reduced.stl" />
@@ -14,18 +13,11 @@
   <xacro:property name="rotor_offset_top" value="0.04" /> <!-- [m] -->
   <xacro:property name="radius_rotor" value="0.45" /> <!-- [m] -->
-  <xacro:property name="motor_constant" value="4.63e-04" /> <!-- [kg m/s^2] -->
-  <xacro:property name="moment_constant" value="0.0173" /> <!-- [m] -->
-  <xacro:property name="time_constant_up" value="0.0125" /> <!-- [s] -->
-  <xacro:property name="time_constant_down" value="0.025" /> <!-- [s] -->
-  <xacro:property name="max_rot_velocity" value="650" /> <!-- [rad/s] -->
-  <xacro:property name="rotor_drag_coefficient" value="8.06428e-05" />
-  <xacro:property name="rolling_moment_coefficient" value="0.000001" />
   <!-- Property Blocks -->
   <xacro:property name="body_inertia">
-    <inertia ixx="1.57" ixy="0.0" ixz="0.0" iyy="3.93" iyz="0.0" izz="2.59" /> <!-- [kg m^2] [kg m^2] [kg m^2] [kg m^2] [kg m^2] [kg m^2] -->
+    <inertia ixx="1.57" ixy="0.0" ixz="0.0" iyy="3.93" iyz="0.0" izz="2.59" /> <!-- [kg m^2] -->
   </xacro:property>
   <!-- inertia of a single rotor, assuming it is a cuboid. Height=3mm, width=15mm -->
   <xacro:property name="rotor_inertia">
-    <xacro:box_inertia x="${radius_rotor}" y="0.1" z="0.003" mass="${mass_rotor * rotor_velocity_slowdown_sim}" />
+    <xacro:box_inertia x="${radius_rotor}" y="0.1" z="0.003" mass="${mass_rotor}" />
   </xacro:property>
   <!-- Included URDF Files. It requires some properties defined beforehand. -->

File: tobas_description/urdf/hummingbird.xacro (robot description, xacro)
@@ -5,5 +5,4 @@
   <!-- Properties (Taken from Novel Dynamic Inversion Architecture Design for Quadrocopter Control by Jian Wang et al.) -->
   <xacro:property name="namespace" value="hummingbird" />
-  <xacro:property name="rotor_velocity_slowdown_sim" value="10" />
   <xacro:property name="use_mesh_file" value="true" />
   <xacro:property name="mesh_file" value="package://tobas_description/meshes/hummingbird.dae" />
@@ -15,18 +14,11 @@
   <xacro:property name="rotor_offset_top" value="0.01" /> <!-- [m] -->
   <xacro:property name="radius_rotor" value="0.1" /> <!-- [m] -->
-  <xacro:property name="motor_constant" value="8.54858e-06" /> <!-- [kg m/s^2] -->
-  <xacro:property name="moment_constant" value="0.016" /> <!-- [m] -->
-  <xacro:property name="time_constant_up" value="0.0125" /> <!-- [s] -->
-  <xacro:property name="time_constant_down" value="0.025" /> <!-- [s] -->
-  <xacro:property name="max_rot_velocity" value="838" /> <!-- [rad/s] -->
-  <xacro:property name="rotor_drag_coefficient" value="8.06428e-05" />
-  <xacro:property name="rolling_moment_coefficient" value="0.000001" />
   <!-- Property Blocks -->
   <xacro:property name="body_inertia">
-    <inertia ixx="0.007" ixy="0.0" ixz="0.0" iyy="0.007" iyz="0.0" izz="0.012" /> <!-- [kg m^2] [kg m^2] [kg m^2] [kg m^2] [kg m^2] [kg m^2] -->
+    <inertia ixx="0.007" ixy="0.0" ixz="0.0" iyy="0.007" iyz="0.0" izz="0.012" /> <!-- [kg m^2] -->
   </xacro:property>
   <!-- inertia of a single rotor, assuming it is a cuboid. Height=3mm, width=15mm -->
   <xacro:property name="rotor_inertia">
-    <xacro:box_inertia x="${radius_rotor}" y="0.015" z="0.003" mass="${mass_rotor*rotor_velocity_slowdown_sim}" />
+    <xacro:box_inertia x="${radius_rotor}" y="0.015" z="0.003" mass="${mass_rotor}" />
   </xacro:property>
   <!-- Instantiate multirotor_base_macro once -->

File: tobas_description/urdf/iris.xacro (robot description, xacro)
@@ -3,7 +3,10 @@
   <!-- Included URDF Files -->
   <xacro:include filename="$(find tobas_description)/urdf/components/multirotor_base.xacro" />
+  <!-- Constants -->
+  <xacro:property name="sin30" value="0.5" />
+  <xacro:property name="cos30" value="0.866025403784" />
+  <xacro:property name="sqrt2" value="1.4142135623730951" />
   <!-- Properties -->
   <xacro:property name="namespace" value="iris" />
-  <xacro:property name="rotor_velocity_slowdown_sim" value="10" />
   <xacro:property name="use_mesh_file" value="true" />
   <xacro:property name="mesh_file" value="package://tobas_description/meshes/iris.dae" />
@@ -18,21 +21,11 @@
   <xacro:property name="rotor_offset_top" value="0.023" /> <!-- [m] -->
   <xacro:property name="radius_rotor" value="0.1" /> <!-- [m] -->
-  <xacro:property name="motor_constant" value="8.54858e-06" /> <!-- [kg.m/s^2] -->
-  <xacro:property name="moment_constant" value="0.016" /> <!-- [m] -->
-  <xacro:property name="time_constant_up" value="0.0125" /> <!-- [s] -->
-  <xacro:property name="time_constant_down" value="0.025" /> <!-- [s] -->
-  <xacro:property name="max_rot_velocity" value="838" /> <!-- [rad/s] -->
-  <xacro:property name="sin30" value="0.5" />
-  <xacro:property name="cos30" value="0.866025403784" />
-  <xacro:property name="sqrt2" value="1.4142135623730951" />
-  <xacro:property name="rotor_drag_coefficient" value="8.06428e-05" />
-  <xacro:property name="rolling_moment_coefficient" value="0.000001" />
   <!-- Property Blocks -->
   <xacro:property name="body_inertia">
-    <inertia ixx="0.0347563" ixy="0.0" ixz="0.0" iyy="0.0458929" iyz="0.0" izz="0.0977" /> <!-- [kg.m^2] [kg.m^2] [kg.m^2] [kg.m^2] [kg.m^2] [kg.m^2] -->
+    <inertia ixx="0.0347563" ixy="0.0" ixz="0.0" iyy="0.0458929" iyz="0.0" izz="0.0977" /> <!-- [kg m^2] -->
   </xacro:property>
   <!-- inertia of a single rotor, assuming it is a cuboid. Height=3mm, width=15mm -->
   <xacro:property name="rotor_inertia">
-    <xacro:box_inertia x="${radius_rotor}" y="0.015" z="0.003" mass="${mass_rotor*rotor_velocity_slowdown_sim}" />
+    <xacro:box_inertia x="${radius_rotor}" y="0.015" z="0.003" mass="${mass_rotor}" />
   </xacro:property>
   <!-- Instantiate multirotor_base_macro once -->

File: tobas_description/urdf/neo11.xacro (robot description, xacro)
@@ -3,7 +3,9 @@
   <!-- Included URDF Files -->
   <xacro:include filename="$(find tobas_description)/urdf/components/multirotor_base.xacro" />
+  <!-- Constants -->
+  <xacro:property name="sin30" value="0.5" />
+  <xacro:property name="cos30" value="0.866025403784" />
   <!-- Properties -->
   <xacro:property name="namespace" value="neo11" />
-  <xacro:property name="rotor_velocity_slowdown_sim" value="10" />
   <xacro:property name="use_mesh_file" value="true" />
   <xacro:property name="mesh_file" value="package://tobas_description/meshes/neo11.dae" />
@@ -15,11 +17,4 @@
   <xacro:property name="rotor_offset_top" value="0.028" /> <!-- [m] -->
   <xacro:property name="radius_rotor" value="0.1397" /> <!-- [m] -->
-  <xacro:property name="motor_constant" value="1.269e-05" /> <!-- [kg m/s^2] -->
-  <xacro:property name="moment_constant" value="0.016754" /> <!-- [m] -->
-  <xacro:property name="time_constant_up" value="0.0182" /> <!-- [s] -->
-  <xacro:property name="time_constant_down" value="0.0182" /> <!-- [s] -->
-  <xacro:property name="max_rot_velocity" value="1047.2" /> <!-- [rad/s] -->
-  <xacro:property name="sin30" value="0.5" />
-  <xacro:property name="cos30" value="0.866025403784" />
   <xacro:property name="front_propeller_x" value="0.247" />
   <xacro:property name="front_propeller_y" value="0.1506" />
@@ -28,13 +23,11 @@
   <xacro:property name="back_propeller_x" value="-0.2501" />
   <xacro:property name="back_propeller_y" value="0.1454" />
-  <xacro:property name="rotor_drag_coefficient" value="2.0673e-04" />
-  <xacro:property name="rolling_moment_coefficient" value="0.0" />
   <!-- Property Blocks -->
   <xacro:property name="body_inertia">
-    <inertia ixx="6.08870e-02" ixy="0.0" ixz="0.0" iyy="6.87913e-02" iyz="0.0" izz="1.48916e-01" /> <!-- [kg m^2] [kg m^2] [kg m^2] [kg m^2] [kg m^2] [kg m^2] -->
+    <inertia ixx="6.08870e-02" ixy="0.0" ixz="0.0" iyy="6.87913e-02" iyz="0.0" izz="1.48916e-01" /> <!-- [kg m^2] -->
   </xacro:property>
   <!-- inertia of a single rotor, assuming it is a cuboid. Height=3mm, width=15mm -->
   <xacro:property name="rotor_inertia">
-    <xacro:box_inertia x="${radius_rotor}" y="0.015" z="0.003" mass="${mass_rotor*rotor_velocity_slowdown_sim}" />
+    <xacro:box_inertia x="${radius_rotor}" y="0.015" z="0.003" mass="${mass_rotor}" />
   </xacro:property>
   <!-- Instantiate multirotor_base_macro once -->

File: tobas_description/urdf/neo9.xacro (robot description, xacro)
@@ -3,7 +3,9 @@
   <!-- Included URDF Files -->
   <xacro:include filename="$(find tobas_description)/urdf/components/multirotor_base.xacro" />
+  <!-- Constants -->
+  <xacro:property name="sin30" value="0.5" />
+  <xacro:property name="cos30" value="0.866025403784" />
   <!-- Properties -->
   <xacro:property name="namespace" value="neo9" />
-  <xacro:property name="rotor_velocity_slowdown_sim" value="10" />
   <xacro:property name="use_mesh_file" value="true" />
   <xacro:property name="mesh_file" value="package://tobas_description/meshes/neo9.dae" />
@@ -15,11 +17,4 @@
   <xacro:property name="rotor_offset_top" value="0.028" /> <!-- [m] -->
   <xacro:property name="radius_rotor" value="0.1143" /> <!-- [m] -->
-  <xacro:property name="motor_constant" value="6.8e-06" /> <!-- [kg m/s^2] -->
-  <xacro:property name="moment_constant" value="0.016754" /> <!-- [m] -->
-  <xacro:property name="time_constant_up" value="0.0182" /> <!-- [s] -->
-  <xacro:property name="time_constant_down" value="0.0182" /> <!-- [s] -->
-  <xacro:property name="max_rot_velocity" value="1047.2" /> <!-- [rad/s] -->
-  <xacro:property name="sin30" value="0.5" />
-  <xacro:property name="cos30" value="0.866025403784" />
   <xacro:property name="front_propeller_x" value="0.213" />
   <xacro:property name="front_propeller_y" value="0.12988" />
@@ -28,13 +23,11 @@
   <xacro:property name="back_propeller_x" value="-0.21561" />
   <xacro:property name="back_propeller_y" value="0.12535" />
-  <xacro:property name="rotor_drag_coefficient" value="2.0673e-04" />
-  <xacro:property name="rolling_moment_coefficient" value="0.0" />
   <!-- Property Blocks -->
   <xacro:property name="body_inertia">
-    <inertia ixx="0.0331" ixy="0.0" ixz="0.0" iyy="0.0350" iyz="0.0" izz="0.0605" /> <!-- [kg m^2] [kg m^2] [kg m^2] [kg m^2] [kg m^2] [kg m^2] -->
+    <inertia ixx="0.0331" ixy="0.0" ixz="0.0" iyy="0.0350" iyz="0.0" izz="0.0605" /> <!-- [kg m^2] -->
   </xacro:property>
   <!-- inertia of a single rotor, assuming it is a cuboid. Height=3mm, width=15mm -->
   <xacro:property name="rotor_inertia">
-    <xacro:box_inertia x="${radius_rotor}" y="0.015" z="0.003" mass="${mass_rotor*rotor_velocity_slowdown_sim}" />
+    <xacro:box_inertia x="${radius_rotor}" y="0.015" z="0.003" mass="${mass_rotor}" />
   </xacro:property>
   <!-- Instantiate multirotor_base_macro once -->

File: tobas_description/urdf/pelican.xacro (robot description, xacro)
@@ -5,5 +5,4 @@
   <!-- Properties  -->
   <xacro:property name="namespace" value="pelican" />
-  <xacro:property name="rotor_velocity_slowdown_sim" value="10" />
   <xacro:property name="use_mesh_file" value="true" />
   <xacro:property name="mesh_file" value="package://tobas_description/meshes/pelican.dae" />
@@ -15,18 +14,11 @@
   <xacro:property name="rotor_offset_top" value="0.05" /> <!-- [m] -->
   <xacro:property name="radius_rotor" value="0.128" /> <!-- [m] -->
-  <xacro:property name="motor_constant" value="9.9865e-06" /> <!-- [kg m/s^2] -->
-  <xacro:property name="moment_constant" value="0.016" /> <!-- [m] -->
-  <xacro:property name="time_constant_up" value="0.0125" /> <!-- [s] -->
-  <xacro:property name="time_constant_down" value="0.025" /> <!-- [s] -->
-  <xacro:property name="max_rot_velocity" value="838" /> <!-- [rad/s] -->
-  <xacro:property name="rotor_drag_coefficient" value="8.06428e-05" />
-  <xacro:property name="rolling_moment_coefficient" value="0.000001" />
   <!-- Property Blocks -->
   <xacro:property name="body_inertia">
-    <inertia ixx="0.01" ixy="0.0" ixz="0.0" iyy="0.01" iyz="0.0" izz="0.02" /> <!-- [kg m^2] [kg m^2] [kg m^2] [kg m^2] [kg m^2] [kg m^2] -->
+    <inertia ixx="0.01" ixy="0.0" ixz="0.0" iyy="0.01" iyz="0.0" izz="0.02" /> <!-- [kg m^2] -->
   </xacro:property>
   <!-- inertia of a single rotor, assuming it is a cuboid. Height=3mm, width=15mm -->
   <xacro:property name="rotor_inertia">
-    <xacro:box_inertia x="${radius_rotor}" y="0.015" z="0.003" mass="${mass_rotor*rotor_velocity_slowdown_sim}" />
+    <xacro:box_inertia x="${radius_rotor}" y="0.015" z="0.003" mass="${mass_rotor}" />
   </xacro:property>
   <!-- Instantiate multirotor_base_macro once -->

File: tobas_description/urdf/techpod.xacro (robot description, xacro)
@@ -1,11 +1,10 @@
 <?xml version="1.0"?>
 <robot name="techpod" xmlns:xacro="http://ros.org/wiki/xacro">
-  <!-- Global properties -->
-  <xacro:property name="namespace" value="techpod" />
-  <xacro:property name="rotor_velocity_slowdown_sim" value="10" />
-  <xacro:property name="use_mesh" value="true" />
   <!-- Constants -->
   <xacro:property name="PI" value="3.1415926535897931" />
   <xacro:property name="DEG2RAD" value="${PI / 180.0}" />
+  <!-- Global properties -->
+  <xacro:property name="namespace" value="techpod" />
+  <xacro:property name="use_mesh" value="true" />
   <!-- Component masses -->
   <xacro:property name="mass_fuselage" value="2.05" /> <!-- [kg] -->
@@ -96,5 +95,5 @@
   <!-- Inertia of the propeller, assuming it is a cylinder -->
   <xacro:property name="propeller_inertia">
-    <xacro:cylinder_inertia r="${propeller_radius}" h="${propeller_height}" mass="${mass_propeller * rotor_velocity_slowdown_sim}" />
+    <xacro:cylinder_inertia r="${propeller_radius}" h="${propeller_height}" mass="${mass_propeller}" />
   </xacro:property>
   <!-- Inertia of the wheels, assuming it is a cylinder -->

Commit message: 未使用の定数を削除

File: tobas_description/urdf/ardrone.xacro (robot description, xacro)
@@ -4,6 +4,4 @@
   <xacro:include filename="$(find tobas_description)/urdf/components/multirotor_base.xacro" />
   <!-- Constants -->
-  <xacro:property name="sin30" value="0.5" />
-  <xacro:property name="cos30" value="0.866025403784" />
   <xacro:property name="sqrt2" value="1.4142135623730951" />
   <!-- Properties -->

File: tobas_description/urdf/iris.xacro (robot description, xacro)
@@ -3,8 +3,4 @@
   <!-- Included URDF Files -->
   <xacro:include filename="$(find tobas_description)/urdf/components/multirotor_base.xacro" />
-  <!-- Constants -->
-  <xacro:property name="sin30" value="0.5" />
-  <xacro:property name="cos30" value="0.866025403784" />
-  <xacro:property name="sqrt2" value="1.4142135623730951" />
   <!-- Properties -->
   <xacro:property name="namespace" value="iris" />

File: tobas_description/urdf/neo11.xacro (robot description, xacro)
@@ -3,7 +3,4 @@
   <!-- Included URDF Files -->
   <xacro:include filename="$(find tobas_description)/urdf/components/multirotor_base.xacro" />
-  <!-- Constants -->
-  <xacro:property name="sin30" value="0.5" />
-  <xacro:property name="cos30" value="0.866025403784" />
   <!-- Properties -->
   <xacro:property name="namespace" value="neo11" />

File: tobas_description/urdf/neo9.xacro (robot description, xacro)
@@ -3,7 +3,4 @@
   <!-- Included URDF Files -->
   <xacro:include filename="$(find tobas_description)/urdf/components/multirotor_base.xacro" />
-  <!-- Constants -->
-  <xacro:property name="sin30" value="0.5" />
-  <xacro:property name="cos30" value="0.866025403784" />
   <!-- Properties -->
   <xacro:property name="namespace" value="neo9" />
