Commit message: add DJI F450 model

File: tobas_description/urdf/ardrone.xacro (robot description, xacro)
@@ -3,6 +3,4 @@
   <!-- Included URDF Files -->
   <xacro:include filename="$(find tobas_description)/urdf/components/multirotor_base.xacro" />
-  <!-- Constants -->
-  <xacro:property name="sqrt2" value="1.4142135623730951" />
   <!-- Properties -->
   <xacro:property name="namespace" value="ardrone" />

File: tobas_description/urdf/components/common.xacro (robot description, xacro)
@@ -2,6 +2,12 @@
 <robot xmlns:xacro="http://ros.org/wiki/xacro">
   <!-- Constants -->
+  <xacro:property name="sqrt2" value="1.4142135623730951"/>
+  <xacro:property name="sqrt3" value="1.73205080757"/>
   <xacro:property name="sin30" value="0.5"/>
-  <xacro:property name="cos30" value="0.866025403784"/>
+  <xacro:property name="cos30" value="${sqrt3 / 2}"/>
+  <xacro:property name="sin45" value="${1 / sqrt2}"/>
+  <xacro:property name="cos45" value="${sin45}"/>
+  <xacro:property name="sin60" value="${cos30}"/>
+  <xacro:property name="cos60" value="${sin30}"/>
   <!-- Properties -->
   <xacro:property name="deg2rad" value="${pi / 180}"/>

Commit message: edit *.xacro, *.urdf

File: tobas_description/urdf/ardrone.xacro (robot description, xacro)
@@ -40,9 +40,9 @@
     radius_rotor="${radius_rotor}"
     motor_number="0"
-    color="Red"
     use_own_mesh="false"
     mesh="">
     <origin xyz="${sqrt2 * arm_length} -${sqrt2 * arm_length} ${rotor_offset_top}" rpy="0 0 0"/>
     <xacro:insert_block name="rotor_inertia"/>
+    <xacro:insert_block name="red"/>
   </xacro:vertical_rotor>
   <xacro:vertical_rotor
@@ -53,9 +53,9 @@
     radius_rotor="${radius_rotor}"
     motor_number="1"
-    color="Blue"
     use_own_mesh="false"
     mesh="">
     <origin xyz="-${sqrt2 * arm_length} ${sqrt2 * arm_length} ${rotor_offset_top}" rpy="0 0 0"/>
     <xacro:insert_block name="rotor_inertia"/>
+    <xacro:insert_block name="red"/>
   </xacro:vertical_rotor>
   <xacro:vertical_rotor
@@ -66,9 +66,9 @@
     radius_rotor="${radius_rotor}"
     motor_number="2"
-    color="Red"
     use_own_mesh="false"
     mesh="">
     <origin xyz="${sqrt2 * arm_length} ${sqrt2 * arm_length} ${rotor_offset_top}" rpy="0 0 0"/>
     <xacro:insert_block name="rotor_inertia"/>
+    <xacro:insert_block name="blue"/>
   </xacro:vertical_rotor>
   <xacro:vertical_rotor
@@ -79,9 +79,9 @@
     radius_rotor="${radius_rotor}"
     motor_number="3"
-    color="Blue"
     use_own_mesh="false"
     mesh="">
     <origin xyz="-${sqrt2 * arm_length} -${sqrt2 * arm_length} ${rotor_offset_top}" rpy="0 0 0"/>
     <xacro:insert_block name="rotor_inertia"/>
+    <xacro:insert_block name="blue"/>
   </xacro:vertical_rotor>
 </robot>

File: tobas_description/urdf/components/common.xacro (robot description, xacro)
@@ -59,5 +59,5 @@
       <origin xyz="${x0} ${y0} ${z0}" rpy="0 0 0"/>
       <geometry>
-        <box size="${sqrt3*side} ${side} ${height}"/>
+        <box size="${sqrt3 * side} ${side} ${height}"/>
       </geometry>
     </collision>
@@ -65,5 +65,5 @@
       <origin xyz="${x0} ${y0} ${z0}" rpy="0 0 ${60*deg2rad}"/>
       <geometry>
-        <box size="${sqrt3*side} ${side} ${height}"/>
+        <box size="${sqrt3 * side} ${side} ${height}"/>
       </geometry>
     </collision>
@@ -71,5 +71,5 @@
       <origin xyz="${x0} ${y0} ${z0}" rpy="0 0 ${-60*deg2rad}"/>
       <geometry>
-        <box size="${sqrt3*side} ${side} ${height}"/>
+        <box size="${sqrt3 * side} ${side} ${height}"/>
       </geometry>
     </collision>

File: tobas_description/urdf/components/harrier/multirotor_base_harrier.xacro (robot description, xacro)
@@ -73,7 +73,4 @@
       </collision>
     </link>
-    <gazebo reference="${robot_namespace}/rotor_${motor_number}">
-      <material>Gazebo/Black</material>
-    </gazebo>
   </xacro:macro>
 </robot>

File: tobas_description/urdf/components/multirotor_base.xacro (robot description, xacro)
@@ -50,9 +50,9 @@
       radius_rotor
       motor_number
-      color
       use_own_mesh
       mesh
       *origin
-      *inertia">
+      *inertia
+      *material">
     <joint name="${robot_namespace}/rotor_${motor_number}_joint" type="continuous">
       <xacro:insert_block name="origin"/>
@@ -75,4 +75,5 @@
           </xacro:unless>
         </geometry>
+        <xacro:insert_block name="material"/>
       </visual>
       <collision>
@@ -82,7 +83,4 @@
       </collision>
     </link>
-    <gazebo reference="${robot_namespace}/rotor_${motor_number}">
-      <material>Gazebo/${color}</material>
-    </gazebo>
   </xacro:macro>
   <!-- Virtual frame for visualization -->
@@ -102,7 +100,5 @@
           <box size="1e-3 1e-3 1e-3"/>
         </geometry>
-        <material name="Red">
-          <color rgba="1.0 0.0 0.0 1.0"/>
-        </material>
+        <xacro:insert_block name="red"/>
       </visual>
       <collision>

File: tobas_description/urdf/firefly.xacro (robot description, xacro)
@@ -40,9 +40,9 @@
     radius_rotor="${radius_rotor}"
     motor_number="0"
-    color="Red"
     use_own_mesh="false"
     mesh="">
     <origin xyz="${cos30*arm_length} ${sin30*arm_length} ${rotor_offset_top}" rpy="0 0 0"/>
     <xacro:insert_block name="rotor_inertia"/>
+    <xacro:insert_block name="red"/>
   </xacro:vertical_rotor>
   <xacro:vertical_rotor
@@ -53,9 +53,9 @@
     radius_rotor="${radius_rotor}"
     motor_number="1"
-    color="Blue"
     use_own_mesh="false"
     mesh="">
     <origin xyz="0 ${arm_length} ${rotor_offset_top}" rpy="0 0 0"/>
     <xacro:insert_block name="rotor_inertia"/>
+    <xacro:insert_block name="blue"/>
   </xacro:vertical_rotor>
   <xacro:vertical_rotor
@@ -66,9 +66,9 @@
     radius_rotor="${radius_rotor}"
     motor_number="2"
-    color="Blue"
     use_own_mesh="false"
     mesh="">
     <origin xyz="-${cos30*arm_length} ${sin30*arm_length} ${rotor_offset_top}" rpy="0 0 0"/>
     <xacro:insert_block name="rotor_inertia"/>
+    <xacro:insert_block name="red"/>
   </xacro:vertical_rotor>
   <xacro:vertical_rotor
@@ -79,9 +79,9 @@
     radius_rotor="${radius_rotor}"
     motor_number="3"
-    color="Blue"
     use_own_mesh="false"
     mesh="">
     <origin xyz="-${cos30*arm_length} -${sin30*arm_length} ${rotor_offset_top}" rpy="0 0 0"/>
     <xacro:insert_block name="rotor_inertia"/>
+    <xacro:insert_block name="blue"/>
   </xacro:vertical_rotor>
   <xacro:vertical_rotor
@@ -92,9 +92,9 @@
     radius_rotor="${radius_rotor}"
     motor_number="4"
-    color="Blue"
     use_own_mesh="false"
     mesh="">
     <origin xyz="0 -${arm_length} ${rotor_offset_top}" rpy="0 0 0"/>
     <xacro:insert_block name="rotor_inertia"/>
+    <xacro:insert_block name="red"/>
   </xacro:vertical_rotor>
   <xacro:vertical_rotor
@@ -105,9 +105,9 @@
     radius_rotor="${radius_rotor}"
     motor_number="5"
-    color="Red"
     use_own_mesh="false"
     mesh="">
     <origin xyz="${cos30*arm_length} -${sin30*arm_length} ${rotor_offset_top}" rpy="0 0 0"/>
     <xacro:insert_block name="rotor_inertia"/>
+    <xacro:insert_block name="blue"/>
   </xacro:vertical_rotor>
 </robot>

File: tobas_description/urdf/hummingbird.xacro (robot description, xacro)
@@ -40,9 +40,9 @@
     radius_rotor="${radius_rotor}"
     motor_number="0"
-    color="Red"
     use_own_mesh="false"
     mesh="">
     <origin xyz="${arm_length} 0 ${rotor_offset_top}" rpy="0 0 0"/>
     <xacro:insert_block name="rotor_inertia"/>
+    <xacro:insert_block name="blue"/>
   </xacro:vertical_rotor>
   <xacro:vertical_rotor
@@ -53,9 +53,9 @@
     radius_rotor="${radius_rotor}"
     motor_number="1"
-    color="Blue"
     use_own_mesh="false"
     mesh="">
     <origin xyz="0 ${arm_length} ${rotor_offset_top}" rpy="0 0 0"/>
     <xacro:insert_block name="rotor_inertia"/>
+    <xacro:insert_block name="red"/>
   </xacro:vertical_rotor>
   <xacro:vertical_rotor
@@ -66,9 +66,9 @@
     radius_rotor="${radius_rotor}"
     motor_number="2"
-    color="Blue"
     use_own_mesh="false"
     mesh="">
     <origin xyz="-${arm_length} 0 ${rotor_offset_top}" rpy="0 0 0"/>
     <xacro:insert_block name="rotor_inertia"/>
+    <xacro:insert_block name="blue"/>
   </xacro:vertical_rotor>
   <xacro:vertical_rotor
@@ -79,9 +79,9 @@
     radius_rotor="${radius_rotor}"
     motor_number="3"
-    color="Blue"
     use_own_mesh="false"
     mesh="">
     <origin xyz="0 -${arm_length} ${rotor_offset_top}" rpy="0 0 0"/>
     <xacro:insert_block name="rotor_inertia"/>
+    <xacro:insert_block name="red"/>
   </xacro:vertical_rotor>
 </robot>

File: tobas_description/urdf/iris.xacro (robot description, xacro)
@@ -43,9 +43,9 @@
     radius_rotor="${radius_rotor}"
     motor_number="0"
-    color="Blue"
     use_own_mesh="false"
     mesh="">
     <origin xyz="${arm_length_front_x} -${arm_length_front_y} ${rotor_offset_top}" rpy="0 0 0"/>
     <xacro:insert_block name="rotor_inertia"/>
+    <xacro:insert_block name="red"/>
   </xacro:vertical_rotor>
   <xacro:vertical_rotor
@@ -56,9 +56,9 @@
     radius_rotor="${radius_rotor}"
     motor_number="1"
-    color="Red"
     use_own_mesh="false"
     mesh="">
     <origin xyz="-${arm_length_back_x} ${arm_length_back_y} ${rotor_offset_top}" rpy="0 0 0"/>
     <xacro:insert_block name="rotor_inertia"/>
+    <xacro:insert_block name="red"/>
   </xacro:vertical_rotor>
   <xacro:vertical_rotor
@@ -69,9 +69,9 @@
     radius_rotor="${radius_rotor}"
     motor_number="2"
-    color="Blue"
     use_own_mesh="false"
     mesh="">
     <origin xyz="${arm_length_front_x} ${arm_length_front_y} ${rotor_offset_top}" rpy="0 0 0"/>
     <xacro:insert_block name="rotor_inertia"/>
+    <xacro:insert_block name="blue"/>
   </xacro:vertical_rotor>
   <xacro:vertical_rotor
@@ -82,9 +82,9 @@
     radius_rotor="${radius_rotor}"
     motor_number="3"
-    color="Red"
     use_own_mesh="false"
     mesh="">
     <origin xyz="-${arm_length_back_x} -${arm_length_back_y} ${rotor_offset_top}" rpy="0 0 0"/>
     <xacro:insert_block name="rotor_inertia"/>
+    <xacro:insert_block name="blue"/>
   </xacro:vertical_rotor>
 </robot>

File: tobas_description/urdf/neo11.xacro (robot description, xacro)
@@ -46,9 +46,9 @@
     radius_rotor="${radius_rotor}"
     motor_number="0"
-    color="Red"
     use_own_mesh="true"
     mesh="package://tobas_description/meshes/neo11_propeller_ccw.dae">
     <origin xyz="${front_propeller_x} ${front_propeller_y} ${rotor_offset_top}" rpy="${5*pi/180} 0 ${30*pi/180}"/>
     <xacro:insert_block name="rotor_inertia"/>
+    <xacro:insert_block name="red"/>
   </xacro:vertical_rotor>
   <xacro:vertical_rotor
@@ -59,9 +59,9 @@
     radius_rotor="${radius_rotor}"
     motor_number="1"
-    color="Blue"
     use_own_mesh="true"
     mesh="package://tobas_description/meshes/neo11_propeller_cw.dae">
     <origin xyz="${side_propeller_x} ${side_propeller_y} ${rotor_offset_top}" rpy="0 ${-5*pi/180} 0"/>
     <xacro:insert_block name="rotor_inertia"/>
+    <xacro:insert_block name="blue"/>
   </xacro:vertical_rotor>
   <xacro:vertical_rotor
@@ -72,9 +72,9 @@
     radius_rotor="${radius_rotor}"
     motor_number="2"
-    color="Blue"
     use_own_mesh="true"
     mesh="package://tobas_description/meshes/neo11_propeller_ccw.dae">
     <origin xyz="${back_propeller_x} ${back_propeller_y} ${rotor_offset_top}" rpy="${5*pi/180} 0 ${150*pi/180}"/>
     <xacro:insert_block name="rotor_inertia"/>
+    <xacro:insert_block name="red"/>
   </xacro:vertical_rotor>
   <xacro:vertical_rotor
@@ -85,9 +85,9 @@
     radius_rotor="${radius_rotor}"
     motor_number="3"
-    color="Blue"
     use_own_mesh="true"
     mesh="package://tobas_description/meshes/neo11_propeller_cw.dae">
     <origin xyz="${back_propeller_x} -${back_propeller_y} ${rotor_offset_top}" rpy="${-5*pi/180} 0 ${-150*pi/180}"/>
     <xacro:insert_block name="rotor_inertia"/>
+    <xacro:insert_block name="blue"/>
   </xacro:vertical_rotor>
   <xacro:vertical_rotor
@@ -98,9 +98,9 @@
     radius_rotor="${radius_rotor}"
     motor_number="4"
-    color="Blue"
     use_own_mesh="true"
     mesh="package://tobas_description/meshes/neo11_propeller_ccw.dae">
     <origin xyz="${side_propeller_x} -${side_propeller_y} ${rotor_offset_top}" rpy="0 ${5*pi/180} ${pi}"/>
     <xacro:insert_block name="rotor_inertia"/>
+    <xacro:insert_block name="red"/>
   </xacro:vertical_rotor>
   <xacro:vertical_rotor
@@ -111,9 +111,9 @@
     radius_rotor="${radius_rotor}"
     motor_number="5"
-    color="Red"
     use_own_mesh="true"
     mesh="package://tobas_description/meshes/neo11_propeller_cw.dae">
     <origin xyz="${front_propeller_x} -${front_propeller_y} ${rotor_offset_top}" rpy="${-5*pi/180} 0 ${-30*pi/180}"/>
     <xacro:insert_block name="rotor_inertia"/>
+    <xacro:insert_block name="blue"/>
   </xacro:vertical_rotor>
 </robot>

File: tobas_description/urdf/neo9.xacro (robot description, xacro)
@@ -46,9 +46,9 @@
     radius_rotor="${radius_rotor}"
     motor_number="0"
-    color="Red"
     use_own_mesh="true"
     mesh="package://tobas_description/meshes/neo9_propeller_ccw.dae">
     <origin xyz="${front_propeller_x} ${front_propeller_y} ${rotor_offset_top}" rpy="${5*pi/180} 0 ${30*pi/180}"/>
     <xacro:insert_block name="rotor_inertia"/>
+    <xacro:insert_block name="red"/>
   </xacro:vertical_rotor>
   <xacro:vertical_rotor
@@ -59,9 +59,9 @@
     radius_rotor="${radius_rotor}"
     motor_number="1"
-    color="Blue"
     use_own_mesh="true"
     mesh="package://tobas_description/meshes/neo9_propeller_cw.dae">
     <origin xyz="${side_propeller_x} ${side_propeller_y} ${rotor_offset_top}" rpy="0 ${-5*pi/180} 0"/>
     <xacro:insert_block name="rotor_inertia"/>
+    <xacro:insert_block name="blue"/>
   </xacro:vertical_rotor>
   <xacro:vertical_rotor
@@ -72,9 +72,9 @@
     radius_rotor="${radius_rotor}"
     motor_number="2"
-    color="Blue"
     use_own_mesh="true"
     mesh="package://tobas_description/meshes/neo9_propeller_ccw.dae">
     <origin xyz="${back_propeller_x} ${back_propeller_y} ${rotor_offset_top}" rpy="${5*pi/180} 0 ${150*pi/180}"/>
     <xacro:insert_block name="rotor_inertia"/>
+    <xacro:insert_block name="red"/>
   </xacro:vertical_rotor>
   <xacro:vertical_rotor
@@ -85,9 +85,9 @@
     radius_rotor="${radius_rotor}"
     motor_number="3"
-    color="Blue"
     use_own_mesh="true"
     mesh="package://tobas_description/meshes/neo9_propeller_cw.dae">
     <origin xyz="${back_propeller_x} -${back_propeller_y} ${rotor_offset_top}" rpy="${-5*pi/180} 0 ${-150*pi/180}"/>
     <xacro:insert_block name="rotor_inertia"/>
+    <xacro:insert_block name="blue"/>
   </xacro:vertical_rotor>
   <xacro:vertical_rotor
@@ -103,4 +103,5 @@
     <origin xyz="${side_propeller_x} -${side_propeller_y} ${rotor_offset_top}" rpy="0 ${5*pi/180} ${pi}"/>
     <xacro:insert_block name="rotor_inertia"/>
+    <xacro:insert_block name="red"/>
   </xacro:vertical_rotor>
   <xacro:vertical_rotor
@@ -116,4 +117,5 @@
     <origin xyz="${front_propeller_x} -${front_propeller_y} ${rotor_offset_top}" rpy="${-5*pi/180} 0 ${-30*pi/180}"/>
     <xacro:insert_block name="rotor_inertia"/>
+    <xacro:insert_block name="blue"/>
   </xacro:vertical_rotor>
 </robot>

File: tobas_description/urdf/pelican.xacro (robot description, xacro)
@@ -45,4 +45,5 @@
     <origin xyz="${arm_length} 0 ${rotor_offset_top}" rpy="0 0 0"/>
     <xacro:insert_block name="rotor_inertia"/>
+    <xacro:insert_block name="blue"/>
   </xacro:vertical_rotor>
   <xacro:vertical_rotor
@@ -58,4 +59,5 @@
     <origin xyz="0 ${arm_length} ${rotor_offset_top}" rpy="0 0 0"/>
     <xacro:insert_block name="rotor_inertia"/>
+    <xacro:insert_block name="red"/>
   </xacro:vertical_rotor>
   <xacro:vertical_rotor
@@ -71,4 +73,5 @@
     <origin xyz="-${arm_length} 0 ${rotor_offset_top}" rpy="0 0 0"/>
     <xacro:insert_block name="rotor_inertia"/>
+    <xacro:insert_block name="blue"/>
   </xacro:vertical_rotor>
   <xacro:vertical_rotor
@@ -84,4 +87,5 @@
     <origin xyz="0 -${arm_length} ${rotor_offset_top}" rpy="0 0 0"/>
     <xacro:insert_block name="rotor_inertia"/>
+    <xacro:insert_block name="red"/>
   </xacro:vertical_rotor>
 </robot>
