Commit message: fix: truncated_octahedron.xacro

File: tobas_description/urdf/truncated_octahedron.xacro (robot description, xacro)
@@ -11,4 +11,6 @@
   <xacro:property name="motor_offset" value="0.1705"/>
   <xacro:property name="x" value="${motor_offset/sqrt3}"/>
+  <!-- FIXME: 全ての辺の長さが等しい切頂八面体の6角形部分にプロペラを合わせた場合ピッチ角は45degのはずだが，モデリングの都合上少しずれている． -->
+  <xacro:property name="prop_pitch" value="0.95"/>
   <!-- Base Link -->
   <link name="base_link"/>
@@ -49,26 +51,26 @@
   <!-- Propulsion System -->
   <xacro:dji_a2212_0945 parent="base_link" index="0" direction="ccw">
-    <origin xyz="${x} ${x} ${x}" rpy="0 ${pi/4} ${pi/4*1}"/>
+    <origin xyz="${x} ${x} ${x}" rpy="0 ${prop_pitch} ${pi/4*1}"/>
   </xacro:dji_a2212_0945>
   <xacro:dji_a2212_0945 parent="base_link" index="1" direction="cw">
-    <origin xyz="${-x} ${x} ${x}" rpy="0 ${pi/4} ${pi/4*3}"/>
+    <origin xyz="${-x} ${x} ${x}" rpy="0 ${prop_pitch} ${pi/4*3}"/>
   </xacro:dji_a2212_0945>
   <xacro:dji_a2212_0945 parent="base_link" index="2" direction="ccw">
-    <origin xyz="${-x} ${-x} ${x}" rpy="0 ${pi/4} ${pi/4*5}"/>
+    <origin xyz="${-x} ${-x} ${x}" rpy="0 ${prop_pitch} ${pi/4*5}"/>
   </xacro:dji_a2212_0945>
   <xacro:dji_a2212_0945 parent="base_link" index="3" direction="cw">
-    <origin xyz="${x} ${-x} ${x}" rpy="0 ${pi/4} ${pi/4*7}"/>
+    <origin xyz="${x} ${-x} ${x}" rpy="0 ${prop_pitch} ${pi/4*7}"/>
   </xacro:dji_a2212_0945>
   <xacro:dji_a2212_0945 parent="base_link" index="4" direction="cw">
-    <origin xyz="${x} ${x} ${-x}" rpy="0 ${pi/4*3} ${pi/4*1}"/>
+    <origin xyz="${x} ${x} ${-x}" rpy="0 ${pi-prop_pitch} ${pi/4*1}"/>
   </xacro:dji_a2212_0945>
   <xacro:dji_a2212_0945 parent="base_link" index="5" direction="ccw">
-    <origin xyz="${-x} ${x} ${-x}" rpy="0 ${pi/4*3} ${pi/4*3}"/>
+    <origin xyz="${-x} ${x} ${-x}" rpy="0 ${pi-prop_pitch} ${pi/4*3}"/>
   </xacro:dji_a2212_0945>
   <xacro:dji_a2212_0945 parent="base_link" index="6" direction="cw">
-    <origin xyz="${-x} ${-x} ${-x}" rpy="0 ${pi/4*3} ${pi/4*5}"/>
+    <origin xyz="${-x} ${-x} ${-x}" rpy="0 ${pi-prop_pitch} ${pi/4*5}"/>
   </xacro:dji_a2212_0945>
   <xacro:dji_a2212_0945 parent="base_link" index="7" direction="ccw">
-    <origin xyz="${x} ${-x} ${-x}" rpy="0 ${pi/4*3} ${pi/4*7}"/>
+    <origin xyz="${x} ${-x} ${-x}" rpy="0 ${pi-prop_pitch} ${pi/4*7}"/>
   </xacro:dji_a2212_0945>
 </robot>

Commit message: バッテリーを軽量化

File: tobas_description/urdf/truncated_octahedron.xacro (robot description, xacro)
@@ -3,5 +3,5 @@
   <xacro:include filename="$(find tobas_description)/urdf/components/multirotor_base.xacro"/>
   <xacro:include filename="$(find tobas_description)/urdf/components/fmu/tobas_t1.xacro"/>
-  <xacro:include filename="$(find tobas_description)/urdf/components/battery/hrb_6s_5000mah_50c.xacro"/>
+  <xacro:include filename="$(find tobas_description)/urdf/components/battery/sigp_6s_1100mah_120c.xacro"/>
   <xacro:include filename="$(find tobas_description)/urdf/components/combo/mt3508_0945.xacro"/>
   <!-- Properties -->
@@ -41,10 +41,10 @@
   <!-- Flight Controller -->
   <xacro:tobas_t1 parent="base_link">
-    <origin xyz="0 0 0.0617" rpy="0 0 0"/>
+    <origin xyz="0 0 0.0425" rpy="0 0 0"/>
   </xacro:tobas_t1>
   <!-- Battery -->
-  <xacro:hrb_6s_5000mah_50c parent="base_link">
-    <origin xyz="0 0 -0.0635" rpy="0 0 0"/>
-  </xacro:hrb_6s_5000mah_50c>
+  <xacro:sigp_6s_1100mah_120c parent="base_link">
+    <origin xyz="0 0 -0.060" rpy="${pi/2} 0 0"/>
+  </xacro:sigp_6s_1100mah_120c>
   <!-- Propulsion System -->
   <xacro:mt3508_0945 parent="base_link" index="0" direction="ccw">

File: tobas_example_packages/tobas_truncated_octahedron.TBS/backup/original.urdf (robot description, URDF)
Before this commit: robot truncated_octahedron, 20 links, 19 joints
Links:
- link battery: mass 0.725 -> 0.205; geometry collision box size=0.077 0.035 0.042; visual box size=0.077 0.035 0.042
Joints:
- joint battery_joint: origin xyz=0 0 -0.0635 rpy=0 -0 0 -> xyz=0 0 -0.06 rpy=1.5708 -0 0
- joint fmu_joint: origin xyz=0 0 0.0617 rpy=0 -0 0 -> xyz=0 0 0.0425 rpy=0 -0 0

File: tobas_example_packages/tobas_truncated_octahedron.TBS/tobas_truncated_octahedron_config/urdf/drone.xacro (robot description, xacro)
@@ -3,4 +3,8 @@
         <texture/>
         <color rgba="0 0 0 1"/>
+    </material>
+    <material name="blue">
+        <texture/>
+        <color rgba="0 0 1 1"/>
     </material>
     <material name="orange">
@@ -16,29 +20,25 @@
         <color rgba="1 1 1 1"/>
     </material>
-    <material name="yellow">
-        <texture/>
-        <color rgba="1 1 0 1"/>
-    </material>
     <link name="base_link"/>
     <link name="battery">
         <inertial>
-            <mass value="0.725"/>
-            <origin xyz="0 0 0" rpy="0 -0 0"/>
-            <inertia ixx="0.0002784" ixy="0" ixz="0" iyy="0.00159071" iyz="0" izz="0.00159071"/>
-        </inertial>
-        <visual>
-            <origin xyz="0 0 0" rpy="0 -0 0"/>
-            <geometry>
-                <box size="0.155 0.048 0.048"/>
-            </geometry>
-            <material name="yellow">
-                <texture/>
-                <color rgba="1 1 0 1"/>
-            </material>
-        </visual>
-        <collision>
-            <origin xyz="0 0 0" rpy="0 -0 0"/>
-            <geometry>
-                <box size="0.155 0.048 0.048"/>
+            <mass value="0.205"/>
+            <origin xyz="0 0 0" rpy="0 -0 0"/>
+            <inertia ixx="5.10621e-05" ixy="0" ixz="0" iyy="0.000131422" iyz="0" izz="0.000122214"/>
+        </inertial>
+        <visual>
+            <origin xyz="0 0 0" rpy="0 -0 0"/>
+            <geometry>
+                <box size="0.077 0.035 0.042"/>
+            </geometry>
+            <material name="blue">
+                <texture/>
+                <color rgba="0 0 1 1"/>
+            </material>
+        </visual>
+        <collision>
+            <origin xyz="0 0 0" rpy="0 -0 0"/>
+            <geometry>
+                <box size="0.077 0.035 0.042"/>
             </geometry>
         </collision>
@@ -47,5 +47,5 @@
         <inertial>
             <mass value="0.2"/>
-            <origin xyz="0 0 0.009" rpy="0 -0 0"/>
+            <origin xyz="0 0 0.014" rpy="0 -0 0"/>
             <inertia ixx="7.71333e-05" ixy="0" ixz="0" iyy="0.000148067" iyz="0" izz="0.000199067"/>
         </inertial>
@@ -61,5 +61,5 @@
         </visual>
         <collision>
-            <origin xyz="0 0 0.009" rpy="0 -0 0"/>
+            <origin xyz="0 0 0.014" rpy="0 -0 0"/>
             <geometry>
                 <box size="0.09 0.062 0.028"/>
@@ -459,5 +459,5 @@
     </link>
     <joint name="battery_joint" type="fixed">
-        <origin xyz="0 0 -0.0635" rpy="0 -0 0"/>
+        <origin xyz="0 0 -0.06" rpy="1.5708 -0 0"/>
         <axis xyz="0 0 0"/>
         <parent link="base_link"/>
@@ -465,5 +465,5 @@
     </joint>
     <joint name="fmu_joint" type="fixed">
-        <origin xyz="0 0 0.0617" rpy="0 -0 0"/>
+        <origin xyz="0 0 0.0425" rpy="0 -0 0"/>
         <axis xyz="0 0 0"/>
         <parent link="base_link"/>
@@ -644,6 +644,6 @@
             <maxVoltage>25.200000000000003</maxVoltage>
             <sagVoltage>20.399999999999999</sagVoltage>
-            <maxCurrent>250</maxCurrent>
-            <currentCapacity>18000</currentCapacity>
+            <maxCurrent>132</maxCurrent>
+            <currentCapacity>3960</currentCapacity>
             <internalRegistance>0.018000000000000002</internalRegistance>
             <rotorLinkNames>
