Commit message: edit: f450.xacro

File: tobas_description/urdf/f450.xacro (robot description, xacro)
@@ -8,9 +8,9 @@
   <xacro:property name="battery_y" value="0.035"/>
   <xacro:property name="battery_z" value="0.026"/>
-  <xacro:property name="battery_mass" value="0.18"/>
+  <xacro:property name="battery_mass" value="0.186"/>
   <xacro:property name="propeller_offset" value="0.225"/>
   <xacro:property name="propeller_radius" value="0.125"/>
   <xacro:property name="propeller_height" value="0.009"/>
-  <xacro:property name="propeller_mass" value="0.01"/>
+  <xacro:property name="propeller_mass" value="0.012"/>
   <!-- Base Link -->
   <link name="base_link"/>
@@ -30,5 +30,5 @@
     </visual>
     <inertial>
-      <mass value="0.83"/>
+      <mass value="0.780"/>
       <origin xyz="0.001573 -0.000596 -0.003436" rpy="0 0 0"/>
       <inertia ixx="9.613e-3" ixy="-6.070442e-6" ixz="-4.7933683e-5" iyy="9.702e-3" iyz="-3.987551e-6" izz="1.867e-2"/>

Commit message: edit: f450.xacro

File: tobas_description/urdf/f450.xacro (robot description, xacro)
@@ -5,4 +5,6 @@
   <xacro:include filename="$(find tobas_description)/urdf/components/multirotor_base.xacro"/>
   <!-- Properties0 -->
+  <xacro:property name="frame_width" value="0.35"/>
+  <xacro:property name="frame_height" value="0.06"/>
   <xacro:property name="battery_x" value="0.106"/>
   <xacro:property name="battery_y" value="0.035"/>
@@ -35,7 +37,7 @@
     </inertial>
     <collision>
-      <origin xyz="0 0 0" rpy="0 0 0"/>
+      <origin xyz="0 0 ${-frame_height/2}" rpy="0 0 0"/>
       <geometry>
-        <mesh filename="package://tobas_description/meshes/f450/frame.stl" scale="1e-3 1e-3 1e-3"/>
+        <box size="${frame_width} ${frame_width} ${frame_height}"/>
       </geometry>
     </collision>

Commit message: メッシュのパスを変更

File: tobas_description/urdf/f450.xacro (robot description, xacro)
@@ -29,5 +29,5 @@
         <mesh filename="package://tobas_description/meshes/f450/frame.stl" scale="1e-3 1e-3 1e-3"/>
       </geometry>
-      <xacro:insert_block name="white"/>
+      <xacro:insert_block name="black"/>
     </visual>
     <inertial>
@@ -52,5 +52,5 @@
     <visual>
       <geometry>
-        <mesh filename="package://tobas_description/meshes/f450/sigp_3s_30c.stl" scale="1e-3 1e-3 1e-3"/>
+        <mesh filename="package://tobas_description/meshes/common/battery/sigp_3s_30c.stl" scale="1e-3 1e-3 1e-3"/>
       </geometry>
       <xacro:insert_block name="blue"/>
@@ -69,5 +69,5 @@
   </link>
   <!-- Propellers -->
-  <xacro:macro name="propeller" params="index yaw_deg origin_x origin_y">
+  <xacro:macro name="propeller" params="index direction yaw_deg origin_x origin_y">
     <joint name="propeller_${index}_joint" type="continuous">
       <origin xyz="${origin_x} ${origin_y} 0.0247" rpy="0 0 ${yaw_deg*deg2rad}"/>
@@ -79,7 +79,7 @@
       <visual>
         <geometry>
-          <mesh filename="package://tobas_description/meshes/f450/propeller.stl" scale="1e-3 1e-3 1e-3"/>
+          <mesh filename="package://tobas_description/meshes/common/propeller/phantom3_0945_${direction}.stl" scale="1e-3 1e-3 1e-3"/>
         </geometry>
-        <xacro:insert_block name="black"/>
+        <xacro:insert_block name="white"/>
       </visual>
       <inertial>
@@ -96,7 +96,7 @@
     </link>
   </xacro:macro>
-  <xacro:propeller index="0" yaw_deg="-45" origin_x="${propeller_offset*cos45}" origin_y="${-propeller_offset*cos45}"/>
-  <xacro:propeller index="1" yaw_deg="135" origin_x="${-propeller_offset*cos45}" origin_y="${propeller_offset*cos45}"/>
-  <xacro:propeller index="2" yaw_deg="45" origin_x="${propeller_offset*cos45}" origin_y="${propeller_offset*cos45}"/>
-  <xacro:propeller index="3" yaw_deg="225" origin_x="${-propeller_offset*cos45}" origin_y="${-propeller_offset*cos45}"/>
+  <xacro:propeller index="0" direction="ccw" yaw_deg="-45" origin_x="${propeller_offset*cos45}" origin_y="${-propeller_offset*cos45}"/>
+  <xacro:propeller index="1" direction="ccw" yaw_deg="135" origin_x="${-propeller_offset*cos45}" origin_y="${propeller_offset*cos45}"/>
+  <xacro:propeller index="2" direction="cw" yaw_deg="45" origin_x="${propeller_offset*cos45}" origin_y="${propeller_offset*cos45}"/>
+  <xacro:propeller index="3" direction="cw" yaw_deg="225" origin_x="${-propeller_offset*cos45}" origin_y="${-propeller_offset*cos45}"/>
 </robot>

File: tobas_description/urdf/f550_np.xacro (robot description, xacro)
@@ -78,5 +78,5 @@
       <visual>
         <geometry>
-          <mesh filename="package://tobas_description/meshes/f550_np/phantom3_0945_${direction}.stl" scale="1e-3 1e-3 1e-3"/>
+          <mesh filename="package://tobas_description/meshes/common/propeller/phantom3_0945_${direction}.stl" scale="1e-3 1e-3 1e-3"/>
         </geometry>
         <xacro:insert_block name="white"/>

File: tobas_description/urdf/f550_np_rmx52.xacro (robot description, xacro)
@@ -115,5 +115,5 @@
       <visual>
         <geometry>
-          <mesh filename="package://tobas_description/meshes/f550_np/phantom3_0945_${direction}.stl" scale="1e-3 1e-3 1e-3"/>
+          <mesh filename="package://tobas_description/meshes/common/propeller/phantom3_0945_${direction}.stl" scale="1e-3 1e-3 1e-3"/>
         </geometry>
         <xacro:insert_block name="white"/>

Commit message: edit: f450.xacro

File: tobas_description/urdf/f450.xacro (robot description, xacro)
@@ -7,12 +7,14 @@
   <xacro:property name="frame_width" value="0.35"/>
   <xacro:property name="frame_height" value="0.06"/>
+  <xacro:property name="frame_mass" value="0.780"/>
   <xacro:property name="battery_x" value="0.106"/>
   <xacro:property name="battery_y" value="0.035"/>
   <xacro:property name="battery_z" value="0.026"/>
   <xacro:property name="battery_mass" value="0.186"/>
+  <xacro:property name="propeller_diameter" value="${9*inch2meter}"/>
+  <xacro:property name="propeller_radius" value="${propeller_diameter/2}"/>
   <xacro:property name="propeller_offset" value="0.225"/>
-  <xacro:property name="propeller_radius" value="0.125"/>
-  <xacro:property name="propeller_height" value="0.009"/>
-  <xacro:property name="propeller_mass" value="0.012"/>
+  <xacro:property name="propeller_height" value="0.01"/>
+  <xacro:property name="propeller_mass" value="0.011"/>
   <!-- Base Link -->
   <link name="base_link"/>
@@ -32,5 +34,5 @@
     </visual>
     <inertial>
-      <mass value="0.780"/>
+      <mass value="${frame_mass}"/>
       <origin xyz="0.001573 -0.000596 -0.003436" rpy="0 0 0"/>
       <inertia ixx="9.613e-3" ixy="-6.070442e-6" ixz="-4.7933683e-5" iyy="9.702e-3" iyz="-3.987551e-6" izz="1.867e-2"/>
@@ -69,7 +71,7 @@
   </link>
   <!-- Propellers -->
-  <xacro:macro name="propeller" params="index direction yaw_deg origin_x origin_y">
+  <xacro:macro name="propeller" params="index direction yaw_deg">
     <joint name="propeller_${index}_joint" type="continuous">
-      <origin xyz="${origin_x} ${origin_y} 0.0247" rpy="0 0 ${yaw_deg*deg2rad}"/>
+      <origin xyz="${propeller_offset*cos(yaw_deg*deg2rad)} ${propeller_offset*sin(yaw_deg*deg2rad)} 0.0247" rpy="0 0 ${yaw_deg*deg2rad}"/>
       <axis xyz="0 0 1"/>
       <parent link="base_link"/>
@@ -96,7 +98,7 @@
     </link>
   </xacro:macro>
-  <xacro:propeller index="0" direction="ccw" yaw_deg="-45" origin_x="${propeller_offset*cos45}" origin_y="${-propeller_offset*cos45}"/>
-  <xacro:propeller index="1" direction="ccw" yaw_deg="135" origin_x="${-propeller_offset*cos45}" origin_y="${propeller_offset*cos45}"/>
-  <xacro:propeller index="2" direction="cw" yaw_deg="45" origin_x="${propeller_offset*cos45}" origin_y="${propeller_offset*cos45}"/>
-  <xacro:propeller index="3" direction="cw" yaw_deg="225" origin_x="${-propeller_offset*cos45}" origin_y="${-propeller_offset*cos45}"/>
+  <xacro:propeller index="0" direction="ccw" yaw_deg="-45"/>
+  <xacro:propeller index="1" direction="ccw" yaw_deg="135"/>
+  <xacro:propeller index="2" direction="cw" yaw_deg="45"/>
+  <xacro:propeller index="3" direction="cw" yaw_deg="-135"/>
 </robot>

Commit message: update f450 & f550 model

File: tobas_description/urdf/f450.xacro (robot description, xacro)
@@ -7,5 +7,9 @@
   <xacro:property name="frame_width" value="0.35"/>
   <xacro:property name="frame_height" value="0.06"/>
-  <xacro:property name="frame_mass" value="0.780"/>
+  <xacro:property name="frame_mass" value="0.55346"/>
+  <xacro:property name="fc_x" value="0.09"/>
+  <xacro:property name="fc_y" value="0.055"/>
+  <xacro:property name="fc_z" value="0.05"/>
+  <xacro:property name="fc_mass" value="0.2"/>
   <xacro:property name="battery_x" value="0.106"/>
   <xacro:property name="battery_y" value="0.035"/>
@@ -29,5 +33,5 @@
       <origin xyz="0 0 0" rpy="0 0 0"/>
       <geometry>
-        <mesh filename="package://tobas_description/meshes/f450/frame.stl" scale="1e-3 1e-3 1e-3"/>
+        <mesh filename="package://tobas_description/meshes/f450/frame.stl" scale="1 1 1"/>
       </geometry>
       <xacro:insert_block name="black"/>
@@ -35,6 +39,6 @@
     <inertial>
       <mass value="${frame_mass}"/>
-      <origin xyz="0.001573 -0.000596 -0.003436" rpy="0 0 0"/>
-      <inertia ixx="9.613e-3" ixy="-6.070442e-6" ixz="-4.7933683e-5" iyy="9.702e-3" iyz="-3.987551e-6" izz="1.867e-2"/>
+      <origin xyz="0 0 -4.136e-3" rpy="0 0 0"/>
+      <inertia ixx="8.128e-3" ixy="0" ixz="0" iyy="8.193e-3" iyz="0" izz="1.597e-2"/>
     </inertial>
     <collision>
@@ -42,4 +46,29 @@
       <geometry>
         <box size="${frame_width} ${frame_width} ${frame_height}"/>
+      </geometry>
+    </collision>
+  </link>
+  <!-- Flight Controller -->
+  <joint name="flight_controller_joint" type="fixed">
+    <origin xyz="0 0.015 0" rpy="0 0 0"/>
+    <parent link="base_link"/>
+    <child link="flight_controller"/>
+  </joint>
+  <link name="flight_controller">
+    <visual>
+      <geometry>
+        <mesh filename="package://tobas_description/meshes/common/flight_controller/rpi_hat_avm.stl" scale="1 1 1"/>
+      </geometry>
+      <xacro:insert_block name="red"/>
+    </visual>
+    <inertial>
+      <mass value="${fc_mass}"/>
+      <origin xyz="0 0 ${fc_z/2}" rpy="0 0 0"/>
+      <xacro:box_inertia x="${fc_x}" y="${fc_y}" z="${fc_z}" mass="${fc_mass}"/>
+    </inertial>
+    <collision>
+      <origin xyz="0 0 ${fc_z/2}" rpy="0 0 0"/>
+      <geometry>
+        <box size="${fc_x} ${fc_y} ${fc_z}"/>
       </geometry>
     </collision>

File: tobas_description/urdf/f550.xacro (robot description, xacro)
@@ -7,5 +7,9 @@
   <xacro:property name="frame_radius" value="0.294"/>
   <xacro:property name="frame_height" value="0.056"/>
-  <xacro:property name="frame_mass" value="0.979"/>
+  <xacro:property name="frame_mass" value="0.916217"/>
+  <xacro:property name="fc_x" value="0.09"/>
+  <xacro:property name="fc_y" value="0.055"/>
+  <xacro:property name="fc_z" value="0.05"/>
+  <xacro:property name="fc_mass" value="0.2"/>
   <xacro:property name="battery_x" value="0.155"/>
   <xacro:property name="battery_y" value="0.048"/>
@@ -35,8 +39,33 @@
     <inertial>
       <mass value="${frame_mass}"/>
-      <origin xyz="0.624e-3 1.181e-3 14.463e-3" rpy="0 0 0"/>
-      <inertia ixx="2.006e-2" ixy="-2.872e-6" ixz="-2.083e-5" iyy="2.010e-2" iyz="3.472e-6" izz="3.939e-2"/>
+      <origin xyz="0 0 -6.031e-3" rpy="0 0 0"/>
+      <inertia ixx="1.953e-2" ixy="-2.894e-6" ixz="2.258e-6" iyy="1.953e-2" iyz="3.192e-6" izz="3.837e-2"/>
     </inertial>
     <xacro:hexagonal_prism_collision side="${frame_radius}" height="${frame_height}" x0="0" y0="0" z0="${-frame_height/2}"/>
+  </link>
+  <!-- Flight Controller -->
+  <joint name="flight_controller_joint" type="fixed">
+    <origin xyz="0 0 0" rpy="0 0 0"/>
+    <parent link="base_link"/>
+    <child link="flight_controller"/>
+  </joint>
+  <link name="flight_controller">
+    <visual>
+      <geometry>
+        <mesh filename="package://tobas_description/meshes/common/flight_controller/rpi_hat_avm.stl" scale="1 1 1"/>
+      </geometry>
+      <xacro:insert_block name="red"/>
+    </visual>
+    <inertial>
+      <mass value="${fc_mass}"/>
+      <origin xyz="0 0 ${fc_z/2}" rpy="0 0 0"/>
+      <xacro:box_inertia x="${fc_x}" y="${fc_y}" z="${fc_z}" mass="${fc_mass}"/>
+    </inertial>
+    <collision>
+      <origin xyz="0 0 ${fc_z/2}" rpy="0 0 0"/>
+      <geometry>
+        <box size="${fc_x} ${fc_y} ${fc_z}"/>
+      </geometry>
+    </collision>
   </link>
   <!-- Battery -->

Commit message: edit urdfs

File: tobas_description/urdf/f450.xacro (robot description, xacro)
@@ -4,12 +4,9 @@
   <!-- Included URDF Files -->
   <xacro:include filename="$(find tobas_description)/urdf/components/multirotor_base.xacro"/>
+  <xacro:include filename="$(find tobas_description)/urdf/components/flight_controller/tobas_aso.xacro"/>
   <!-- Properties -->
   <xacro:property name="frame_width" value="0.35"/>
   <xacro:property name="frame_height" value="0.06"/>
   <xacro:property name="frame_mass" value="0.55346"/>
-  <xacro:property name="fc_x" value="0.09"/>
-  <xacro:property name="fc_y" value="0.055"/>
-  <xacro:property name="fc_z" value="0.05"/>
-  <xacro:property name="fc_mass" value="0.2"/>
   <xacro:property name="battery_x" value="0.106"/>
   <xacro:property name="battery_y" value="0.035"/>
@@ -50,28 +47,7 @@
   </link>
   <!-- Flight Controller -->
-  <joint name="flight_controller_joint" type="fixed">
+  <xacro:tobas_aso parent="base_link">
     <origin xyz="0 0.015 0" rpy="0 0 0"/>
-    <parent link="base_link"/>
-    <child link="flight_controller"/>
-  </joint>
-  <link name="flight_controller">
-    <visual>
-      <geometry>
-        <mesh filename="package://tobas_description/meshes/common/flight_controller/rpi_hat_avm.stl" scale="1 1 1"/>
-      </geometry>
-      <xacro:insert_block name="red"/>
-    </visual>
-    <inertial>
-      <mass value="${fc_mass}"/>
-      <origin xyz="0 0 ${fc_z/2}" rpy="0 0 0"/>
-      <xacro:box_inertia x="${fc_x}" y="${fc_y}" z="${fc_z}" mass="${fc_mass}"/>
-    </inertial>
-    <collision>
-      <origin xyz="0 0 ${fc_z/2}" rpy="0 0 0"/>
-      <geometry>
-        <box size="${fc_x} ${fc_y} ${fc_z}"/>
-      </geometry>
-    </collision>
-  </link>
+  </xacro:tobas_aso>
   <!-- Battery -->
   <joint name="battery_joint" type="fixed">

File: tobas_description/urdf/f550.xacro (robot description, xacro)
@@ -4,12 +4,9 @@
   <!-- Included URDF Files -->
   <xacro:include filename="$(find tobas_description)/urdf/components/multirotor_base.xacro"/>
+  <xacro:include filename="$(find tobas_description)/urdf/components/flight_controller/tobas_aso.xacro"/>
   <!-- Properties -->
   <xacro:property name="frame_radius" value="0.294"/>
   <xacro:property name="frame_height" value="0.056"/>
   <xacro:property name="frame_mass" value="0.916217"/>
-  <xacro:property name="fc_x" value="0.09"/>
-  <xacro:property name="fc_y" value="0.055"/>
-  <xacro:property name="fc_z" value="0.05"/>
-  <xacro:property name="fc_mass" value="0.2"/>
   <xacro:property name="battery_x" value="0.155"/>
   <xacro:property name="battery_y" value="0.048"/>
@@ -45,28 +42,7 @@
   </link>
   <!-- Flight Controller -->
-  <joint name="flight_controller_joint" type="fixed">
+  <xacro:tobas_aso parent="base_link">
     <origin xyz="0 0 0" rpy="0 0 0"/>
-    <parent link="base_link"/>
-    <child link="flight_controller"/>
-  </joint>
-  <link name="flight_controller">
-    <visual>
-      <geometry>
-        <mesh filename="package://tobas_description/meshes/common/flight_controller/rpi_hat_avm.stl" scale="1 1 1"/>
-      </geometry>
-      <xacro:insert_block name="red"/>
-    </visual>
-    <inertial>
-      <mass value="${fc_mass}"/>
-      <origin xyz="0 0 ${fc_z/2}" rpy="0 0 0"/>
-      <xacro:box_inertia x="${fc_x}" y="${fc_y}" z="${fc_z}" mass="${fc_mass}"/>
-    </inertial>
-    <collision>
-      <origin xyz="0 0 ${fc_z/2}" rpy="0 0 0"/>
-      <geometry>
-        <box size="${fc_x} ${fc_y} ${fc_z}"/>
-      </geometry>
-    </collision>
-  </link>
+  </xacro:tobas_aso>
   <!-- Battery -->
   <joint name="battery_joint" type="fixed">

Commit message: edit battery

File: tobas_description/urdf/f450.xacro (robot description, xacro)
@@ -5,5 +5,5 @@
   <xacro:include filename="$(find tobas_description)/urdf/components/multirotor_base.xacro"/>
   <xacro:include filename="$(find tobas_description)/urdf/components/flight_controller/tobas_aso.xacro"/>
-  <xacro:include filename="$(find tobas_description)/urdf/components/battery/sigp_3s_2250mah_30c.xacro"/>
+  <xacro:include filename="$(find tobas_description)/urdf/components/battery/sigp_3s_2250mah_60c.xacro"/>
   <xacro:include filename="$(find tobas_description)/urdf/components/propeller/phantom3_0945.xacro"/>
   <!-- Properties -->
@@ -45,7 +45,7 @@
   </xacro:tobas_aso>
   <!-- Battery -->
-  <xacro:sigp_3s_2250mah_30c parent="base_link">
-    <origin xyz="-0.035 0 -0.024647" rpy="0 0 0"/>
-  </xacro:sigp_3s_2250mah_30c>
+  <xacro:sigp_3s_2250mah_60c parent="base_link">
+    <origin xyz="-0.037 0 -0.023" rpy="0 0 0"/>
+  </xacro:sigp_3s_2250mah_60c>
   <!-- Propellers -->
   <xacro:macro name="propeller" params="index direction yaw_deg">

Commit message: edit fmu model

File: tobas_description/urdf/f450.xacro (robot description, xacro)
@@ -4,5 +4,5 @@
   <!-- Included URDF Files -->
   <xacro:include filename="$(find tobas_description)/urdf/components/multirotor_base.xacro"/>
-  <xacro:include filename="$(find tobas_description)/urdf/components/flight_controller/tobas_aso.xacro"/>
+  <xacro:include filename="$(find tobas_description)/urdf/components/fmu/tobas_aso.xacro"/>
   <xacro:include filename="$(find tobas_description)/urdf/components/battery/sigp_3s_2250mah_60c.xacro"/>
   <xacro:include filename="$(find tobas_description)/urdf/components/propeller/phantom3_0945.xacro"/>
@@ -42,5 +42,5 @@
   <!-- Flight Controller -->
   <xacro:tobas_aso parent="base_link">
-    <origin xyz="0 0.015 0" rpy="0 0 0"/>
+    <origin xyz="0 0.015 0.020" rpy="0 0 0"/>
   </xacro:tobas_aso>
   <!-- Battery -->

File: tobas_description/urdf/f550.xacro (robot description, xacro)
@@ -4,5 +4,5 @@
   <!-- Included URDF Files -->
   <xacro:include filename="$(find tobas_description)/urdf/components/multirotor_base.xacro"/>
-  <xacro:include filename="$(find tobas_description)/urdf/components/flight_controller/tobas_aso.xacro"/>
+  <xacro:include filename="$(find tobas_description)/urdf/components/fmu/tobas_aso.xacro"/>
   <xacro:include filename="$(find tobas_description)/urdf/components/battery/hrb_4s_5000mah_50c.xacro"/>
   <xacro:include filename="$(find tobas_description)/urdf/components/propeller/phantom3_0945.xacro"/>
@@ -37,5 +37,5 @@
   <!-- Flight Controller -->
   <xacro:tobas_aso parent="base_link">
-    <origin xyz="0 0 0" rpy="0 0 0"/>
+    <origin xyz="0 0 0.020" rpy="0 0 0"/>
   </xacro:tobas_aso>
   <!-- Battery -->

File: tobas_description/urdf/hydrus.xacro (robot description, xacro)
@@ -28,5 +28,5 @@
   <!-- 1.  processor -->
   <!-- 1.1 flight controller -->
-  <xacro:extra_module name="fc" parent="link2" visible="1" model_url="package://tobas_description/meshes/hydrus/ver2/flight_controller/spinal.dae">    <!-- same with intel euclid -->
+  <xacro:extra_module name="fc" parent="link2" visible="1" model_url="package://tobas_description/meshes/hydrus/ver2/fmu/spinal.dae">    <!-- same with intel euclid -->
     <origin xyz="${link_length / 2 + 0.2221} ${-4.4*0.001} 0.02135" rpy="0 0 0"/>
     <inertial>

File: tobas_description/urdf/voliro_like.xacro (robot description, xacro)
@@ -4,5 +4,5 @@
   <!-- Included URDF Files -->
   <xacro:include filename="$(find tobas_description)/urdf/components/multirotor_base.xacro"/>
-  <xacro:include filename="$(find tobas_description)/urdf/components/flight_controller/tobas_aso.xacro"/>
+  <xacro:include filename="$(find tobas_description)/urdf/components/fmu/tobas_aso.xacro"/>
   <xacro:include filename="$(find tobas_description)/urdf/components/propeller/phantom3_0945.xacro"/>
   <!-- Properties -->
@@ -33,5 +33,5 @@
   <!-- Flight Controller -->
   <xacro:tobas_aso parent="base_link">
-    <origin xyz="0 0 0.037" rpy="0 0 0"/>
+    <origin xyz="0 0 0.057" rpy="0 0 0"/>
   </xacro:tobas_aso>
   <!-- Tilt Rotor -->

Commit message: fix: Fix FMU position

File: tobas_description/urdf/f450.xacro (robot description, xacro)
@@ -39,5 +39,5 @@
   <!-- Flight Controller -->
   <xacro:tobas_t1 parent="base_link">
-    <origin xyz="0 0.015 0.020" rpy="0 0 0"/>
+    <origin xyz="0 0.015 0" rpy="0 0 0"/>
   </xacro:tobas_t1>
   <!-- Battery -->

File: tobas_description/urdf/f550.xacro (robot description, xacro)
@@ -35,5 +35,5 @@
   <!-- Flight Controller -->
   <xacro:tobas_t1 parent="base_link">
-    <origin xyz="0 0 0.020" rpy="0 0 0"/>
+    <origin xyz="0 0 0" rpy="0 0 0"/>
   </xacro:tobas_t1>
   <!-- Battery -->
