Commit message: .

File: tobas_description/urdf/components/fixed_wing_base.xacro (robot description, xacro)
@@ -1,12 +1,5 @@
 <?xml version="1.0"?>
 <robot xmlns:xacro="http://ros.org/wiki/xacro">
-  <!-- Macro for the inertia of a box -->
-  <xacro:macro name="box_inertia" params="x y z mass">
-    <inertia ixx="${0.0833333 * mass * (y*y + z*z)}" ixy="0.0" ixz="0.0" iyy="${0.0833333 * mass * (x*x + z*z)}" iyz="0.0" izz="${0.0833333 * mass * (x*x + y*y)}" />
-  </xacro:macro>
-  <!-- Macro for the inertia of a cylinder -->
-  <xacro:macro name="cylinder_inertia" params="r h mass">
-    <inertia ixx="${0.0833333 * mass * (3*r*r + h*h)}" ixy="0.0" ixz="0.0" iyy="${0.0833333 * mass * (3*r*r + h*h)}" iyz="0.0" izz="${0.5 * mass * r * r}" />
-  </xacro:macro>
+  <xacro:include filename="$(find tobas_description)/urdf/components/common.xacro"/>
   <!-- Fixed-wing main body link -->
   <xacro:macro name="fixed_wing_base_macro" params="robot_namespace

File: tobas_description/urdf/components/multirotor_base.xacro (robot description, xacro)
@@ -1,30 +1,5 @@
 <?xml version="1.0"?>
 <robot xmlns:xacro="http://ros.org/wiki/xacro">
-  <!-- Constants -->
-  <xacro:property name="sin30" value="0.5"/>
-  <xacro:property name="cos30" value="0.866025403784"/>
-  <!-- Properties -->
-  <xacro:property name="deg2rad" value="${pi / 180}"/>
-  <xacro:property name="rad2deg" value="${180 / pi}"/>
-  <!-- Macro for the inertia of a cylinder -->
-	<xacro:macro name="cylinder_inertia" params="radius length mass">
-		<inertia ixx="${mass*radius*radius/4 + mass*length*length/12}" ixy="0.0" ixz="0.0" iyy="${mass*radius*radius/4 + mass*length*length/12}" iyz="0.0" izz="${mass*radius*radius/2}" />
-	</xacro:macro>
-  <!-- Macro for the inertia of a sphere -->
-	<xacro:macro name="sphere_inertia" params="radius mass">
-		<inertia ixx="${0.4 * mass * radius*radius}" ixy="0.0" ixz="0.0" iyy="${0.4 * mass * radius*radius}" iyz="0.0" izz="${0.4 * mass * radius*radius}" />
-	</xacro:macro>
-  <!-- Macro for the inertia of a box -->
-  <xacro:macro name="box_inertia" params="x y z mass">
-    <inertia ixx="${mass * (y*y + z*z) / 12}" ixy="0.0" ixz="0.0" iyy="${mass * (x*x + z*z) / 12}" iyz="0.0" izz="${mass * (x*x + y*y) / 12}" />
-  </xacro:macro>
-  <!-- Macro for the inertial properties of a box -->
-  <xacro:macro name="box_inertial" params="x y z mass *origin">
-    <inertial>
-      <mass value="${mass}" />
-      <xacro:insert_block name="origin" />
-      <xacro:box_inertia x="${x}" y="${y}" z="${z}" mass="${mass}" />
-    </inertial>
-  </xacro:macro>
+  <xacro:include filename="$(find tobas_description)/urdf/components/common.xacro"/>
   <!-- Main multirotor link -->
   <xacro:macro name="multirotor_base_macro" params="robot_namespace

File: tobas_description/urdf/firefly.xacro (robot description, xacro)
@@ -3,7 +3,4 @@
   <!-- Included URDF Files -->
   <xacro:include filename="$(find tobas_description)/urdf/components/multirotor_base.xacro" />
-  <!-- Constants -->
-  <xacro:property name="sin30" value="0.5" />
-  <xacro:property name="cos30" value="0.866025403784" />
   <!-- Properties -->
   <xacro:property name="namespace" value="firefly" />

File: tobas_description/urdf/s900.xacro (robot description, xacro)
@@ -35,7 +35,5 @@
         <mesh filename="package://tobas_description/meshes/s900/center_frame.stl" scale="1e-3 1e-3 1e-3"/>
       </geometry>
-      <material name="White">
-        <color rgba="1 1 1 1"/>
-      </material>
+      <xacro:insert_block name="white"/>
     </visual>
     <inertial>
@@ -62,7 +60,5 @@
         <mesh filename="package://tobas_description/meshes/s900/battery.stl" scale="1e-3 1e-3 1e-3"/>
       </geometry>
-      <material name="Black">
-        <color rgba="0 0 0 1"/>
-      </material>
+      <xacro:insert_block name="black"/>
     </visual>
     <inertial>
@@ -91,7 +87,5 @@
           <mesh filename="package://tobas_description/meshes/s900/landing_gear_upper.stl" scale="1e-3 1e-3 1e-3"/>
         </geometry>
-        <material name="Black">
-          <color rgba="0 0 0 1"/>
-        </material>
+        <xacro:insert_block name="black"/>
       </visual>
       <inertial>
@@ -118,7 +112,5 @@
           <mesh filename="package://tobas_description/meshes/s900/landing_gear_lower.stl" scale="1e-3 1e-3 1e-3"/>
         </geometry>
-        <material name="Black">
-          <color rgba="0 0 0 1"/>
-        </material>
+        <xacro:insert_block name="black"/>
       </visual>
       <inertial>
@@ -150,7 +142,5 @@
           <mesh filename="package://tobas_description/meshes/s900/arm.stl" scale="1e-3 1e-3 1e-3"/>
         </geometry>
-        <material name="Black">
-          <color rgba="0 0 0 1"/>
-        </material>
+        <xacro:insert_block name="black"/>
       </visual>
       <inertial>
@@ -177,7 +167,5 @@
           <mesh filename="package://tobas_description/meshes/s900/motor.stl" scale="1e-3 1e-3 1e-3"/>
         </geometry>
-        <material name="Black">
-          <color rgba="0 0 0 1"/>
-        </material>
+        <xacro:insert_block name="black"/>
       </visual>
       <inertial>
@@ -205,7 +193,5 @@
           <mesh filename="package://tobas_description/meshes/s900/propeller_${direction}.stl" scale="1e-3 1e-3 1e-3"/>
         </geometry>
-        <material name="Black">
-          <color rgba="0.0 0.0 0.0 1.0"/>
-        </material>
+        <xacro:insert_block name="black"/>
       </visual>
       <inertial>

Commit message: fix: xacro

File: tobas_description/urdf/components/fixed_wing_base.xacro (robot description, xacro)
@@ -3,7 +3,10 @@
   <xacro:include filename="$(find tobas_description)/urdf/components/common.xacro"/>
   <!-- Fixed-wing main body link -->
-  <xacro:macro name="fixed_wing_base_macro" params="robot_namespace
-      mass length
-      width height
+  <xacro:macro name="fixed_wing_base_macro" params="
+      robot_namespace
+      mass
+      length
+      width
+      height
       color
       use_mesh_file
@@ -46,5 +49,6 @@
   </xacro:macro>
   <!-- Control surface joint and link -->
-  <xacro:macro name="control_surface" params="robot_namespace
+  <xacro:macro name="control_surface" params="
+      robot_namespace
       surface_name
       parent
@@ -105,5 +109,6 @@
   </xacro:macro>
   <!-- Propeller joint and link -->
-  <xacro:macro name="propeller" params="robot_namespace
+  <xacro:macro name="propeller" params="
+      robot_namespace
       suffix
       parent
@@ -152,5 +157,6 @@
   </xacro:macro>
   <!-- Wheel joint and link -->
-  <xacro:macro name="wheel" params="robot_namespace
+  <xacro:macro name="wheel" params="
+      robot_namespace
       suffix
       parent

File: tobas_description/urdf/components/multirotor_base.xacro (robot description, xacro)
@@ -3,5 +3,6 @@
   <xacro:include filename="$(find tobas_description)/urdf/components/common.xacro"/>
   <!-- Main multirotor link -->
-  <xacro:macro name="multirotor_base_macro" params="robot_namespace
+  <xacro:macro name="multirotor_base_macro" params="
+      robot_namespace
       mass
       body_width
@@ -42,5 +43,6 @@
   </xacro:macro>
   <!-- Rotor joint and link -->
-  <xacro:macro name="vertical_rotor" params="robot_namespace
+  <xacro:macro name="vertical_rotor" params="
+      robot_namespace
       direction
       parent

File: tobas_description/urdf/techpod.xacro (robot description, xacro)
@@ -95,9 +95,9 @@
   <!-- Inertia of the propeller, assuming it is a cylinder -->
   <xacro:property name="propeller_inertia">
-    <xacro:cylinder_inertia r="${propeller_radius}" h="${propeller_height}" mass="${mass_propeller}"/>
+    <xacro:cylinder_inertia radius="${propeller_radius}" length="${propeller_height}" mass="${mass_propeller}"/>
   </xacro:property>
   <!-- Inertia of the wheels, assuming it is a cylinder -->
   <xacro:property name="wheel_inertia">
-    <xacro:cylinder_inertia r="${wheel_radius}" h="${wheel_height}" mass="${wheel_mass}"/>
+    <xacro:cylinder_inertia radius="${wheel_radius}" length="${wheel_height}" mass="${wheel_mass}"/>
   </xacro:property>
   <!-- Included URDF Files -->

Commit message: fix

File: tobas_description/urdf/components/fixed_wing_base.xacro (robot description, xacro)
@@ -120,5 +120,5 @@
       *origin
       *inertia">
-    <joint name="${robot_namespace}/propeller_{suffix}_joint" type="continuous">
+    <joint name="${robot_namespace}/propeller_${suffix}_joint" type="continuous">
       <xacro:insert_block name="origin"/>
       <axis xyz="0 0 1"/>
