Commit message: add: f500_non_planar

File: tobas_description/urdf/components/common.xacro (robot description, xacro)
@@ -10,7 +10,7 @@
   <xacro:property name="sin60" value="${cos30}"/>
   <xacro:property name="cos60" value="${sin30}"/>
-  <!-- Properties -->
   <xacro:property name="deg2rad" value="${pi / 180}"/>
   <xacro:property name="rad2deg" value="${180 / pi}"/>
+  <xacro:property name="inch2meter" value="0.0254"/>
   <!-- Colors -->
   <xacro:property name="black">

Commit message: .

File: tobas_description/urdf/components/common.xacro (robot description, xacro)
@@ -22,4 +22,9 @@
     <material name="white">
       <color rgba="1 1 1 1"/>
+    </material>
+  </xacro:property>
+  <xacro:property name="gray">
+    <material name="gray">
+      <color rgba="0.5 0.5 0.5 1"/>
     </material>
   </xacro:property>

Commit message: 6角柱のcollisionを定義

File: tobas_description/urdf/components/common.xacro (robot description, xacro)
@@ -44,4 +44,25 @@
     </material>
   </xacro:property>
+  <!-- Collisions -->
+  <xacro:macro name="hexagonal_prism_collision" params="side height x0 y0 z0">
+    <collision>
+      <origin xyz="${x0} ${y0} ${z0}" rpy="0 0 0"/>
+      <geometry>
+        <box size="${sqrt3*side} ${side} ${height}"/>
+      </geometry>
+    </collision>
+    <collision>
+      <origin xyz="${x0} ${y0} ${z0}" rpy="0 0 ${60*deg2rad}"/>
+      <geometry>
+        <box size="${sqrt3*side} ${side} ${height}"/>
+      </geometry>
+    </collision>
+    <collision>
+      <origin xyz="${x0} ${y0} ${z0}" rpy="0 0 ${-60*deg2rad}"/>
+      <geometry>
+        <box size="${sqrt3*side} ${side} ${height}"/>
+      </geometry>
+    </collision>
+  </xacro:macro>
   <!-- Inertia of primitive shapes -->
   <xacro:macro name="cylinder_inertia" params="radius length mass">
@@ -58,6 +79,6 @@
     <inertial>
       <mass value="${mass}" />
-      <xacro:insert_block name="origin" />
-      <xacro:box_inertia x="${x}" y="${y}" z="${z}" mass="${mass}" />
+      <xacro:insert_block name="origin"/>
+      <xacro:box_inertia x="${x}" y="${y}" z="${z}" mass="${mass}"/>
     </inertial>
   </xacro:macro>

File: tobas_description/urdf/f550_non_planar.xacro (robot description, xacro)
@@ -34,10 +34,5 @@
       <inertia ixx="4.970e-2" ixy="-1.85346e-7" ixz="-8.26373e-6" iyy="4.975e-2" iyz="-5.7596072e-5" izz="9.558e-2"/>
     </inertial>
-    <collision>
-      <origin xyz="0 0 ${-frame_height/2}" rpy="0 0 0"/>
-      <geometry>
-        <cylinder radius="${frame_radius}" length="${frame_height}"/>
-      </geometry>
-    </collision>
+    <xacro:hexagonal_prism_collision side="${frame_radius}" height="${frame_height}" x0="0" y0="0" z0="${-frame_height/2}"/>
   </link>
   <!-- Propellers -->

Commit message: F550 NP RM-X52のURDFを追加

File: tobas_description/urdf/components/common.xacro (robot description, xacro)
@@ -44,4 +44,14 @@
     </material>
   </xacro:property>
+  <xacro:property name="orange">
+    <material name="orange">
+      <color rgba="${255/255} ${108/255} ${10/255} 1"/>
+    </material>
+  </xacro:property>
+  <xacro:property name="brown">
+    <material name="brown">
+      <color rgba="${222/255} ${207/255} ${195/255} 1"/>
+    </material>
+  </xacro:property>
   <!-- Collisions -->
   <xacro:macro name="hexagonal_prism_collision" params="side height x0 y0 z0">

File: tobas_description/urdf/f550_np_rmx52.xacro (robot description, xacro)
@@ -1,7 +1,8 @@
 <?xml version="1.0"?>
-<robot name="f550_np"
+<robot name="f550_np_rmx52"
   xmlns:xacro="http://ros.org/wiki/xacro">
   <!-- Included URDF Files -->
   <xacro:include filename="$(find tobas_description)/urdf/components/multirotor_base.xacro"/>
+  <xacro:include filename="$(find tobas_description)/urdf/components/rmx52/rmx52.xacro"/>
   <!-- Properties -->
   <xacro:property name="frame_mass" value="1.579"/>
@@ -116,3 +117,10 @@
     <origin xyz="0.242082 -0.130355 ${propeller_origin_z}" rpy="${-rotor_tilt} 0 ${330*deg2rad}"/>
   </xacro:propeller>
+  <!-- Robot Arm -->
+  <joint name="rmx52_joint" type="fixed">
+    <origin xyz="0.004 0 -0.0445" rpy="${pi} 0 0"/>
+    <parent link="base_link"/>
+    <child link="rmx52/link1"/>
+  </joint>
+  <xacro:rmx52/>
 </robot>

Commit message: Custom Jointsの設定画面を実装

File: tobas_description/urdf/components/common.xacro (robot description, xacro)
@@ -93,3 +93,30 @@
     </inertial>
   </xacro:macro>
+  <!-- Transmissions -->
+  <xacro:macro name="simple_transmission" params="jnt_name *hardware_interface">
+    <transmission name="${jnt_name}_trans">
+      <type>transmission_interface/SimpleTransmission</type>
+      <joint name="${jnt_name}">
+        <xacro:insert_block name="hardware_interface"/>
+      </joint>
+      <actuator name="${jnt_name}_actuator">
+        <mechanicalReduction>1</mechanicalReduction>
+      </actuator>
+    </transmission>
+  </xacro:macro>
+  <xacro:macro name="simple_transmission_position" params="jnt_name">
+    <xacro:simple_transmission jnt_name="${jnt_name}">
+      <hardwareInterface>hardware_interface/PositionJointInterface</hardwareInterface>
+    </xacro:simple_transmission>
+  </xacro:macro>
+  <xacro:macro name="simple_transmission_velocity" params="jnt_name">
+    <xacro:simple_transmission jnt_name="${jnt_name}">
+      <hardwareInterface>hardware_interface/VelocityJointInterface</hardwareInterface>
+    </xacro:simple_transmission>
+  </xacro:macro>
+  <xacro:macro name="simple_transmission_effort" params="jnt_name">
+    <xacro:simple_transmission jnt_name="${jnt_name}">
+      <hardwareInterface>hardware_interface/EffortJointInterface</hardwareInterface>
+    </xacro:simple_transmission>
+  </xacro:macro>
 </robot>

File: tobas_description/urdf/components/rmx52/rmx52.xacro (robot description, xacro)
@@ -7,4 +7,6 @@
     <!-- Import all Gazebo-customization elements, including Gazebo colors -->
     <xacro:include filename="$(find tobas_description)/urdf/components/rmx52/gazebo.xacro"/>
+    <!-- Import transmissions -->
+    <xacro:include filename="$(find tobas_description)/urdf/components/rmx52/transmission.xacro"/>
   </xacro:macro>
 </robot>

Commit message: .

File: tobas_description/urdf/components/common.xacro (robot description, xacro)
@@ -75,5 +75,8 @@
     </collision>
   </xacro:macro>
-  <!-- Inertia of primitive shapes -->
+  <!-- Inertia wrt. CoM of primitive shapes -->
+  <xacro:macro name="box_inertia" params="x y z mass">
+    <inertia ixx="${mass * (y*y + z*z) / 12}" ixy="0.0" ixz="0.0" iyy="${mass * (x*x + z*z) / 12}" iyz="0.0" izz="${mass * (x*x + y*y) / 12}"/>
+  </xacro:macro>
   <xacro:macro name="cylinder_inertia" params="radius length mass">
     <inertia ixx="${mass*radius*radius/4 + mass*length*length/12}" ixy="0.0" ixz="0.0" iyy="${mass*radius*radius/4 + mass*length*length/12}" iyz="0.0" izz="${mass*radius*radius/2}"/>
@@ -81,7 +84,4 @@
   <xacro:macro name="sphere_inertia" params="radius mass">
     <inertia ixx="${0.4 * mass * radius*radius}" ixy="0.0" ixz="0.0" iyy="${0.4 * mass * radius*radius}" iyz="0.0" izz="${0.4 * mass * radius*radius}"/>
-  </xacro:macro>
-  <xacro:macro name="box_inertia" params="x y z mass">
-    <inertia ixx="${mass * (y*y + z*z) / 12}" ixy="0.0" ixz="0.0" iyy="${mass * (x*x + z*z) / 12}" iyz="0.0" izz="${mass * (x*x + y*y) / 12}"/>
   </xacro:macro>
   <!-- Macro for the inertial properties of a box -->

Commit message: edit xacros

File: tobas_description/urdf/components/common.xacro (robot description, xacro)
@@ -93,30 +93,3 @@
     </inertial>
   </xacro:macro>
-  <!-- Transmissions -->
-  <xacro:macro name="simple_transmission" params="jnt_name *hardware_interface">
-    <transmission name="${jnt_name}_trans">
-      <type>transmission_interface/SimpleTransmission</type>
-      <joint name="${jnt_name}">
-        <xacro:insert_block name="hardware_interface"/>
-      </joint>
-      <actuator name="${jnt_name}_actuator">
-        <mechanicalReduction>1</mechanicalReduction>
-      </actuator>
-    </transmission>
-  </xacro:macro>
-  <xacro:macro name="simple_transmission_position" params="jnt_name">
-    <xacro:simple_transmission jnt_name="${jnt_name}">
-      <hardwareInterface>hardware_interface/PositionJointInterface</hardwareInterface>
-    </xacro:simple_transmission>
-  </xacro:macro>
-  <xacro:macro name="simple_transmission_velocity" params="jnt_name">
-    <xacro:simple_transmission jnt_name="${jnt_name}">
-      <hardwareInterface>hardware_interface/VelocityJointInterface</hardwareInterface>
-    </xacro:simple_transmission>
-  </xacro:macro>
-  <xacro:macro name="simple_transmission_effort" params="jnt_name">
-    <xacro:simple_transmission jnt_name="${jnt_name}">
-      <hardwareInterface>hardware_interface/EffortJointInterface</hardwareInterface>
-    </xacro:simple_transmission>
-  </xacro:macro>
 </robot>

File: tobas_description/urdf/components/fixed_wing_base.xacro (robot description, xacro)
@@ -95,10 +95,5 @@
         <xacro:insert_block name="link_origin"/>
         <geometry>
-          <xacro:if value="${use_mesh_file}">
-            <mesh filename="${mesh_file}" scale="1 1 1"/>
-          </xacro:if>
-          <xacro:unless value="${use_mesh_file}">
-            <box size="${surface_length} ${surface_width} ${surface_height}"/>
-          </xacro:unless>
+          <box size="${surface_length} ${surface_width} ${surface_height}"/>
         </geometry>
       </collision>
@@ -143,10 +138,5 @@
       <collision>
         <geometry>
-          <xacro:if value="${use_mesh_file}">
-            <mesh filename="${mesh_file}" scale="${propeller_radius} ${propeller_radius} ${propeller_radius}"/>
-          </xacro:if>
-          <xacro:unless value="${use_mesh_file}">
-            <cylinder length="0.005" radius="${propeller_radius}"/>
-          </xacro:unless>
+          <cylinder length="0.005" radius="${propeller_radius}"/>
         </geometry>
       </collision>

File: tobas_description/urdf/techpod.xacro (robot description, xacro)
@@ -1,7 +1,4 @@
 <?xml version="1.0"?>
 <robot name="techpod" xmlns:xacro="http://ros.org/wiki/xacro">
-  <!-- Constants -->
-  <xacro:property name="PI" value="3.1415926535897931"/>
-  <xacro:property name="DEG2RAD" value="${PI / 180.0}"/>
   <!-- Global properties -->
   <xacro:property name="namespace" value="techpod"/>
@@ -24,6 +21,6 @@
   <xacro:property name="aileron_width" value="0.349"/> <!-- [m] -->
   <xacro:property name="aileron_height" value="0.013"/> <!-- [m] -->
-  <xacro:property name="aileron_min_angle" value="-${20.0 * DEG2RAD}"/> <!-- [rad] -->
-  <xacro:property name="aileron_max_angle" value="${20.0 * DEG2RAD}"/> <!-- [rad] -->
+  <xacro:property name="aileron_min_angle" value="-${20.0 * deg2rad}"/> <!-- [rad] -->
+  <xacro:property name="aileron_max_angle" value="${20.0 * deg2rad}"/> <!-- [rad] -->
   <xacro:property name="aileron_max_velocity" value="10.0"/> <!-- [rad/s] -->
   <xacro:property name="aileron_max_effort" value="1e+6"/> <!-- [Nm] -->
@@ -35,6 +32,6 @@
   <xacro:property name="elevator_width" value="0.457"/> <!-- [m] -->
   <xacro:property name="elevator_height" value="0.012"/> <!-- [m] -->
-  <xacro:property name="elevator_min_angle" value="-${20.0 * DEG2RAD}"/> <!-- [rad] -->
-  <xacro:property name="elevator_max_angle" value="${20.0 * DEG2RAD}"/> <!-- [rad] -->
+  <xacro:property name="elevator_min_angle" value="-${20.0 * deg2rad}"/> <!-- [rad] -->
+  <xacro:property name="elevator_max_angle" value="${20.0 * deg2rad}"/> <!-- [rad] -->
   <xacro:property name="elevator_max_velocity" value="10.0"/> <!-- [rad/s] -->
   <xacro:property name="elevator_max_effort" value="1e+6"/> <!-- [Nm] -->
@@ -45,6 +42,6 @@
   <xacro:property name="flap_width" value="0.459"/> <!-- [m] -->
   <xacro:property name="flap_height" value="0.016"/> <!-- [m] -->
-  <xacro:property name="flap_min_angle" value="-${20.0 * DEG2RAD}"/> <!-- [rad] -->
-  <xacro:property name="flap_max_angle" value="${20.0 * DEG2RAD}"/> <!-- [rad] -->
+  <xacro:property name="flap_min_angle" value="-${20.0 * deg2rad}"/> <!-- [rad] -->
+  <xacro:property name="flap_max_angle" value="${20.0 * deg2rad}"/> <!-- [rad] -->
   <xacro:property name="flap_max_velocity" value="10.0"/> <!-- [rad/s] -->
   <xacro:property name="flap_max_effort" value="1e+6"/> <!-- [Nm] -->
@@ -56,6 +53,6 @@
   <xacro:property name="rudder_width" value="0.018"/>
   <xacro:property name="rudder_height" value="0.241"/>
-  <xacro:property name="rudder_min_angle" value="-${20.0 * DEG2RAD}"/>
-  <xacro:property name="rudder_max_angle" value="${20.0 * DEG2RAD}"/>
+  <xacro:property name="rudder_min_angle" value="-${20.0 * deg2rad}"/>
+  <xacro:property name="rudder_max_angle" value="${20.0 * deg2rad}"/>
   <xacro:property name="rudder_max_velocity" value="10.0"/>
   <xacro:property name="rudder_max_effort" value="1e+6"/>
@@ -124,5 +121,5 @@
     radius="${wheel_radius}"
     color="${wheel_color}">
-		<origin xyz="0.3 0.2 -0.2" rpy="${PI / 2} 0 0"/>
+		<origin xyz="0.3 0.2 -0.2" rpy="${pi / 2} 0 0"/>
     <xacro:insert_block name="wheel_inertia"/>
   </xacro:wheel>
@@ -135,5 +132,5 @@
     radius="${wheel_radius}"
     color="${wheel_color}">
-		<origin xyz="0.3 -0.2 -0.2" rpy="${PI / 2} 0 0"/>
+		<origin xyz="0.3 -0.2 -0.2" rpy="${pi / 2} 0 0"/>
     <xacro:insert_block name="wheel_inertia"/>
   </xacro:wheel>
@@ -146,5 +143,5 @@
     radius="${wheel_radius}"
     color="${wheel_color}">
-		<origin xyz="-0.3 0 -0.2" rpy="${PI / 2} 0 0"/>
+		<origin xyz="-0.3 0 -0.2" rpy="${pi / 2} 0 0"/>
     <xacro:insert_block name="wheel_inertia"/>
   </xacro:wheel>
@@ -242,5 +239,5 @@
     use_mesh_file="${use_mesh}"
     mesh_file="${propeller_mesh_file}">
-    <origin xyz="-0.025 0 0.15" rpy="0 ${PI / 2} 0"/>
+    <origin xyz="-0.025 0 0.15" rpy="0 ${pi / 2} 0"/>
     <xacro:insert_block name="propeller_inertia"/>
   </xacro:propeller>
