Commit message: edit: dummy_inertialを質点に

File: tobas_description/urdf/components/dummy.xacro (robot description, xacro)
@@ -1,7 +1,8 @@
 <robot xmlns:xacro="http://ros.org/wiki/xacro">
   <xacro:macro name="dummy_inertial">
+    <!-- A very light point mass -->
     <inertial>
-      <mass value="1e-9"/>
-      <inertia ixx="1e-9" ixy="0" ixz="0" iyy="1e-9" iyz="0" izz="1e-9"/>
+      <mass value="1e-6"/>
+      <inertia ixx="1e-12" ixy="0" ixz="0" iyy="1e-12" iyz="0" izz="1e-12"/>
     </inertial>
   </xacro:macro>
