Commit message: .

File: tobas_description/urdf/components/rmx52/rmx52.xacro (robot description, xacro)
@@ -4,7 +4,7 @@
   <xacro:macro name="rmx52" params="">
     <!-- Import URDF -->
-    <xacro:include filename="$(find tobas_description)/urdf/components/rmx52/urdf.xacro" />
+    <xacro:include filename="$(find tobas_description)/urdf/components/rmx52/urdf.xacro"/>
     <!-- Import all Gazebo-customization elements, including Gazebo colors -->
-    <xacro:include filename="$(find tobas_description)/urdf/components/rmx52/gazebo.xacro" />
+    <xacro:include filename="$(find tobas_description)/urdf/components/rmx52/gazebo.xacro"/>
   </xacro:macro>
 </robot>

File: tobas_description/urdf/components/rmx52/urdf.xacro (robot description, xacro)
@@ -17,7 +17,7 @@
     </collision>
     <inertial>
-      <origin xyz="3.0876154e-04 0.0000000e+00 -1.2176461e-04" />
-      <mass value="7.9119962e-02" />
-      <inertia ixx="1.2505234e-05" ixy="0.0" ixz="-1.7855208e-07" iyy="2.1898364e-05" iyz="0.0" izz="1.9267361e-05" />
+      <origin xyz="3.0876154e-04 0.0000000e+00 -1.2176461e-04"/>
+      <mass value="7.9119962e-02"/>
+      <inertia ixx="1.2505234e-05" ixy="0.0" ixz="-1.7855208e-07" iyy="2.1898364e-05" iyz="0.0" izz="1.9267361e-05"/>
     </inertial>
   </link>
@@ -28,5 +28,5 @@
     <origin xyz="0.012 0.0 0.017" rpy="0 0 0"/>
     <axis xyz="0 0 1"/>
-    <limit velocity="4.8" effort="1" lower="${-pi*0.9}" upper="${pi*0.9}" />
+    <limit velocity="4.8" effort="1" lower="${-pi*0.9}" upper="${pi*0.9}"/>
   </joint>
   <!--  Link 2 -->
@@ -46,7 +46,7 @@
     </collision>
     <inertial>
-      <origin xyz="-3.0184870e-04 5.4043684e-04 ${0.018 + 2.9433464e-02}" />
-      <mass value="9.8406837e-02" />
-      <inertia ixx="3.4543422e-05" ixy="-1.6031095e-08" ixz="-3.8375155e-07" iyy="3.2689329e-05" iyz="2.8511935e-08" izz="1.8850320e-05" />
+      <origin xyz="-3.0184870e-04 5.4043684e-04 ${0.018 + 2.9433464e-02}"/>
+      <mass value="9.8406837e-02"/>
+      <inertia ixx="3.4543422e-05" ixy="-1.6031095e-08" ixz="-3.8375155e-07" iyy="3.2689329e-05" iyz="2.8511935e-08" izz="1.8850320e-05"/>
     </inertial>
   </link>
@@ -57,5 +57,5 @@
     <origin xyz="0.0 0.0 0.0595" rpy="0 0 0"/>
     <axis xyz="0 1 0"/>
-    <limit velocity="4.8" effort="1" lower="${-pi*0.57}" upper="${pi*0.5}" />
+    <limit velocity="4.8" effort="1" lower="${-pi*0.57}" upper="${pi*0.5}"/>
   </joint>
   <!--  Link 3 -->
@@ -75,7 +75,7 @@
     </collision>
     <inertial>
-      <origin xyz="1.0308393e-02 3.7743363e-04 1.0170197e-01" />
-      <mass value="1.3850917e-01" />
-      <inertia ixx="3.3055381e-04" ixy="-9.7940978e-08" ixz="-3.8505711e-05" iyy="3.4290447e-04" iyz="-1.5717516e-06" izz="6.0346498e-05" />
+      <origin xyz="1.0308393e-02 3.7743363e-04 1.0170197e-01"/>
+      <mass value="1.3850917e-01"/>
+      <inertia ixx="3.3055381e-04" ixy="-9.7940978e-08" ixz="-3.8505711e-05" iyy="3.4290447e-04" iyz="-1.5717516e-06" izz="6.0346498e-05"/>
     </inertial>
   </link>
@@ -86,5 +86,5 @@
     <origin xyz="0.024 0 0.128" rpy="0 0 0"/>
     <axis xyz="0 1 0"/>
-    <limit velocity="4.8" effort="1" lower="${-pi*0.3}" upper="${pi*0.44}" />
+    <limit velocity="4.8" effort="1" lower="${-pi*0.3}" upper="${pi*0.44}"/>
   </joint>
   <!--  Link 4 -->
@@ -104,7 +104,7 @@
     </collision>
     <inertial>
-      <origin xyz="9.0909590e-02 3.8929816e-04 2.2413279e-04" />
-      <mass value="1.3274562e-01" />
-      <inertia ixx="3.0654178e-05" ixy="-1.2764155e-06" ixz="-2.6874417e-07" iyy="2.4230292e-04" iyz="1.1559550e-08" izz="2.5155057e-04" />
+      <origin xyz="9.0909590e-02 3.8929816e-04 2.2413279e-04"/>
+      <mass value="1.3274562e-01"/>
+      <inertia ixx="3.0654178e-05" ixy="-1.2764155e-06" ixz="-2.6874417e-07" iyy="2.4230292e-04" iyz="1.1559550e-08" izz="2.5155057e-04"/>
     </inertial>
   </link>
@@ -115,5 +115,5 @@
     <origin xyz="0.124 0.0 0.0" rpy="0 0 0"/>
     <axis xyz="0 1 0"/>
-    <limit velocity="4.8" effort="1" lower="${-pi*0.57}" upper="${pi*0.65}" />
+    <limit velocity="4.8" effort="1" lower="${-pi*0.57}" upper="${pi*0.65}"/>
   </joint>
   <!--  Link 5 -->
@@ -133,7 +133,7 @@
     </collision>
     <inertial>
-      <origin xyz="4.4206755e-02 3.6839985e-07 8.9142216e-03" />
-      <mass value="1.4327573e-01" />
-      <inertia ixx="8.0870749e-05" ixy="0.0" ixz="-1.0157896e-06" iyy="7.5980465e-05" iyz="0.0" izz="9.3127351e-05" />
+      <origin xyz="4.4206755e-02 3.6839985e-07 8.9142216e-03"/>
+      <mass value="1.4327573e-01"/>
+      <inertia ixx="8.0870749e-05" ixy="0.0" ixz="-1.0157896e-06" iyy="7.5980465e-05" iyz="0.0" izz="9.3127351e-05"/>
     </inertial>
   </link>
@@ -144,5 +144,5 @@
     <origin xyz="0.0817 0.021 0.0" rpy="0 0 0"/>
     <axis xyz="0 1 0"/>
-    <limit velocity="4.8" effort="1" lower="-0.010" upper="0.019" />
+    <limit velocity="4.8" effort="1" lower="-0.010" upper="0.019"/>
   </joint>
   <!--  Gripper link -->
@@ -162,7 +162,7 @@
     </collision>
     <inertial>
-      <origin xyz="0 0 0" />
-      <mass value="1.0e-03" />
-      <inertia ixx="1.0e-03" ixy="0.0" ixz="0.0" iyy="1.0e-03" iyz="0.0" izz="1.0e-03" />
+      <origin xyz="0 0 0"/>
+      <mass value="1.0e-03"/>
+      <inertia ixx="1.0e-03" ixy="0.0" ixz="0.0" iyy="1.0e-03" iyz="0.0" izz="1.0e-03"/>
     </inertial>
   </link>
@@ -173,5 +173,5 @@
     <origin xyz="0.0817 -0.021 0" rpy="0 0 0"/>
     <axis xyz="0 -1 0"/>
-    <limit velocity="4.8" effort="1" lower="-0.010" upper="0.019" />
+    <limit velocity="4.8" effort="1" lower="-0.010" upper="0.019"/>
     <mimic joint="rmx52/gripper" multiplier="1"/>
   </joint>
@@ -192,7 +192,7 @@
     </collision>
     <inertial>
-      <origin xyz="0 0 0" />
-      <mass value="1.0e-03" />
-      <inertia ixx="1.0e-03" ixy="0.0" ixz="0.0" iyy="1.0e-03" iyz="0.0" izz="1.0e-03" />
+      <origin xyz="0 0 0"/>
+      <mass value="1.0e-03"/>
+      <inertia ixx="1.0e-03" ixy="0.0" ixz="0.0" iyy="1.0e-03" iyz="0.0" izz="1.0e-03"/>
     </inertial>
   </link>
@@ -208,12 +208,12 @@
       <origin xyz="0 0 0" rpy="0 0 0"/>
       <geometry>
-        <box size="0.01 0.01 0.01" />
+        <box size="0.01 0.01 0.01"/>
       </geometry>
       <xacro:insert_block name="red"/>
     </visual>
     <inertial>
-      <origin xyz="0 0 0" />
-      <mass value="1.0e-03" />
-      <inertia ixx="1.0e-03" ixy="0.0" ixz="0.0" iyy="1.0e-03" iyz="0.0" izz="1.0e-03" />
+      <origin xyz="0 0 0"/>
+      <mass value="1.0e-03"/>
+      <inertia ixx="1.0e-03" ixy="0.0" ixz="0.0" iyy="1.0e-03" iyz="0.0" izz="1.0e-03"/>
     </inertial>
   </link>
