Commit message: 各関節に静止摩擦力を設定

File: tobas_description/urdf/components/rmx52/urdf.xacro (robot description, xacro)
@@ -6,12 +6,12 @@
       <origin xyz="0 0 0" rpy="0 0 0"/>
       <geometry>
-        <mesh filename="package://tobas_description/meshes/rmx52/chain_link1.stl" scale="0.001 0.001 0.001"/>
-      </geometry>
-      <xacro:insert_block name="gray"/>
-    </visual>
-    <collision>
-      <origin xyz="0 0 0" rpy="0 0 0"/>
-      <geometry>
-        <mesh filename="package://tobas_description/meshes/rmx52/chain_link1.stl" scale="0.001 0.001 0.001"/>
+        <mesh filename="package://tobas_description/meshes/rmx52/chain_link1.stl" scale="1e-3 1e-3 1e-3"/>
+      </geometry>
+      <xacro:insert_block name="gray"/>
+    </visual>
+    <collision>
+      <origin xyz="0 0 0" rpy="0 0 0"/>
+      <geometry>
+        <mesh filename="package://tobas_description/meshes/rmx52/chain_link1.stl" scale="1e-3 1e-3 1e-3"/>
       </geometry>
     </collision>
@@ -29,4 +29,5 @@
     <axis xyz="0 0 1"/>
     <limit velocity="4.8" effort="1" lower="${-pi*0.9}" upper="${pi*0.9}"/>
+    <dynamics damping="0" friction="0.01"/>
   </joint>
   <!--  Link 2 -->
@@ -35,5 +36,5 @@
       <origin xyz="0 0 0.019" rpy="0 0 0"/>
       <geometry>
-        <mesh filename="package://tobas_description/meshes/rmx52/chain_link2.stl" scale="0.001 0.001 0.001"/>
+        <mesh filename="package://tobas_description/meshes/rmx52/chain_link2.stl" scale="1e-3 1e-3 1e-3"/>
       </geometry>
       <xacro:insert_block name="gray"/>
@@ -42,5 +43,5 @@
       <origin xyz="0 0 0.019" rpy="0 0 0"/>
       <geometry>
-        <mesh filename="package://tobas_description/meshes/rmx52/chain_link2.stl" scale="0.001 0.001 0.001"/>
+        <mesh filename="package://tobas_description/meshes/rmx52/chain_link2.stl" scale="1e-3 1e-3 1e-3"/>
       </geometry>
     </collision>
@@ -58,4 +59,5 @@
     <axis xyz="0 1 0"/>
     <limit velocity="4.8" effort="1" lower="${-pi*0.57}" upper="${pi*0.5}"/>
+    <dynamics damping="0" friction="0.01"/>
   </joint>
   <!--  Link 3 -->
@@ -64,12 +66,12 @@
       <origin xyz="0 0 0" rpy="0 0 0"/>
       <geometry>
-        <mesh filename="package://tobas_description/meshes/rmx52/chain_link3.stl" scale="0.001 0.001 0.001"/>
-      </geometry>
-      <xacro:insert_block name="gray"/>
-    </visual>
-    <collision>
-      <origin xyz="0 0 0" rpy="0 0 0"/>
-      <geometry>
-        <mesh filename="package://tobas_description/meshes/rmx52/chain_link3.stl" scale="0.001 0.001 0.001"/>
+        <mesh filename="package://tobas_description/meshes/rmx52/chain_link3.stl" scale="1e-3 1e-3 1e-3"/>
+      </geometry>
+      <xacro:insert_block name="gray"/>
+    </visual>
+    <collision>
+      <origin xyz="0 0 0" rpy="0 0 0"/>
+      <geometry>
+        <mesh filename="package://tobas_description/meshes/rmx52/chain_link3.stl" scale="1e-3 1e-3 1e-3"/>
       </geometry>
     </collision>
@@ -87,4 +89,5 @@
     <axis xyz="0 1 0"/>
     <limit velocity="4.8" effort="1" lower="${-pi*0.3}" upper="${pi*0.44}"/>
+    <dynamics damping="0" friction="0.01"/>
   </joint>
   <!--  Link 4 -->
@@ -93,12 +96,12 @@
       <origin xyz="0 0 0" rpy="0 0 0"/>
       <geometry>
-        <mesh filename="package://tobas_description/meshes/rmx52/chain_link4.stl" scale="0.001 0.001 0.001"/>
-      </geometry>
-      <xacro:insert_block name="gray"/>
-    </visual>
-    <collision>
-      <origin xyz="0 0 0" rpy="0 0 0"/>
-      <geometry>
-        <mesh filename="package://tobas_description/meshes/rmx52/chain_link4.stl" scale="0.001 0.001 0.001"/>
+        <mesh filename="package://tobas_description/meshes/rmx52/chain_link4.stl" scale="1e-3 1e-3 1e-3"/>
+      </geometry>
+      <xacro:insert_block name="gray"/>
+    </visual>
+    <collision>
+      <origin xyz="0 0 0" rpy="0 0 0"/>
+      <geometry>
+        <mesh filename="package://tobas_description/meshes/rmx52/chain_link4.stl" scale="1e-3 1e-3 1e-3"/>
       </geometry>
     </collision>
@@ -116,4 +119,5 @@
     <axis xyz="0 1 0"/>
     <limit velocity="4.8" effort="1" lower="${-pi*0.57}" upper="${pi*0.65}"/>
+    <dynamics damping="0" friction="0.01"/>
   </joint>
   <!--  Link 5 -->
@@ -122,12 +126,12 @@
       <origin xyz="0 0 0" rpy="0 0 0"/>
       <geometry>
-        <mesh filename="package://tobas_description/meshes/rmx52/chain_link5.stl" scale="0.001 0.001 0.001"/>
-      </geometry>
-      <xacro:insert_block name="gray"/>
-    </visual>
-    <collision>
-      <origin xyz="0 0 0" rpy="0 0 0"/>
-      <geometry>
-        <mesh filename="package://tobas_description/meshes/rmx52/chain_link5.stl" scale="0.001 0.001 0.001"/>
+        <mesh filename="package://tobas_description/meshes/rmx52/chain_link5.stl" scale="1e-3 1e-3 1e-3"/>
+      </geometry>
+      <xacro:insert_block name="gray"/>
+    </visual>
+    <collision>
+      <origin xyz="0 0 0" rpy="0 0 0"/>
+      <geometry>
+        <mesh filename="package://tobas_description/meshes/rmx52/chain_link5.stl" scale="1e-3 1e-3 1e-3"/>
       </geometry>
     </collision>
@@ -145,4 +149,5 @@
     <axis xyz="0 1 0"/>
     <limit velocity="4.8" effort="1" lower="-0.010" upper="0.019"/>
+    <dynamics damping="0" friction="1e-4"/>
   </joint>
   <!--  Gripper link -->
@@ -151,5 +156,5 @@
       <origin xyz="0.0 0.0 0" rpy="0 0 0"/>
       <geometry>
-        <mesh filename="package://tobas_description/meshes/rmx52/chain_link_grip_l.stl" scale="0.001 0.001 0.001"/>
+        <mesh filename="package://tobas_description/meshes/rmx52/chain_link_grip_l.stl" scale="1e-3 1e-3 1e-3"/>
       </geometry>
       <xacro:insert_block name="gray"/>
@@ -158,5 +163,5 @@
       <origin xyz="0.0 0.0 0" rpy="0 0 0"/>
       <geometry>
-        <mesh filename="package://tobas_description/meshes/rmx52/chain_link_grip_l.stl" scale="0.001 0.001 0.001"/>
+        <mesh filename="package://tobas_description/meshes/rmx52/chain_link_grip_l.stl" scale="1e-3 1e-3 1e-3"/>
       </geometry>
     </collision>
@@ -174,4 +179,5 @@
     <axis xyz="0 -1 0"/>
     <limit velocity="4.8" effort="1" lower="-0.010" upper="0.019"/>
+    <dynamics damping="0" friction="1e-4"/>
     <mimic joint="rmx52/gripper" multiplier="1"/>
   </joint>
@@ -181,5 +187,5 @@
       <origin xyz="0.0 -0.0 0" rpy="0 0 0"/>
       <geometry>
-        <mesh filename="package://tobas_description/meshes/rmx52/chain_link_grip_r.stl" scale="0.001 0.001 0.001"/>
+        <mesh filename="package://tobas_description/meshes/rmx52/chain_link_grip_r.stl" scale="1e-3 1e-3 1e-3"/>
       </geometry>
       <xacro:insert_block name="gray"/>
@@ -188,5 +194,5 @@
       <origin xyz="0.0 -0.0 0" rpy="0 0 0"/>
       <geometry>
-        <mesh filename="package://tobas_description/meshes/rmx52/chain_link_grip_r.stl" scale="0.001 0.001 0.001"/>
+        <mesh filename="package://tobas_description/meshes/rmx52/chain_link_grip_r.stl" scale="1e-3 1e-3 1e-3"/>
       </geometry>
     </collision>

Commit message: gripper jointの最大速度を変更

File: tobas_description/urdf/components/rmx52/urdf.xacro (robot description, xacro)
@@ -148,5 +148,5 @@
     <origin xyz="0.0817 0.021 0.0" rpy="0 0 0"/>
     <axis xyz="0 1 0"/>
-    <limit velocity="4.8" effort="1" lower="-0.010" upper="0.019"/>
+    <limit velocity="0.1" effort="1" lower="-0.010" upper="0.019"/>
     <dynamics damping="0" friction="1e-4"/>
   </joint>
@@ -178,5 +178,5 @@
     <origin xyz="0.0817 -0.021 0" rpy="0 0 0"/>
     <axis xyz="0 -1 0"/>
-    <limit velocity="4.8" effort="1" lower="-0.010" upper="0.019"/>
+    <limit velocity="0.1" effort="1" lower="-0.010" upper="0.019"/>
     <dynamics damping="0" friction="1e-4"/>
     <mimic joint="rmx52/gripper" multiplier="1"/>
