Commit message: edit: hydrus/link.xacro

File: tobas_description/urdf/components/hydrus/link.xacro (robot description, xacro)
@@ -172,5 +172,6 @@
         <origin rpy="0 0 0" xyz="${link_length* 0.5} 0 0.013"/>
       </xacro:unless>
-      <axis xyz="0 0 ${rotor_direction}"/>
+      <!-- <axis xyz="0 0 ${rotor_direction}"/> -->
+      <axis xyz="0 0 1"/>
     </joint>
     <link name="thrust${self}">
@@ -268,9 +269,9 @@
       <!-- dummy root link for KDL -->
       <link name="root">
-        <inertial>
+        <!-- <inertial>
           <origin xyz="0 0 0" rpy="0 0 0"/>
           <mass value="0.00001"/>
           <inertia ixx="0.000001" ixy="0.0" ixz="0.0" iyy="0.000001" iyz="0.0" izz="0.000002"/>
-        </inertial>
+        </inertial> -->
       </link>
       <joint name="root_joint" type="fixed">

Commit message: edit: link.xacro

File: tobas_description/urdf/components/hydrus/link.xacro (robot description, xacro)
@@ -267,12 +267,5 @@
     </xacro:unless>
     <xacro:if value="${self == 1}">
-      <!-- dummy root link for KDL -->
-      <link name="root">
-        <!-- <inertial>
-          <origin xyz="0 0 0" rpy="0 0 0"/>
-          <mass value="0.00001"/>
-          <inertia ixx="0.000001" ixy="0.0" ixz="0.0" iyy="0.000001" iyz="0.0" izz="0.000002"/>
-        </inertial> -->
-      </link>
+      <link name="root"/>
       <joint name="root_joint" type="fixed">
         <parent link="root"/>
@@ -287,9 +280,7 @@
         <type>transmission_interface/SimpleTransmission</type>
         <joint name="joint${self}">
-          <!-- TODO: effort is torque, maybe position is enough -->
           <hardwareInterface>hardware_interface/EffortJointInterface</hardwareInterface>
         </joint>
         <actuator name="servo{self}">
-          <!-- TODO: effort is torque, maybe position is enough -->
           <hardwareInterface>hardware_interface/EffortJointInterface</hardwareInterface>
           <mechanicalReduction>1</mechanicalReduction>
@@ -297,16 +288,4 @@
       </transmission>
     </xacro:unless>
-    <transmission name="rotor_tran${self}">
-      <type>transmission_interface/SimpleTransmission</type>
-      <joint name="rotor${self}">
-        <!-- TODO: effort is torque, maybe position is enough -->
-        <hardwareInterface>RotorInterface</hardwareInterface>
-      </joint>
-      <actuator name="rotor${self}">
-        <!-- TODO: effort is torque, maybe position is enough -->
-        <hardwareInterface>RotorInterface</hardwareInterface>
-        <mechanicalReduction>1</mechanicalReduction>
-      </actuator>
-    </transmission>
     <xacro:friction self ="${self}"/>
   </xacro:macro>

Commit message: remove rotor limit

File: tobas_description/urdf/components/hydrus/link.xacro (robot description, xacro)
@@ -158,5 +158,4 @@
     <!-- rotor -->
     <joint name="rotor${self}" type="continuous">
-      <limit effort="100.0" lower="${min_force}" upper="${max_force}" velocity="0.5"/>
       <parent link="link${self}"/>
       <child link="thrust${self}"/>
