Commit message: update

File: tobas_example_packages/tobas_f550.TBS/tobas_f550_config/urdf/drone.xacro (robot description, xacro)
@@ -475,4 +475,10 @@
         </plugin>
     </gazebo>
+    <gazebo>
+        <plugin filename="tobas_gazebo_lookat_position_plugin" name="gazebo::GazeboLookAtPositionPlugin">
+            <robotNamespace>f550</robotNamespace>
+            <linkName>base_link</linkName>
+        </plugin>
+    </gazebo>
     <ros2_control name="GazeboSimSystem" type="system">
         <hardware>

File: tobas_example_packages/tobas_f550_np.TBS/backup/original.urdf (robot description, URDF)
Before this commit: robot f550_np, 9 links, 8 joints
Joints:
- joint propeller_0_joint: origin xyz=0.242082 0.130702 0.060597 rpy=0.523599 1.38778e-17 0.523599 -> xyz=0.242082 0.130702 0.060597 rpy=0.523599 2.77556e-17 0.523599
- joint propeller_1_joint: origin xyz=-0.007851 0.275 0.060597 rpy=-0.523599 -0 1.5708 -> xyz=-0.007851 0.275 0.060597 rpy=-0.523599 5.55112e-17 1.5708
- joint propeller_2_joint: origin xyz=-0.234232 0.144298 0.060597 rpy=0.523599 -1.38778e-17 2.61799 -> xyz=-0.234232 0.144298 0.060597 rpy=0.523599 2.77556e-17 2.61799
- joint propeller_3_joint: origin xyz=-0.234232 -0.144645 0.060597 rpy=-0.523599 -0 -2.61799 -> xyz=-0.234232 -0.144645 0.060597 rpy=-0.523599 2.77556e-17 -2.61799
- joint propeller_4_joint: origin xyz=-0.007851 -0.275 0.060597 rpy=0.523599 -0 -1.5708 -> xyz=-0.007851 -0.275 0.060597 rpy=0.523599 5.55112e-17 -1.5708
- joint propeller_5_joint: origin xyz=0.242082 -0.130355 0.060597 rpy=-0.523599 -0 -0.523599 -> xyz=0.242082 -0.130355 0.060597 rpy=-0.523599 2.77556e-17 -0.523599

File: tobas_example_packages/tobas_f550_np.TBS/tobas_f550_np_config/urdf/drone.xacro (robot description, xacro)
@@ -222,5 +222,5 @@
     </joint>
     <joint name="propeller_0_joint" type="continuous">
-        <origin xyz="0.242082 0.130702 0.060597" rpy="0.523599 1.38778e-17 0.523599"/>
+        <origin xyz="0.242082 0.130702 0.060597" rpy="0.523599 2.77556e-17 0.523599"/>
         <axis xyz="0 0 1"/>
         <parent link="base_link"/>
@@ -228,5 +228,5 @@
     </joint>
     <joint name="propeller_1_joint" type="continuous">
-        <origin xyz="-0.007851 0.275 0.060597" rpy="-0.523599 -0 1.5708"/>
+        <origin xyz="-0.007851 0.275 0.060597" rpy="-0.523599 5.55112e-17 1.5708"/>
         <axis xyz="0 0 1"/>
         <parent link="base_link"/>
@@ -234,5 +234,5 @@
     </joint>
     <joint name="propeller_2_joint" type="continuous">
-        <origin xyz="-0.234232 0.144298 0.060597" rpy="0.523599 -1.38778e-17 2.61799"/>
+        <origin xyz="-0.234232 0.144298 0.060597" rpy="0.523599 2.77556e-17 2.61799"/>
         <axis xyz="0 0 1"/>
         <parent link="base_link"/>
@@ -240,5 +240,5 @@
     </joint>
     <joint name="propeller_3_joint" type="continuous">
-        <origin xyz="-0.234232 -0.144645 0.060597" rpy="-0.523599 -0 -2.61799"/>
+        <origin xyz="-0.234232 -0.144645 0.060597" rpy="-0.523599 2.77556e-17 -2.61799"/>
         <axis xyz="0 0 1"/>
         <parent link="base_link"/>
@@ -246,5 +246,5 @@
     </joint>
     <joint name="propeller_4_joint" type="continuous">
-        <origin xyz="-0.007851 -0.275 0.060597" rpy="0.523599 -0 -1.5708"/>
+        <origin xyz="-0.007851 -0.275 0.060597" rpy="0.523599 5.55112e-17 -1.5708"/>
         <axis xyz="0 0 1"/>
         <parent link="base_link"/>
@@ -252,5 +252,5 @@
     </joint>
     <joint name="propeller_5_joint" type="continuous">
-        <origin xyz="0.242082 -0.130355 0.060597" rpy="-0.523599 -0 -0.523599"/>
+        <origin xyz="0.242082 -0.130355 0.060597" rpy="-0.523599 2.77556e-17 -0.523599"/>
         <axis xyz="0 0 1"/>
         <parent link="base_link"/>
@@ -442,4 +442,10 @@
         </plugin>
     </gazebo>
+    <gazebo>
+        <plugin filename="tobas_gazebo_lookat_position_plugin" name="gazebo::GazeboLookAtPositionPlugin">
+            <robotNamespace>f550_np</robotNamespace>
+            <linkName>base_link</linkName>
+        </plugin>
+    </gazebo>
     <ros2_control name="GazeboSimSystem" type="system">
         <hardware>

File: tobas_example_packages/tobas_truncated_octahedron.TBS/tobas_truncated_octahedron_config/urdf/drone.xacro (robot description, xacro)
@@ -787,4 +787,10 @@
         </plugin>
     </gazebo>
+    <gazebo>
+        <plugin filename="tobas_gazebo_lookat_position_plugin" name="gazebo::GazeboLookAtPositionPlugin">
+            <robotNamespace>truncated_octahedron</robotNamespace>
+            <linkName>base_link</linkName>
+        </plugin>
+    </gazebo>
     <ros2_control name="GazeboSimSystem" type="system">
         <hardware>
