Commit message: update: TOF package

File: tobas_example_packages/tobas_truncated_octahedron.TBS/backup/original.urdf (robot description, URDF)
Before this commit: robot truncated_octahedron, 20 links, 19 joints
Links:
- link motor_0: mass 0.053 -> 0.086; geometry collision cylinder length=0.024 radius=0.021; visual mesh filename=file:///home/dohi/colcon_ws_tobas/src/tobas/tobas_example_p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 scale=1 1 1
- link motor_1: mass 0.053 -> 0.086; geometry collision cylinder length=0.024 radius=0.021; visual mesh filename=file:///home/dohi/colcon_ws_tobas/src/tobas/tobas_example_p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 scale=1 1 1
- link motor_2: mass 0.053 -> 0.086; geometry collision cylinder length=0.024 radius=0.021; visual mesh filename=file:///home/dohi/colcon_ws_tobas/src/tobas/tobas_example_p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 scale=1 1 1
- link motor_3: mass 0.053 -> 0.086; geometry collision cylinder length=0.024 radius=0.021; visual mesh filename=file:///home/dohi/colcon_ws_tobas/src/tobas/tobas_example_p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 scale=1 1 1
- link motor_4: mass 0.053 -> 0.086; geometry collision cylinder length=0.024 radius=0.021; visual mesh filename=file:///home/dohi/colcon_ws_tobas/src/tobas/tobas_example_p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 scale=1 1 1
- link motor_5: mass 0.053 -> 0.086; geometry collision cylinder length=0.024 radius=0.021; visual mesh filename=file:///home/dohi/colcon_ws_tobas/src/tobas/tobas_example_p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 scale=1 1 1
- link motor_6: mass 0.053 -> 0.086; geometry collision cylinder length=0.024 radius=0.021; visual mesh filename=file:///home/dohi/colcon_ws_tobas/src/tobas/tobas_example_p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 scale=1 1 1
- link motor_7: mass 0.053 -> 0.086; geometry collision cylinder length=0.024 radius=0.021; visual mesh filename=file:///home/dohi/colcon_ws_tobas/src/tobas/tobas_example_p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 scale=1 1 1
Joints:
- joint propeller_0_joint: origin xyz=0 0 0.0245 rpy=0 -0 0 -> xyz=0 0 0.029 rpy=0 -0 0
- joint propeller_1_joint: origin xyz=0 0 0.0245 rpy=0 -0 0 -> xyz=0 0 0.029 rpy=0 -0 0
- joint propeller_2_joint: origin xyz=0 0 0.0245 rpy=0 -0 0 -> xyz=0 0 0.029 rpy=0 -0 0
- joint propeller_3_joint: origin xyz=0 0 0.0245 rpy=0 -0 0 -> xyz=0 0 0.029 rpy=0 -0 0
- joint propeller_4_joint: origin xyz=0 0 0.0245 rpy=0 -0 0 -> xyz=0 0 0.029 rpy=0 -0 0
- joint propeller_5_joint: origin xyz=0 0 0.0245 rpy=0 -0 0 -> xyz=0 0 0.029 rpy=0 -0 0
- joint propeller_6_joint: origin xyz=0 0 0.0245 rpy=0 -0 0 -> xyz=0 0 0.029 rpy=0 -0 0
- joint propeller_7_joint: origin xyz=0 0 0.0245 rpy=0 -0 0 -> xyz=0 0 0.029 rpy=0 -0 0

File: tobas_example_packages/tobas_truncated_octahedron.TBS/tobas_truncated_octahedron_config/urdf/drone.xacro (robot description, xacro)
@@ -3,4 +3,8 @@
         <texture/>
         <color rgba="0 0 0 1"/>
+    </material>
+    <material name="orange">
+        <texture/>
+        <color rgba="1 0.423529 0.0392157 1"/>
     </material>
     <material name="red">
@@ -88,22 +92,22 @@
     <link name="motor_0">
         <inertial>
-            <mass value="0.053"/>
-            <origin xyz="0 0 0.01225" rpy="0 -0 0"/>
-            <inertia ixx="5.2481e-06" ixy="0" ixz="0" iyy="5.2481e-06" iyz="0" izz="5.194e-06"/>
-        </inertial>
-        <visual>
-            <origin xyz="0 0 0" rpy="0 -0 0"/>
-            <geometry>
-                <mesh filename="file://$(find tobas_truncated_octahedron_config)/meshes/a2212_920kv.stl" scale="1 1 1"/>
-            </geometry>
-            <material name="red">
-                <texture/>
-                <color rgba="1 0 0 1"/>
-            </material>
-        </visual>
-        <collision>
-            <origin xyz="0 0 0.01225" rpy="0 -0 0"/>
-            <geometry>
-                <cylinder radius="0.014" length="0.0245"/>
+            <mass value="0.086"/>
+            <origin xyz="0 0 0.012" rpy="0 -0 0"/>
+            <inertia ixx="1.36095e-05" ixy="0" ixz="0" iyy="1.36095e-05" iyz="0" izz="1.8963e-05"/>
+        </inertial>
+        <visual>
+            <origin xyz="0 0 0" rpy="0 -0 0"/>
+            <geometry>
+                <mesh filename="file://$(find tobas_truncated_octahedron_config)/meshes/mt3508_580kv.stl" scale="1 1 1"/>
+            </geometry>
+            <material name="orange">
+                <texture/>
+                <color rgba="1 0.423529 0.0392157 1"/>
+            </material>
+        </visual>
+        <collision>
+            <origin xyz="0 0 0.012" rpy="0 -0 0"/>
+            <geometry>
+                <cylinder radius="0.021" length="0.024"/>
             </geometry>
         </collision>
@@ -111,22 +115,22 @@
     <link name="motor_1">
         <inertial>
-            <mass value="0.053"/>
-            <origin xyz="0 0 0.01225" rpy="0 -0 0"/>
-            <inertia ixx="5.2481e-06" ixy="0" ixz="0" iyy="5.2481e-06" iyz="0" izz="5.194e-06"/>
-        </inertial>
-        <visual>
-            <origin xyz="0 0 0" rpy="0 -0 0"/>
-            <geometry>
-                <mesh filename="file://$(find tobas_truncated_octahedron_config)/meshes/a2212_920kv.stl" scale="1 1 1"/>
-            </geometry>
-            <material name="red">
-                <texture/>
-                <color rgba="1 0 0 1"/>
-            </material>
-        </visual>
-        <collision>
-            <origin xyz="0 0 0.01225" rpy="0 -0 0"/>
-            <geometry>
-                <cylinder radius="0.014" length="0.0245"/>
+            <mass value="0.086"/>
+            <origin xyz="0 0 0.012" rpy="0 -0 0"/>
+            <inertia ixx="1.36095e-05" ixy="0" ixz="0" iyy="1.36095e-05" iyz="0" izz="1.8963e-05"/>
+        </inertial>
+        <visual>
+            <origin xyz="0 0 0" rpy="0 -0 0"/>
+            <geometry>
+                <mesh filename="file://$(find tobas_truncated_octahedron_config)/meshes/mt3508_580kv.stl" scale="1 1 1"/>
+            </geometry>
+            <material name="orange">
+                <texture/>
+                <color rgba="1 0.423529 0.0392157 1"/>
+            </material>
+        </visual>
+        <collision>
+            <origin xyz="0 0 0.012" rpy="0 -0 0"/>
+            <geometry>
+                <cylinder radius="0.021" length="0.024"/>
             </geometry>
         </collision>
@@ -134,22 +138,22 @@
     <link name="motor_2">
         <inertial>
-            <mass value="0.053"/>
-            <origin xyz="0 0 0.01225" rpy="0 -0 0"/>
-            <inertia ixx="5.2481e-06" ixy="0" ixz="0" iyy="5.2481e-06" iyz="0" izz="5.194e-06"/>
-        </inertial>
-        <visual>
-            <origin xyz="0 0 0" rpy="0 -0 0"/>
-            <geometry>
-                <mesh filename="file://$(find tobas_truncated_octahedron_config)/meshes/a2212_920kv.stl" scale="1 1 1"/>
-            </geometry>
-            <material name="red">
-                <texture/>
-                <color rgba="1 0 0 1"/>
-            </material>
-        </visual>
-        <collision>
-            <origin xyz="0 0 0.01225" rpy="0 -0 0"/>
-            <geometry>
-                <cylinder radius="0.014" length="0.0245"/>
+            <mass value="0.086"/>
+            <origin xyz="0 0 0.012" rpy="0 -0 0"/>
+            <inertia ixx="1.36095e-05" ixy="0" ixz="0" iyy="1.36095e-05" iyz="0" izz="1.8963e-05"/>
+        </inertial>
+        <visual>
+            <origin xyz="0 0 0" rpy="0 -0 0"/>
+            <geometry>
+                <mesh filename="file://$(find tobas_truncated_octahedron_config)/meshes/mt3508_580kv.stl" scale="1 1 1"/>
+            </geometry>
+            <material name="orange">
+                <texture/>
+                <color rgba="1 0.423529 0.0392157 1"/>
+            </material>
+        </visual>
+        <collision>
+            <origin xyz="0 0 0.012" rpy="0 -0 0"/>
+            <geometry>
+                <cylinder radius="0.021" length="0.024"/>
             </geometry>
         </collision>
@@ -157,22 +161,22 @@
     <link name="motor_3">
         <inertial>
-            <mass value="0.053"/>
-            <origin xyz="0 0 0.01225" rpy="0 -0 0"/>
-            <inertia ixx="5.2481e-06" ixy="0" ixz="0" iyy="5.2481e-06" iyz="0" izz="5.194e-06"/>
-        </inertial>
-        <visual>
-            <origin xyz="0 0 0" rpy="0 -0 0"/>
-            <geometry>
-                <mesh filename="file://$(find tobas_truncated_octahedron_config)/meshes/a2212_920kv.stl" scale="1 1 1"/>
-            </geometry>
-            <material name="red">
-                <texture/>
-                <color rgba="1 0 0 1"/>
-            </material>
-        </visual>
-        <collision>
-            <origin xyz="0 0 0.01225" rpy="0 -0 0"/>
-            <geometry>
-                <cylinder radius="0.014" length="0.0245"/>
+            <mass value="0.086"/>
+            <origin xyz="0 0 0.012" rpy="0 -0 0"/>
+            <inertia ixx="1.36095e-05" ixy="0" ixz="0" iyy="1.36095e-05" iyz="0" izz="1.8963e-05"/>
+        </inertial>
+        <visual>
+            <origin xyz="0 0 0" rpy="0 -0 0"/>
+            <geometry>
+                <mesh filename="file://$(find tobas_truncated_octahedron_config)/meshes/mt3508_580kv.stl" scale="1 1 1"/>
+            </geometry>
+            <material name="orange">
+                <texture/>
+                <color rgba="1 0.423529 0.0392157 1"/>
+            </material>
+        </visual>
+        <collision>
+            <origin xyz="0 0 0.012" rpy="0 -0 0"/>
+            <geometry>
+                <cylinder radius="0.021" length="0.024"/>
             </geometry>
         </collision>
@@ -180,22 +184,22 @@
     <link name="motor_4">
         <inertial>
-            <mass value="0.053"/>
-            <origin xyz="0 0 0.01225" rpy="0 -0 0"/>
-            <inertia ixx="5.2481e-06" ixy="0" ixz="0" iyy="5.2481e-06" iyz="0" izz="5.194e-06"/>
-        </inertial>
-        <visual>
-            <origin xyz="0 0 0" rpy="0 -0 0"/>
-            <geometry>
-                <mesh filename="file://$(find tobas_truncated_octahedron_config)/meshes/a2212_920kv.stl" scale="1 1 1"/>
-            </geometry>
-            <material name="red">
-                <texture/>
-                <color rgba="1 0 0 1"/>
-            </material>
-        </visual>
-        <collision>
-            <origin xyz="0 0 0.01225" rpy="0 -0 0"/>
-            <geometry>
-                <cylinder radius="0.014" length="0.0245"/>
+            <mass value="0.086"/>
+            <origin xyz="0 0 0.012" rpy="0 -0 0"/>
+            <inertia ixx="1.36095e-05" ixy="0" ixz="0" iyy="1.36095e-05" iyz="0" izz="1.8963e-05"/>
+        </inertial>
+        <visual>
+            <origin xyz="0 0 0" rpy="0 -0 0"/>
+            <geometry>
+                <mesh filename="file://$(find tobas_truncated_octahedron_config)/meshes/mt3508_580kv.stl" scale="1 1 1"/>
+            </geometry>
+            <material name="orange">
+                <texture/>
+                <color rgba="1 0.423529 0.0392157 1"/>
+            </material>
+        </visual>
+        <collision>
+            <origin xyz="0 0 0.012" rpy="0 -0 0"/>
+            <geometry>
+                <cylinder radius="0.021" length="0.024"/>
             </geometry>
         </collision>
@@ -203,22 +207,22 @@
     <link name="motor_5">
         <inertial>
-            <mass value="0.053"/>
-            <origin xyz="0 0 0.01225" rpy="0 -0 0"/>
-            <inertia ixx="5.2481e-06" ixy="0" ixz="0" iyy="5.2481e-06" iyz="0" izz="5.194e-06"/>
-        </inertial>
-        <visual>
-            <origin xyz="0 0 0" rpy="0 -0 0"/>
-            <geometry>
-                <mesh filename="file://$(find tobas_truncated_octahedron_config)/meshes/a2212_920kv.stl" scale="1 1 1"/>
-            </geometry>
-            <material name="red">
-                <texture/>
-                <color rgba="1 0 0 1"/>
-            </material>
-        </visual>
-        <collision>
-            <origin xyz="0 0 0.01225" rpy="0 -0 0"/>
-            <geometry>
-                <cylinder radius="0.014" length="0.0245"/>
+            <mass value="0.086"/>
+            <origin xyz="0 0 0.012" rpy="0 -0 0"/>
+            <inertia ixx="1.36095e-05" ixy="0" ixz="0" iyy="1.36095e-05" iyz="0" izz="1.8963e-05"/>
+        </inertial>
+        <visual>
+            <origin xyz="0 0 0" rpy="0 -0 0"/>
+            <geometry>
+                <mesh filename="file://$(find tobas_truncated_octahedron_config)/meshes/mt3508_580kv.stl" scale="1 1 1"/>
+            </geometry>
+            <material name="orange">
+                <texture/>
+                <color rgba="1 0.423529 0.0392157 1"/>
+            </material>
+        </visual>
+        <collision>
+            <origin xyz="0 0 0.012" rpy="0 -0 0"/>
+            <geometry>
+                <cylinder radius="0.021" length="0.024"/>
             </geometry>
         </collision>
@@ -226,22 +230,22 @@
     <link name="motor_6">
         <inertial>
-            <mass value="0.053"/>
-            <origin xyz="0 0 0.01225" rpy="0 -0 0"/>
-            <inertia ixx="5.2481e-06" ixy="0" ixz="0" iyy="5.2481e-06" iyz="0" izz="5.194e-06"/>
-        </inertial>
-        <visual>
-            <origin xyz="0 0 0" rpy="0 -0 0"/>
-            <geometry>
-                <mesh filename="file://$(find tobas_truncated_octahedron_config)/meshes/a2212_920kv.stl" scale="1 1 1"/>
-            </geometry>
-            <material name="red">
-                <texture/>
-                <color rgba="1 0 0 1"/>
-            </material>
-        </visual>
-        <collision>
-            <origin xyz="0 0 0.01225" rpy="0 -0 0"/>
-            <geometry>
-                <cylinder radius="0.014" length="0.0245"/>
+            <mass value="0.086"/>
+            <origin xyz="0 0 0.012" rpy="0 -0 0"/>
+            <inertia ixx="1.36095e-05" ixy="0" ixz="0" iyy="1.36095e-05" iyz="0" izz="1.8963e-05"/>
+        </inertial>
+        <visual>
+            <origin xyz="0 0 0" rpy="0 -0 0"/>
+            <geometry>
+                <mesh filename="file://$(find tobas_truncated_octahedron_config)/meshes/mt3508_580kv.stl" scale="1 1 1"/>
+            </geometry>
+            <material name="orange">
+                <texture/>
+                <color rgba="1 0.423529 0.0392157 1"/>
+            </material>
+        </visual>
+        <collision>
+            <origin xyz="0 0 0.012" rpy="0 -0 0"/>
+            <geometry>
+                <cylinder radius="0.021" length="0.024"/>
             </geometry>
         </collision>
@@ -249,22 +253,22 @@
     <link name="motor_7">
         <inertial>
-            <mass value="0.053"/>
-            <origin xyz="0 0 0.01225" rpy="0 -0 0"/>
-            <inertia ixx="5.2481e-06" ixy="0" ixz="0" iyy="5.2481e-06" iyz="0" izz="5.194e-06"/>
-        </inertial>
-        <visual>
-            <origin xyz="0 0 0" rpy="0 -0 0"/>
-            <geometry>
-                <mesh filename="file://$(find tobas_truncated_octahedron_config)/meshes/a2212_920kv.stl" scale="1 1 1"/>
-            </geometry>
-            <material name="red">
-                <texture/>
-                <color rgba="1 0 0 1"/>
-            </material>
-        </visual>
-        <collision>
-            <origin xyz="0 0 0.01225" rpy="0 -0 0"/>
-            <geometry>
-                <cylinder radius="0.014" length="0.0245"/>
+            <mass value="0.086"/>
+            <origin xyz="0 0 0.012" rpy="0 -0 0"/>
+            <inertia ixx="1.36095e-05" ixy="0" ixz="0" iyy="1.36095e-05" iyz="0" izz="1.8963e-05"/>
+        </inertial>
+        <visual>
+            <origin xyz="0 0 0" rpy="0 -0 0"/>
+            <geometry>
+                <mesh filename="file://$(find tobas_truncated_octahedron_config)/meshes/mt3508_580kv.stl" scale="1 1 1"/>
+            </geometry>
+            <material name="orange">
+                <texture/>
+                <color rgba="1 0.423529 0.0392157 1"/>
+            </material>
+        </visual>
+        <collision>
+            <origin xyz="0 0 0.012" rpy="0 -0 0"/>
+            <geometry>
+                <cylinder radius="0.021" length="0.024"/>
             </geometry>
         </collision>
@@ -521,5 +525,5 @@
     </joint>
     <joint name="propeller_0_joint" type="continuous">
-        <origin xyz="0 0 0.0245" rpy="0 -0 0"/>
+        <origin xyz="0 0 0.029" rpy="0 -0 0"/>
         <axis xyz="0 0 1"/>
         <parent link="motor_0"/>
@@ -527,5 +531,5 @@
     </joint>
     <joint name="propeller_1_joint" type="continuous">
-        <origin xyz="0 0 0.0245" rpy="0 -0 0"/>
+        <origin xyz="0 0 0.029" rpy="0 -0 0"/>
         <axis xyz="0 0 1"/>
         <parent link="motor_1"/>
@@ -533,5 +537,5 @@
     </joint>
     <joint name="propeller_2_joint" type="continuous">
-        <origin xyz="0 0 0.0245" rpy="0 -0 0"/>
+        <origin xyz="0 0 0.029" rpy="0 -0 0"/>
         <axis xyz="0 0 1"/>
         <parent link="motor_2"/>
@@ -539,5 +543,5 @@
     </joint>
     <joint name="propeller_3_joint" type="continuous">
-        <origin xyz="0 0 0.0245" rpy="0 -0 0"/>
+        <origin xyz="0 0 0.029" rpy="0 -0 0"/>
         <axis xyz="0 0 1"/>
         <parent link="motor_3"/>
@@ -545,5 +549,5 @@
     </joint>
     <joint name="propeller_4_joint" type="continuous">
-        <origin xyz="0 0 0.0245" rpy="0 -0 0"/>
+        <origin xyz="0 0 0.029" rpy="0 -0 0"/>
         <axis xyz="0 0 1"/>
         <parent link="motor_4"/>
@@ -551,5 +555,5 @@
     </joint>
     <joint name="propeller_5_joint" type="continuous">
-        <origin xyz="0 0 0.0245" rpy="0 -0 0"/>
+        <origin xyz="0 0 0.029" rpy="0 -0 0"/>
         <axis xyz="0 0 1"/>
         <parent link="motor_5"/>
@@ -557,5 +561,5 @@
     </joint>
     <joint name="propeller_6_joint" type="continuous">
-        <origin xyz="0 0 0.0245" rpy="0 -0 0"/>
+        <origin xyz="0 0 0.029" rpy="0 -0 0"/>
         <axis xyz="0 0 1"/>
         <parent link="motor_6"/>
@@ -563,5 +567,5 @@
     </joint>
     <joint name="propeller_7_joint" type="continuous">
-        <origin xyz="0 0 0.0245" rpy="0 -0 0"/>
+        <origin xyz="0 0 0.029" rpy="0 -0 0"/>
         <axis xyz="0 0 1"/>
         <parent link="motor_7"/>
@@ -659,5 +663,5 @@
             <robotNamespace>truncated_octahedron</robotNamespace>
             <linkName>propeller_0</linkName>
-            <kv>96.342174710086979</kv>
+            <kv>60.737457969402662</kv>
             <internalResistance>0.25</internalResistance>
             <numberOfBlades>2</numberOfBlades>
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