Commit message: fix

File: tobas_description/urdf/components/landing_gear/zhizicathy_electric_150.xacro (robot description, xacro)
@@ -61,5 +61,5 @@
         <mass value="0.0706"/>
         <origin xyz="0 0.029 -0.142" rpy="0 0 0"/>
-        <inertia ixx="2.169e-4" ixy="0" ixz="0" iyy="4.320e-4" iyz="0" izz="2.437e-4"/>
+        <inertia ixx="2.169e-4" ixy="0" ixz="0" iyy="4.320e-4" iyz="4.968e-5" izz="2.437e-4"/>
       </inertial>
     </link>

Commit message: .

File: tobas_description/urdf/components/landing_gear/zhizicathy_electric_150.xacro (robot description, xacro)
@@ -1,5 +1,5 @@
 <robot xmlns:xacro="http://ros.org/wiki/xacro">
   <xacro:include filename="$(find tobas_description)/urdf/components/dummy.xacro"/>
-  <xacro:macro name="landing_gear" params="offset direction reverse suffix">
+  <xacro:macro name="landing_gear" params="offset max_angle direction reverse suffix">
     <joint name="lg_${suffix}_top_joint" type="fixed">
       <origin xyz="0 ${direction*offset} 0" rpy="0 0 ${reverse*pi}"/>
@@ -35,5 +35,5 @@
       <child link="lg_${suffix}_bottom"/>
       <axis xyz="1 0 0"/>
-      <limit velocity="${75*deg2rad/6}" effort="1" lower="0" upper="${75*deg2rad}"/>
+      <limit velocity="${75*deg2rad/6}" effort="1" lower="0" upper="${max_angle}"/>
       <dynamics damping="0" friction="0.01"/>
     </joint>
@@ -65,5 +65,5 @@
     </link>
   </xacro:macro>
-  <xacro:macro name="zhizicathy_electric_150" params="parent distance *origin">
+  <xacro:macro name="zhizicathy_electric_150" params="parent distance max_angle *origin">
     <joint name="lg_base_joint" type="fixed">
       <xacro:insert_block name="origin"/>
@@ -72,6 +72,6 @@
     </joint>
     <xacro:dummy_inertial_link name="lg_base_link"/>
-    <xacro:landing_gear offset="${distance/2}" direction="1" reverse="0" suffix="left"/>
-    <xacro:landing_gear offset="${distance/2}" direction="-1" reverse="1" suffix="right"/>
+    <xacro:landing_gear offset="${distance/2}" max_angle="${max_angle}" direction="1" reverse="0" suffix="left"/>
+    <xacro:landing_gear offset="${distance/2}" max_angle="${max_angle}" direction="-1" reverse="1" suffix="right"/>
   </xacro:macro>
 </robot>

Commit message: fix

File: tobas_description/urdf/components/landing_gear/zhizicathy_electric_150.xacro (robot description, xacro)
@@ -6,7 +6,4 @@
       <parent link="lg_base_link"/>
       <child link="lg_${suffix}_top"/>
-      <axis xyz="1 0 0"/>
-      <limit velocity="${75*deg2rad/6}" effort="1" lower="0" upper="${75*deg2rad}"/>
-      <dynamics damping="0" friction="0.01"/>
     </joint>
     <link name="lg_${suffix}_top">

Commit message: modify: joint limit and dynamics

File: tobas_description/urdf/components/landing_gear/zhizicathy_electric_150.xacro (robot description, xacro)
@@ -32,6 +32,6 @@
       <child link="lg_${suffix}_bottom"/>
       <axis xyz="1 0 0"/>
-      <limit velocity="${75*deg2rad/6}" effort="1" lower="0" upper="${max_angle}"/>
-      <dynamics damping="0" friction="0.01"/>
+      <limit velocity="${75*deg2rad/6}" effort="10" lower="-0.01" upper="${max_angle}"/>
+      <dynamics damping="0" friction="0.1"/>
     </joint>
     <link name="lg_${suffix}_bottom">
