Commit message: .

File: tobas_description/urdf/components/battery/base.xacro (robot description, xacro)
@@ -10,4 +10,5 @@
     <link name="battery">
       <visual>
+        <origin xyz="0 0 0" rpy="0 0 0"/>
         <geometry>
           <box size="${x} ${y} ${z}"/>

File: tobas_description/urdf/components/battery/hrb_4s_5000mah_50c.xacro (robot description, xacro)
@@ -5,5 +5,5 @@
     <xacro:base_lipo parent="${parent}" x="0.155" y="0.048" z="0.032" mass="0.496">
       <xacro:insert_block name="origin"/>
-      <xacro:insert_block name="blue"/>
+      <xacro:insert_block name="yellow"/>
     </xacro:base_lipo>
   </xacro:macro>

File: tobas_description/urdf/components/common.xacro (robot description, xacro)
@@ -42,4 +42,9 @@
     <material name="blue">
       <color rgba="0 0 1 1"/>
+    </material>
+  </xacro:property>
+  <xacro:property name="yellow">
+    <material name="yellow">
+      <color rgba="1 1 0 1"/>
     </material>
   </xacro:property>

File: tobas_description/urdf/components/fmu/tobas_aso.xacro (robot description, xacro)
@@ -1,10 +1,10 @@
 <?xml version="1.0"?>
 <robot xmlns:xacro="http://ros.org/wiki/xacro">
-  <xacro:include filename="$(find tobas_description)/urdf/components/multirotor_base.xacro"/>
+  <xacro:include filename="$(find tobas_description)/urdf/components/common.xacro"/>
   <xacro:macro name="tobas_aso" params="parent *origin">
-    <xacro:property name="fmu_x" value="0.090"/>
-    <xacro:property name="fmu_y" value="0.062"/>
-    <xacro:property name="fmu_z" value="0.028"/>
-    <xacro:property name="fmu_mass" value="0.2"/>
+    <xacro:property name="x" value="0.090"/>
+    <xacro:property name="y" value="0.062"/>
+    <xacro:property name="z" value="0.028"/>
+    <xacro:property name="mass" value="0.2"/>
     <joint name="fmu_joint" type="fixed">
       <xacro:insert_block name="origin"/>
@@ -22,11 +22,11 @@
         <origin xyz="0 0 0.009" rpy="0 0 0"/>
         <geometry>
-          <box size="${fmu_x} ${fmu_y} ${fmu_z}"/>
+          <box size="${x} ${y} ${z}"/>
         </geometry>
       </collision>
       <inertial>
-        <mass value="${fmu_mass}"/>
+        <mass value="${mass}"/>
         <origin xyz="0 0 0.009" rpy="0 0 0"/>
-        <xacro:box_inertia x="${fmu_x}" y="${fmu_y}" z="${fmu_z}" mass="${fmu_mass}"/>
+        <xacro:box_inertia x="${x}" y="${y}" z="${z}" mass="${mass}"/>
       </inertial>
     </link>

File: tobas_description/urdf/components/propeller/phantom3_0945.xacro (robot description, xacro)
@@ -1,17 +1,19 @@
 <?xml version="1.0"?>
 <robot xmlns:xacro="http://ros.org/wiki/xacro">
-  <xacro:include filename="$(find tobas_description)/urdf/components/multirotor_base.xacro"/>
+  <xacro:include filename="$(find tobas_description)/urdf/components/common.xacro"/>
   <xacro:macro name="phantom3_0945" params="parent index direction *origin">
-    <xacro:property name="propeller_diameter" value="${9*inch2meter}"/>
-    <xacro:property name="propeller_radius" value="${propeller_diameter/2}"/>
-    <xacro:property name="propeller_height" value="0.01"/>
-    <xacro:property name="propeller_mass" value="0.011"/>
-    <joint name="propeller_${index}_joint" type="continuous">
+    <xacro:property name="diameter" value="${9*inch2meter}"/>
+    <xacro:property name="radius" value="${diameter/2}"/>
+    <xacro:property name="height" value="0.012"/>
+    <xacro:property name="mass" value="0.011"/>
+    <xacro:property name="link_name" value="propeller_${index}"/>
+    <xacro:property name="joint_name" value="${link_name}_joint"/>
+    <joint name="${joint_name}" type="continuous">
       <xacro:insert_block name="origin"/>
       <axis xyz="0 0 1"/>
       <parent link="${parent}"/>
-      <child link="propeller_${index}"/>
+      <child link="${link_name}"/>
     </joint>
-    <link name="propeller_${index}">
+    <link name="${link_name}">
       <visual>
         <geometry>
@@ -21,13 +23,13 @@
       </visual>
       <collision>
-        <origin xyz="0 0 0" rpy="0 0 0"/>
+        <origin xyz="0 0 ${height/2}" rpy="0 0 0"/>
         <geometry>
-          <cylinder radius="${propeller_radius}" length="${propeller_height}"/>
+          <cylinder radius="${radius}" length="${height}"/>
         </geometry>
       </collision>
       <inertial>
-        <mass value="${propeller_mass}"/>
-        <origin xyz="0 0 0" rpy="0 0 0"/>
-        <xacro:cylinder_inertia radius="${propeller_radius}" length="${propeller_height}" mass="${propeller_mass}"/>
+        <mass value="${mass}"/>
+        <origin xyz="0 0 ${height/2}" rpy="0 0 0"/>
+        <xacro:cylinder_inertia radius="${radius}" length="${height}" mass="${mass}"/>
       </inertial>
     </link>

File: tobas_description/urdf/f450.xacro (robot description, xacro)
@@ -10,5 +10,4 @@
   <xacro:property name="frame_width" value="0.35"/>
   <xacro:property name="frame_height" value="0.06"/>
-  <xacro:property name="frame_mass" value="0.55346"/>
   <xacro:property name="propeller_offset" value="0.225"/>
   <!-- Base Link -->
@@ -29,5 +28,5 @@
     </visual>
     <inertial>
-      <mass value="${frame_mass}"/>
+      <mass value="0.55346"/>
       <origin xyz="0 0 -4.136e-3" rpy="0 0 0"/>
       <inertia ixx="8.128e-3" ixy="0" ixz="0" iyy="8.193e-3" iyz="0" izz="1.597e-2"/>

File: tobas_description/urdf/f550_np.xacro (robot description, xacro)
@@ -9,5 +9,4 @@
   <xacro:property name="frame_radius" value="0.294"/>
   <xacro:property name="frame_height" value="0.056"/>
-  <xacro:property name="frame_mass" value="1.423"/>
   <xacro:property name="propeller_origin_z" value="0.060597"/>
   <xacro:property name="rotor_tilt" value="${30*deg2rad}"/>
@@ -29,5 +28,5 @@
     </visual>
     <inertial>
-      <mass value="${frame_mass}"/>
+      <mass value="1.423"/>
       <origin xyz="0.624e-3 1.181e-3 14.463e-3" rpy="0 0 0"/>
       <inertia ixx="3.692e-2" ixy="1.71388e-7" ixz="-2.219266e-6" iyy="3.681e-2" iyz="-5.1639988e-5" izz="7.082e-2"/>

Commit message: modify: battery models

File: tobas_description/urdf/components/battery/base.xacro (robot description, xacro)
@@ -1,11 +1,11 @@
 <robot xmlns:xacro="http://ros.org/wiki/xacro">
   <xacro:include filename="$(find tobas_description)/urdf/components/multirotor_base.xacro"/>
-  <xacro:macro name="base_lipo" params="parent x y z mass *origin *material">
-    <joint name="battery_joint" type="fixed">
+  <xacro:macro name="base_lipo" params="link_name parent x y z mass *origin *material">
+    <joint name="${link_name}_joint" type="fixed">
       <xacro:insert_block name="origin"/>
       <parent link="${parent}"/>
-      <child link="battery"/>
+      <child link="${link_name}"/>
     </joint>
-    <link name="battery">
+    <link name="${link_name}">
       <visual>
         <origin xyz="0 0 0" rpy="0 0 0"/>

File: tobas_description/urdf/components/battery/hrb_6s_1800mah_50c.xacro (robot description, xacro)
@@ -1,6 +1,6 @@
 <robot xmlns:xacro="http://ros.org/wiki/xacro">
   <xacro:include filename="$(find tobas_description)/urdf/components/battery/base.xacro"/>
-  <xacro:macro name="hrb_6s_1800mah_50c" params="parent *origin">
-    <xacro:base_lipo parent="${parent}" x="0.105" y="0.034" z="0.040" mass="0.270">
+  <xacro:macro name="hrb_6s_1800mah_50c" params="link_name parent *origin">
+    <xacro:base_lipo link_name="${link_name}" parent="${parent}" x="0.105" y="0.034" z="0.040" mass="0.270">
       <xacro:insert_block name="origin"/>
       <xacro:insert_block name="yellow"/>

File: tobas_description/urdf/components/battery/hrb_6s_5000mah_50c.xacro (robot description, xacro)
@@ -1,6 +1,6 @@
 <robot xmlns:xacro="http://ros.org/wiki/xacro">
   <xacro:include filename="$(find tobas_description)/urdf/components/battery/base.xacro"/>
-  <xacro:macro name="hrb_6s_5000mah_50c" params="parent *origin">
-    <xacro:base_lipo parent="${parent}" x="0.155" y="0.048" z="0.048" mass="0.725">
+  <xacro:macro name="hrb_6s_5000mah_50c" params="link_name parent *origin">
+    <xacro:base_lipo link_name="${link_name}" parent="${parent}" x="0.155" y="0.048" z="0.048" mass="0.725">
       <xacro:insert_block name="origin"/>
       <xacro:insert_block name="yellow"/>

File: tobas_description/urdf/components/battery/sigp_2s_1050mah_20c.xacro (robot description, xacro)
@@ -1,8 +1,8 @@
 <robot xmlns:xacro="http://ros.org/wiki/xacro">
   <xacro:include filename="$(find tobas_description)/urdf/components/battery/base.xacro"/>
-  <xacro:macro name="hrb_4s_5000mah_50c" params="link_name parent *origin">
-    <xacro:base_lipo link_name="${link_name}" parent="${parent}" x="0.155" y="0.048" z="0.032" mass="0.496">
+  <xacro:macro name="sigp_2s_1050mah_20c" params="link_name parent *origin">
+    <xacro:base_lipo link_name="${link_name}" parent="${parent}" x="0.073" y="0.035" z="0.015" mass="0.57">
       <xacro:insert_block name="origin"/>
-      <xacro:insert_block name="yellow"/>
+      <xacro:insert_block name="blue"/>
     </xacro:base_lipo>
   </xacro:macro>

File: tobas_description/urdf/components/battery/sigp_3s_2250mah_30c.xacro (robot description, xacro)
@@ -1,6 +1,6 @@
 <robot xmlns:xacro="http://ros.org/wiki/xacro">
   <xacro:include filename="$(find tobas_description)/urdf/components/battery/base.xacro"/>
-  <xacro:macro name="sigp_3s_2250mah_30c" params="parent *origin">
-    <xacro:base_lipo parent="${parent}" x="0.106" y="0.035" z="0.026" mass="0.186">
+  <xacro:macro name="sigp_3s_2250mah_30c" params="link_name parent *origin">
+    <xacro:base_lipo link_name="${link_name}" parent="${parent}" x="0.106" y="0.035" z="0.026" mass="0.186">
       <xacro:insert_block name="origin"/>
       <xacro:insert_block name="blue"/>

File: tobas_description/urdf/components/battery/sigp_3s_2250mah_60c.xacro (robot description, xacro)
@@ -1,6 +1,6 @@
 <robot xmlns:xacro="http://ros.org/wiki/xacro">
   <xacro:include filename="$(find tobas_description)/urdf/components/battery/base.xacro"/>
-  <xacro:macro name="sigp_3s_2250mah_60c" params="parent *origin">
-    <xacro:base_lipo parent="${parent}" x="0.107" y="0.035" z="0.028" mass="0.201">
+  <xacro:macro name="sigp_3s_2250mah_60c" params="link_name parent *origin">
+    <xacro:base_lipo link_name="${link_name}" parent="${parent}" x="0.107" y="0.035" z="0.028" mass="0.201">
       <xacro:insert_block name="origin"/>
       <xacro:insert_block name="blue"/>

File: tobas_description/urdf/components/battery/sigp_6s_1100mah_120c.xacro (robot description, xacro)
@@ -1,6 +1,6 @@
 <robot xmlns:xacro="http://ros.org/wiki/xacro">
   <xacro:include filename="$(find tobas_description)/urdf/components/battery/base.xacro"/>
-  <xacro:macro name="sigp_6s_1100mah_120c" params="parent *origin">
-    <xacro:base_lipo parent="${parent}" x="0.077" y="0.035" z="0.042" mass="0.205">
+  <xacro:macro name="sigp_6s_1100mah_120c" params="link_name parent *origin">
+    <xacro:base_lipo link_name="${link_name}" parent="${parent}" x="0.077" y="0.035" z="0.042" mass="0.205">
       <xacro:insert_block name="origin"/>
       <xacro:insert_block name="blue"/>

File: tobas_description/urdf/f450.xacro (robot description, xacro)
@@ -42,5 +42,5 @@
   </xacro:tobas_t1>
   <!-- Battery -->
-  <xacro:sigp_3s_2250mah_60c parent="base_link">
+  <xacro:sigp_3s_2250mah_60c link_name="battery" parent="base_link">
     <origin xyz="-0.037 0 -0.023" rpy="0 0 0"/>
   </xacro:sigp_3s_2250mah_60c>

File: tobas_description/urdf/f550.xacro (robot description, xacro)
@@ -38,5 +38,5 @@
   </xacro:tobas_t1>
   <!-- Battery -->
-  <xacro:hrb_4s_5000mah_50c parent="base_link">
+  <xacro:hrb_4s_5000mah_50c link_name="battery" parent="base_link">
     <origin xyz="0 0 -0.021" rpy="0 0 0"/>
   </xacro:hrb_4s_5000mah_50c>
