Commit message: .

File: tobas_core/tobas_description/urdf/components/common.xacro (robot description, xacro)
@@ -12,4 +12,5 @@
   <xacro:property name="rad2deg" value="${180 / pi}"/>
   <xacro:property name="inch2meter" value="0.0254"/>
+  <xacro:property name="gravity" value="9.80665"/>
   <!-- Colors -->
   <xacro:property name="black">

Commit message: .

File: tobas_core/tobas_description/urdf/components/common.xacro (robot description, xacro)
@@ -82,5 +82,5 @@
   <!-- Inertia wrt. CoM of primitive shapes -->
   <xacro:macro name="box_inertia" params="x y z mass">
-    <inertia ixx="${mass * (y*y + z*z) / 12}" ixy="0.0" ixz="0.0" iyy="${mass * (x*x + z*z) / 12}" iyz="0.0" izz="${mass * (x*x + y*y) / 12}"/>
+    <inertia ixx="${mass * (y*y + z*z) / 12}" ixy="0.0" ixz="0.0" iyy="${mass * (z*z + x*x) / 12}" iyz="0.0" izz="${mass * (x*x + y*y) / 12}"/>
   </xacro:macro>
   <xacro:macro name="cylinder_inertia" params="radius length mass">
